Commit message: Fix paths and update workflows

File: urdf/orbbec_astra.gazebo.xacro (robot description, xacro)
@@ -6,5 +6,6 @@
                        tf_prefix:=None
                        topic:=camera/depth/points
-                       frame_id:=depth">
+                       frame_id:=depth
+                       simulation_engine:=gazebo-classic">
     <xacro:if value="${tf_prefix == 'None'}">
       <xacro:property name="tf_prefix_ext" value="" />
@@ -16,5 +17,5 @@
       <visual>
         <geometry>
-            <mesh filename="file://$(find components_description)/meshes/orbbec_astra.stl" scale="0.001 0.001 0.001" />
+            <mesh filename="file://$(find ros_components_description)/meshes/orbbec_astra.stl" scale="0.001 0.001 0.001" />
         </geometry>
         <origin xyz="-0.01 0.0 0.025" rpy="${pi/2} 0.0 ${pi/2}"/>

File: urdf/ouster_os1_32.gazebo.xacro (robot description, xacro)
@@ -6,5 +6,6 @@
                        tf_prefix:=None
                        topic:=os_lidar
-                       frame_id:=os_lidar">
+                       frame_id:=os_lidar
+                       simulation_engine:=gazebo-classic">
     <xacro:if value="${use_gpu}">
       <xacro:property name="ray_type" value="gpu_ray" />
@@ -24,5 +25,5 @@
       <visual>
         <geometry>
-          <mesh filename="file://$(find components_description)/meshes/ouster_os1_32.stl" scale="1 1 0.65" />
+          <mesh filename="file://$(find ros_components_description)/meshes/ouster_os1_32.stl" scale="1 1 0.65" />
         </geometry>
         <origin xyz="0.0 0.0 0.0" rpy="0.0 0.0 ${pi/2.0}"/>

File: urdf/rplidar_s1.gazebo.xacro (robot description, xacro)
@@ -6,5 +6,6 @@
                        tf_prefix:=None
                        topic:=scan
-                       frame_id:=laser">
+                       frame_id:=laser
+                       simulation_engine:=gazebo-classic">
     <xacro:if value="${use_gpu}">
       <xacro:property name="ray_type" value="gpu_lidar" />
@@ -22,5 +23,5 @@
       <visual>
         <geometry>
-          <mesh filename="file://$(find components_description)/meshes/rplidar_s1.stl" scale="0.0001 0.0001 0.0001" />
+          <mesh filename="file://$(find ros_components_description)/meshes/rplidar_s1.stl" scale="0.0001 0.0001 0.0001" />
         </geometry>
         <origin xyz="0.0 0.0 ${0.051/2.0}" rpy="0 0 -${pi/2.0}"/>

File: urdf/velodyne_puck.gazebo.xacro (robot description, xacro)
@@ -6,5 +6,6 @@
                        tf_prefix:=None
                        topic:=scan
-                       frame_id:=velodyne">
+                       frame_id:=velodyne
+                       simulation_engine:=gazebo-classic">
     <xacro:if value="${use_gpu}">
       <xacro:property name="ray_type" value="gpu_ray" />
@@ -22,5 +23,5 @@
       <visual>
         <geometry>
-          <mesh filename="file://$(find components_description)/meshes/velodyne_puck.stl" scale="0.025035 0.025035 0.025035" />
+          <mesh filename="file://$(find ros_components_description)/meshes/velodyne_puck.stl" scale="0.025035 0.025035 0.025035" />
         </geometry>
         <origin xyz="0.0 0.0 0.0" rpy="${pi/2.0} 0.0 ${pi}"/>

Commit message: Introduce model compatibility with ROS2

File: urdf/orbbec_astra.gazebo.xacro (robot description, xacro)
@@ -1,11 +1,23 @@
 <?xml version="1.0"?>
 <robot xmlns:xacro="http://www.ros.org/wiki/xacro">
-  <xacro:macro name="orbbec_astra" params="xyz rpy prefix:=front">
-    <link name="${prefix}_orbbec_astra_link">
+  <xacro:macro name="orbbec_astra"
+               params="parent_link xyz rpy
+                       use_gpu:=false
+                       tf_prefix:=None
+                       topic:=camera/depth/points
+                       frame_id:=depth
+                       simulation_engine:=gazebo-classic">
+    <xacro:if value="${tf_prefix == 'None'}">
+      <xacro:property name="tf_prefix_ext" value="" />
+    </xacro:if>
+    <xacro:unless value="${tf_prefix == 'None'}">
+      <xacro:property name="tf_prefix_ext" value="${tf_prefix}_" />
+    </xacro:unless>
+    <link name="${tf_prefix_ext}orbbec_astra_link">
       <visual>
         <geometry>
-            <mesh filename="package://ros_components_description/meshes/orbbec_astra.stl" scale="0.001 0.001 0.001" />
+            <mesh filename="file://$(find ros_components_description)/meshes/orbbec_astra.stl" scale="0.001 0.001 0.001" />
         </geometry>
-        <origin xyz="-0.01 0 0.025" rpy="${pi/2} 0 ${pi/2}"/>
+        <origin xyz="-0.01 0.0 0.025" rpy="${pi/2} 0.0 ${pi/2}"/>
         <material name="DarkGrey"/>
       </visual>
@@ -14,5 +26,5 @@
           <box size="0.165 0.04 0.05" />
         </geometry>
-        <origin xyz="-0.01 0 0.025" rpy="0 0 ${pi/2}"/>
+        <origin xyz="-0.01 0.0 0.025" rpy="0.0 0.0 ${pi/2}"/>
       </collision>
       <inertial>
@@ -21,20 +33,26 @@
       </inertial>
     </link>
-    <link name="${prefix}_orbbec_astra_depth_link"></link>
-    <joint name="body_link_to_${prefix}_orbbec_astra_link_joint" type="fixed">
+    <link name="${tf_prefix_ext}orbbec_astra_depth_link"></link>
+    <link name="${tf_prefix_ext}${frame_id}"></link>
+    <joint name="${parent_link}_to_${tf_prefix_ext}orbbec_astra_link_joint" type="fixed">
       <origin xyz="${xyz}" rpy="${rpy}" />
-      <parent link="body_link" />
-      <child link="${prefix}_orbbec_astra_link" />
+      <parent link="${parent_link}" />
+      <child link="${tf_prefix_ext}orbbec_astra_link" />
     </joint>
-    <joint name="${prefix}_orbbec_astra_depth_link_joint" type="fixed">
-      <origin xyz="0.01 0 0.035" rpy="${-pi/2} 0 ${-pi/2}" />
-      <parent link="${prefix}_orbbec_astra_link" />
-      <child link="${prefix}_orbbec_astra_depth_link" />
+    <joint name="${tf_prefix_ext}orbbec_astra_depth_link_joint" type="fixed">
+      <origin xyz="0.01 0.0 0.035" rpy="0.0 ${pi/2} 0.0" />
+      <parent link="${tf_prefix_ext}orbbec_astra_link" />
+      <child link="${tf_prefix_ext}orbbec_astra_depth_link" />
     </joint>
-    <gazebo reference="${prefix}_orbbec_astra_link">
+    <joint name="${tf_prefix_ext}orbbec_astra_depth_link_refference_joint" type="fixed">
+      <origin xyz="0.0 0.0 0.0" rpy="${pi/2} ${-pi/2} 0.0" />
+      <parent link="${tf_prefix_ext}orbbec_astra_depth_link" />
+      <child link="${tf_prefix_ext}${frame_id}" />
+    </joint>
+    <gazebo reference="${tf_prefix_ext}orbbec_astra_link">
       <material>Gazebo/DarkGrey</material>
     </gazebo>
-    <gazebo reference="${prefix}_orbbec_astra_link">
-      <sensor type="depth" name="${prefix}_orbbec_astra_camera">
+    <gazebo reference="${tf_prefix_ext}${frame_id}">
+      <sensor type="depth" name="${tf_prefix_ext}orbbec_astra_camera">
         <always_on>1</always_on>
         <visualize>true</visualize>
@@ -57,5 +75,5 @@
           <updateRate>10.0</updateRate>
           <cameraName>camera</cameraName>
-          <frameName>${prefix}_orbbec_astra_depth_link</frameName>
+          <frameName>${tf_prefix_ext}${frame_id}</frameName>
           <imageTopicName>rgb/image_raw</imageTopicName>
           <depthImageTopicName>depth/image_raw</depthImageTopicName>
@@ -65,9 +83,9 @@
           <pointCloudCutoff>0.4</pointCloudCutoff>
           <hackBaseline>0.07</hackBaseline>
-          <distortionK1>0.0</distortionK1>
-          <distortionK2>0.0</distortionK2>
-          <distortionK3>0.0</distortionK3>
-          <distortionT1>0.0</distortionT1>
-          <distortionT2>0.0</distortionT2>
+          <distortionK1>0.07</distortionK1>
+          <distortionK2>0.00</distortionK2>
+          <distortionK3>0.00</distortionK3>
+          <distortionT1>0.00</distortionT1>
+          <distortionT2>0.00</distortionT2>
           <CxPrime>0.0</CxPrime>
           <Cx>0.0</Cx>

File: urdf/ouster_os1_32.gazebo.xacro (robot description, xacro)
@@ -1,26 +1,30 @@
 <?xml version="1.0"?>
 <robot xmlns:xacro="http://www.ros.org/wiki/xacro">
-  <xacro:macro name="ouster_os1_32" params="xyz rpy use_gpu:=false prefix:=front topic:=laser/scan">
-    <xacro:if value="${use_gpu}">
-      <xacro:property name="ray_type" value="gpu_ray" />
-      <xacro:property name="plugin_file_name" value="libgazebo_ros_gpu_laser.so" />
+    <xacro:macro name="ouster_os1_32"
+               params="parent_link xyz rpy
+                       use_gpu:=false
+                       tf_prefix:=None
+                       topic:=os_lidar
+                       frame_id:=os_lidar
+                       simulation_engine:=gazebo-classic">
+    <xacro:if value="${tf_prefix == 'None'}">
+      <xacro:property name="tf_prefix_ext" value="" />
     </xacro:if>
-    <xacro:unless value="${use_gpu}">
-      <xacro:property name="ray_type" value="ray" />
-      <xacro:property name="plugin_file_name" value="libgazebo_ros_laser.so" />
+    <xacro:unless value="${tf_prefix == 'None'}">
+      <xacro:property name="tf_prefix_ext" value="${tf_prefix}" />
     </xacro:unless>
-    <link name="os_sensor">
+    <link name="${tf_prefix_ext}ouster_os1_32_link">
       <visual>
         <geometry>
-          <mesh filename="package://ros_components_description/meshes/ouster_os1_32.stl" scale="1 1 0.65" />
+          <mesh filename="file://$(find ros_components_description)/meshes/ouster_os1_32.stl" scale="1 1 0.65" />
         </geometry>
-        <origin xyz="0 0 0" rpy="0 0 ${pi/2}"/>
+        <origin xyz="0.0 0.0 0.0" rpy="0.0 0.0 ${pi/2.0}"/>
         <material name="Grey"/>
       </visual>
       <collision>
         <geometry>
-          <cylinder radius="${0.0753/2}" length="0.0435" />
+          <cylinder radius="${0.0753/2.0}" length="0.0435" />
         </geometry>
-        <origin xyz="0 0 ${0.0435/2}" rpy="0 0 0"/>
+        <origin xyz="0.0 0.0 ${0.0435/2.0}" rpy="0.0 0.0 0.0"/>
       </collision>
       <inertial>
@@ -29,21 +33,20 @@
       </inertial>
     </link>
-    <link name="os_laser"></link>
-    <joint name="body_link_to_os_sensor_joint" type="fixed">
+    <link name="${tf_prefix_ext}${frame_id}"></link>
+    <joint name="${parent_link}_to_${tf_prefix_ext}ouster_os1_32_link_joint" type="fixed">
       <origin xyz="${xyz}" rpy="${rpy}" />
-      <parent link="body_link" />
-      <child link="os_sensor" />
+      <parent link="${parent_link}" />
+      <child link="${tf_prefix_ext}ouster_os1_32_link" />
     </joint>
-    <joint name="os_laser_joint" type="fixed">
+    <joint name="${tf_prefix_ext}ouster_os1_32_link_to_${tf_prefix_ext}${frame_id}_joint" type="fixed">
       <origin xyz="0 0 0.023" rpy="0 0 0" />
-      <parent link="os_sensor" />
-      <child link="os_laser" />
+      <parent link="${tf_prefix_ext}ouster_os1_32_link" />
+      <child link="${tf_prefix_ext}${frame_id}" />
     </joint>
-    <gazebo reference="os_sensor">
+    <gazebo reference="${tf_prefix_ext}ouster_os1_32_link">
       <material>Gazebo/Grey</material>
     </gazebo>
-    <gazebo reference="os_laser">
-      <sensor type="ray" name="ouster_os1_32_sensor">
-        <pose>0 0 0.0 0 0 0</pose>
+    <gazebo reference="${tf_prefix_ext}${frame_id}">
+      <sensor type="ray" name="${tf_prefix_ext}ouster_os1_32_sensor">
         <visualize>false</visualize>
         <update_rate>10</update_rate>
@@ -74,7 +77,7 @@
           </noise>
         </ray>
-        <plugin name="gazebo_ros_block_laser_controller" filename="libgazebo_ros_block_laser.so">
+        <plugin name="ray" filename="libgazebo_ros_block_laser.so">
           <topicName>${topic}</topicName>
-          <frameName>os_laser</frameName>
+          <frameName>${tf_prefix_ext}${frame_id}</frameName>
           <gaussianNoise>0.0008</gaussianNoise>
           <updateRate>10</updateRate>

File: urdf/rplidar_s1.gazebo.xacro (robot description, xacro)
@@ -1,5 +1,11 @@
 <?xml version="1.0"?>
 <robot xmlns:xacro="http://www.ros.org/wiki/xacro">
-  <xacro:macro name="rplidar_s1" params="xyz rpy use_gpu:=false prefix:=front topic:=laser/scan">
+  <xacro:macro name="rplidar_s1"
+               params="parent_link xyz rpy
+                       use_gpu:=false
+                       tf_prefix:=None
+                       topic:=rp_scan
+                       frame_id:=rp_laser
+                       simulation_engine:=gazebo-classic">
     <xacro:if value="${use_gpu}">
       <xacro:property name="ray_type" value="gpu_ray" />
@@ -10,17 +16,23 @@
       <xacro:property name="plugin_file_name" value="libgazebo_ros_laser.so" />
     </xacro:unless>
-    <link name="${prefix}_rplidar_s1_link">
+    <xacro:if value="${tf_prefix == 'None'}">
+      <xacro:property name="tf_prefix_ext" value="" />
+    </xacro:if>
+    <xacro:unless value="${tf_prefix == 'None'}">
+      <xacro:property name="tf_prefix_ext" value="${tf_prefix}_" />
+    </xacro:unless>
+    <link name="${tf_prefix_ext}rplidar_s1_link">
       <visual>
         <geometry>
-          <mesh filename="package://ros_components_description/meshes/rplidar_s1.stl" scale="0.0001 0.0001 0.0001" />
+          <mesh filename="file://$(find ros_components_description)/meshes/rplidar_s1.stl" scale="0.0001 0.0001 0.0001" />
         </geometry>
-        <origin xyz="0 0 ${0.051/2}" rpy="0 0 -${pi/2}"/>
+        <origin xyz="0.0 0.0 ${0.051/2.0}" rpy="0 0 -${pi/2.0}"/>
         <material name="DarkGrey"/>
       </visual>
       <collision>
         <geometry>
-          <cylinder radius="${0.0555/2}" length="0.051" />
+          <cylinder radius="${0.0555/2.0}" length="0.051" />
         </geometry>
-        <origin xyz="0 0 ${0.051/2}" rpy="0 0 0"/>
+        <origin xyz="0.0 0.0 ${0.051/2.0}" rpy="0.0 0.0 0.0"/>
       </collision>
       <inertial>
@@ -29,20 +41,20 @@
       </inertial>
     </link>
-    <link name="${prefix}_rplidar_s1_laser_link"></link>
-    <joint name="body_link_to_${prefix}_rplidar_s1_link_joint" type="fixed">
+    <link name="${tf_prefix_ext}${frame_id}"></link>
+    <joint name="${parent_link}_to_${tf_prefix_ext}rplidar_s1_link_joint" type="fixed">
       <origin xyz="${xyz}" rpy="${rpy}" />
-      <parent link="body_link" />
-      <child link="${prefix}_rplidar_s1_link" />
+      <parent link="${parent_link}" />
+      <child link="${tf_prefix_ext}rplidar_s1_link" />
     </joint>
-    <joint name="${prefix}_rplidar_s1_laser_link_joint" type="fixed">
-      <origin xyz="0 0 0.04" rpy="0 0 0" />
-      <parent link="${prefix}_rplidar_s1_link" />
-      <child link="${prefix}_rplidar_s1_laser_link" />
+    <joint name="${tf_prefix_ext}${frame_id}_joint" type="fixed">
+      <origin xyz="0 0 0.04" rpy="0.0 0.0 0.0" />
+      <parent link="${tf_prefix_ext}rplidar_s1_link" />
+      <child link="${tf_prefix_ext}${frame_id}" />
     </joint>
-    <gazebo reference="${prefix}_rplidar_s1_link">
+    <gazebo reference="${tf_prefix_ext}rplidar_s1_link">
       <material>Gazebo/DarkGrey</material>
     </gazebo>
-    <gazebo reference="${prefix}_rplidar_s1_laser_link">
-      <sensor type="${ray_type}" name="${prefix}_rplidar_s1_sensor">
+    <gazebo reference="${tf_prefix_ext}${frame_id}">
+      <sensor type="${ray_type}" name="${tf_prefix_ext}rplidar_s1_sensor">
         <pose>0 0 0.04 0 0 0</pose>
         <visualize>false</visualize>
@@ -68,7 +80,7 @@
           </noise>
         </ray>
-        <plugin name="gazebo_ros_head_rplidar_controller" filename="${plugin_file_name}">
+        <plugin name="${ray_type}" filename="${plugin_file_name}">
           <topicName>${topic}</topicName>
-          <frameName>${prefix}_rplidar_s1_laser_link</frameName>
+          <frameName>${tf_prefix_ext}${frame_id}</frameName>
         </plugin>
       </sensor>

File: urdf/velodyne_puck.gazebo.xacro (robot description, xacro)
@@ -1,18 +1,36 @@
 <?xml version="1.0"?>
 <robot xmlns:xacro="http://www.ros.org/wiki/xacro">
-  <xacro:macro name="velodyne_puck" params="xyz rpy use_gpu:=false prefix:=front topic:=laser/scan">
-    <link name="${prefix}_velodyne_puck_link">
+  <xacro:macro name="velodyne_puck"
+               params="parent_link xyz rpy
+                       use_gpu:=false
+                       tf_prefix:=None
+                       topic:=scan
+                       frame_id:=velodyne
+                       simulation_engine:=gazebo-classic">
+    <xacro:if value="${use_gpu}">
+      <xacro:property name="ray_type" value="gpu_ray" />
+    </xacro:if>
+    <xacro:unless value="${use_gpu}">
+      <xacro:property name="ray_type" value="ray" />
+    </xacro:unless>
+    <xacro:if value="${tf_prefix == 'None'}">
+      <xacro:property name="tf_prefix_ext" value="" />
+    </xacro:if>
+    <xacro:unless value="${tf_prefix == 'None'}">
+      <xacro:property name="tf_prefix_ext" value="${tf_prefix}_" />
+    </xacro:unless>
+    <link name="${tf_prefix_ext}velodyne_puck_link">
       <visual>
         <geometry>
-          <mesh filename="package://ros_components_description/meshes/velodyne_puck.stl" scale="0.025035 0.025035 0.025035" />
+          <mesh filename="file://$(find ros_components_description)/meshes/velodyne_puck.stl" scale="0.025035 0.025035 0.025035" />
         </geometry>
-        <origin xyz="0 0 0" rpy="${pi/2} 0 ${pi}"/>
+        <origin xyz="0.0 0.0 0.0" rpy="${pi/2.0} 0.0 ${pi}"/>
         <material name="DarkGrey"/>
       </visual>
       <collision>
         <geometry>
-          <cylinder radius="${0.090/2}" length="0.0717" />
+          <cylinder radius="${0.090/2.0}" length="0.0717" />
         </geometry>
-        <origin xyz="0 0 ${0.0717/2}" rpy="0 0 0"/>
+        <origin xyz="0.0 0.0 ${0.0717/2.0}" rpy="0.0 0.0 0.0"/>
       </collision>
       <inertial>
@@ -21,20 +39,20 @@
       </inertial>
     </link>
-    <link name="${prefix}_velodyne_puck_laser_link"></link>
-    <joint name="body_link_to_${prefix}_velodyne_puck_link_joint" type="fixed">
+    <link name="${tf_prefix_ext}${frame_id}"></link>
+    <joint name="${parent_link}_to_${tf_prefix_ext}velodyne_puck_link_joint" type="fixed">
       <origin xyz="${xyz}" rpy="${rpy}" />
-      <parent link="body_link" />
-      <child link="${prefix}_velodyne_puck_link" />
+      <parent link="${parent_link}" />
+      <child link="${tf_prefix_ext}velodyne_puck_link" />
     </joint>
-    <joint name="${prefix}_velodyne_puck_laser_link_joint" type="fixed">
-      <origin xyz="0 0 0.0378" rpy="0 0 0" />
-      <parent link="${prefix}_velodyne_puck_link" />
-      <child link="${prefix}_velodyne_puck_laser_link" />
+    <joint name="${tf_prefix_ext}velodyne_puck_link_joint_to_${tf_prefix_ext}${frame_id}_joint" type="fixed">
+      <origin xyz="0.0 0.0 0.0378" rpy="0.0 0.0 0.0" />
+      <parent link="${tf_prefix_ext}velodyne_puck_link" />
+      <child link="${tf_prefix_ext}${frame_id}" />
     </joint>
-    <gazebo reference="${prefix}_velodyne_puck_link">
+    <gazebo reference="${tf_prefix_ext}velodyne_puck_link">
       <material>Gazebo/DarkGrey</material>
     </gazebo>
-    <gazebo reference="${prefix}_velodyne_puck_laser_link">
-      <sensor type="ray" name="${prefix}_velodyne_puck_sensor">
+    <gazebo reference="${tf_prefix_ext}${frame_id}">
+      <sensor type="ray" name="${tf_prefix_ext}velodyne_puck_sensor">
         <pose>0 0 0.0378 0 0 0</pose>
         <visualize>false</visualize>
@@ -56,5 +74,5 @@
           </scan>
           <range>
-            <min>${0.051+0.01}</min>
+            <min>0.061</min>
             <max>100.0</max>
             <resolution>0.005</resolution>
@@ -68,5 +86,5 @@
         <plugin name="gazebo_ros_block_laser_controller" filename="libgazebo_ros_block_laser.so">
           <topicName>${topic}</topicName>
-          <frameName>${prefix}_velodyne_puck_laser_link</frameName>
+          <frameName>${tf_prefix_ext}${frame_id}</frameName>
           <gaussianNoise>0.0008</gaussianNoise>
           <updateRate>10</updateRate>
