Commit message: compliance with the coding style

File: urdf/orbbec_astra.gazebo.xacro (robot description, xacro)
@@ -14,10 +14,15 @@
       <xacro:property name="tf_prefix_ext" value="${tf_prefix}_" />
     </xacro:unless>
+    <joint name="${parent_link}_to_${tf_prefix_ext}orbbec_astra_link_joint" type="fixed">
+      <origin xyz="${xyz}" rpy="${rpy}" />
+      <parent link="${parent_link}" />
+      <child link="${tf_prefix_ext}orbbec_astra_link" />
+    </joint>
     <link name="${tf_prefix_ext}orbbec_astra_link">
       <visual>
         <geometry>
-            <mesh filename="file://$(find ros_components_description)/meshes/orbbec_astra.stl" scale="0.001 0.001 0.001" />
+          <mesh filename="file://$(find ros_components_description)/meshes/orbbec_astra.stl" scale="0.001 0.001 0.001" />
         </geometry>
-        <origin xyz="-0.01 0.0 0.025" rpy="${pi/2} 0.0 ${pi/2}"/>
+        <origin xyz="-0.01 0 0.025" rpy="${pi/2} 0 ${pi/2}"/>
         <material name="DarkGrey"/>
       </visual>
@@ -26,5 +31,5 @@
           <box size="0.165 0.04 0.05" />
         </geometry>
-        <origin xyz="-0.01 0.0 0.025" rpy="0.0 0.0 ${pi/2}"/>
+        <origin xyz="-0.01 0 0.025" rpy="0 0 ${pi/2}"/>
       </collision>
       <inertial>
@@ -33,25 +38,11 @@
       </inertial>
     </link>
-    <link name="${tf_prefix_ext}orbbec_astra_depth_link"></link>
-    <link name="${tf_prefix_ext}${frame_id}"></link>
-    <joint name="${parent_link}_to_${tf_prefix_ext}orbbec_astra_link_joint" type="fixed">
-      <origin xyz="${xyz}" rpy="${rpy}" />
-      <parent link="${parent_link}" />
-      <child link="${tf_prefix_ext}orbbec_astra_link" />
-    </joint>
-    <joint name="${tf_prefix_ext}orbbec_astra_depth_link_joint" type="fixed">
-      <origin xyz="0.01 0.0 0.035" rpy="0.0 ${pi/2} 0.0" />
+    <joint name="${tf_prefix_ext}${frame_id}_link_joint" type="fixed">
+      <origin xyz="0.01 0 0.035" rpy="${-pi/2} 0 ${-pi/2}" />
       <parent link="${tf_prefix_ext}orbbec_astra_link" />
-      <child link="${tf_prefix_ext}orbbec_astra_depth_link" />
-    </joint>
-    <joint name="${tf_prefix_ext}orbbec_astra_depth_link_refference_joint" type="fixed">
-      <origin xyz="0.0 0.0 0.0" rpy="${pi/2} ${-pi/2} 0.0" />
-      <parent link="${tf_prefix_ext}orbbec_astra_depth_link" />
       <child link="${tf_prefix_ext}${frame_id}" />
     </joint>
+    <link name="${tf_prefix_ext}${frame_id}"></link>
     <gazebo reference="${tf_prefix_ext}orbbec_astra_link">
-      <material>Gazebo/DarkGrey</material>
-    </gazebo>
-    <gazebo reference="${tf_prefix_ext}${frame_id}">
       <sensor type="depth" name="${tf_prefix_ext}orbbec_astra_camera">
         <always_on>1</always_on>
@@ -83,9 +74,9 @@
           <pointCloudCutoff>0.4</pointCloudCutoff>
           <hackBaseline>0.07</hackBaseline>
-          <distortionK1>0.07</distortionK1>
-          <distortionK2>0.00</distortionK2>
-          <distortionK3>0.00</distortionK3>
-          <distortionT1>0.00</distortionT1>
-          <distortionT2>0.00</distortionT2>
+          <distortionK1>0.0</distortionK1>
+          <distortionK2>0.0</distortionK2>
+          <distortionK3>0.0</distortionK3>
+          <distortionT1>0.0</distortionT1>
+          <distortionT2>0.0</distortionT2>
           <CxPrime>0.0</CxPrime>
           <Cx>0.0</Cx>
@@ -95,4 +86,7 @@
       </sensor>
     </gazebo>
+    <gazebo reference="${tf_prefix_ext}orbbec_astra_link">
+      <material>Gazebo/DarkGrey</material>
+    </gazebo>
   </xacro:macro>
 </robot>

File: urdf/ouster_os1_32.gazebo.xacro (robot description, xacro)
@@ -14,4 +14,9 @@
       <xacro:property name="tf_prefix_ext" value="${tf_prefix}" />
     </xacro:unless>
+    <joint name="${parent_link}_to_${tf_prefix_ext}ouster_os1_32_link_joint" type="fixed">
+      <origin xyz="${xyz}" rpy="${rpy}" />
+      <parent link="${parent_link}" />
+      <child link="${tf_prefix_ext}ouster_os1_32_link" />
+    </joint>
     <link name="${tf_prefix_ext}ouster_os1_32_link">
       <visual>
@@ -33,10 +38,4 @@
       </inertial>
     </link>
-    <link name="${tf_prefix_ext}${frame_id}"></link>
-    <joint name="${parent_link}_to_${tf_prefix_ext}ouster_os1_32_link_joint" type="fixed">
-      <origin xyz="${xyz}" rpy="${rpy}" />
-      <parent link="${parent_link}" />
-      <child link="${tf_prefix_ext}ouster_os1_32_link" />
-    </joint>
     <joint name="${tf_prefix_ext}ouster_os1_32_link_to_${tf_prefix_ext}${frame_id}_joint" type="fixed">
       <origin xyz="0 0 0.023" rpy="0 0 0" />
@@ -44,7 +43,5 @@
       <child link="${tf_prefix_ext}${frame_id}" />
     </joint>
-    <gazebo reference="${tf_prefix_ext}ouster_os1_32_link">
-      <material>Gazebo/Grey</material>
-    </gazebo>
+    <link name="${tf_prefix_ext}${frame_id}"></link>
     <gazebo reference="${tf_prefix_ext}${frame_id}">
       <sensor type="ray" name="${tf_prefix_ext}ouster_os1_32_sensor">
@@ -85,4 +82,7 @@
       </sensor>
     </gazebo>
+    <gazebo reference="${tf_prefix_ext}ouster_os1_32_link">
+      <material>Gazebo/Grey</material>
+    </gazebo>
   </xacro:macro>
 </robot>

File: urdf/rplidar_s1.gazebo.xacro (robot description, xacro)
@@ -22,4 +22,9 @@
       <xacro:property name="tf_prefix_ext" value="${tf_prefix}_" />
     </xacro:unless>
+    <joint name="${parent_link}_to_${tf_prefix_ext}rplidar_s1_link_joint" type="fixed">
+      <origin xyz="${xyz}" rpy="${rpy}" />
+      <parent link="${parent_link}" />
+      <child link="${tf_prefix_ext}rplidar_s1_link" />
+    </joint>
     <link name="${tf_prefix_ext}rplidar_s1_link">
       <visual>
@@ -41,18 +46,10 @@
       </inertial>
     </link>
-    <link name="${tf_prefix_ext}${frame_id}"></link>
-    <joint name="${parent_link}_to_${tf_prefix_ext}rplidar_s1_link_joint" type="fixed">
-      <origin xyz="${xyz}" rpy="${rpy}" />
-      <parent link="${parent_link}" />
-      <child link="${tf_prefix_ext}rplidar_s1_link" />
-    </joint>
-    <joint name="${tf_prefix_ext}${frame_id}_joint" type="fixed">
+    <joint name="${tf_prefix_ext}rplidar_s1_to_${tf_prefix_ext}${frame_id}_joint" type="fixed">
       <origin xyz="0 0 0.04" rpy="0.0 0.0 0.0" />
       <parent link="${tf_prefix_ext}rplidar_s1_link" />
       <child link="${tf_prefix_ext}${frame_id}" />
     </joint>
-    <gazebo reference="${tf_prefix_ext}rplidar_s1_link">
-      <material>Gazebo/DarkGrey</material>
-    </gazebo>
+    <link name="${tf_prefix_ext}${frame_id}"></link>
     <gazebo reference="${tf_prefix_ext}${frame_id}">
       <sensor type="${ray_type}" name="${tf_prefix_ext}rplidar_s1_sensor">
@@ -86,4 +83,7 @@
       </sensor>
     </gazebo>
+    <gazebo reference="${tf_prefix_ext}rplidar_s1_link">
+      <material>Gazebo/DarkGrey</material>
+    </gazebo>
   </xacro:macro>
 </robot>

File: urdf/velodyne_puck.gazebo.xacro (robot description, xacro)
@@ -20,4 +20,9 @@
       <xacro:property name="tf_prefix_ext" value="${tf_prefix}_" />
     </xacro:unless>
+    <joint name="${parent_link}_to_${tf_prefix_ext}velodyne_puck_link_joint" type="fixed">
+      <origin xyz="${xyz}" rpy="${rpy}" />
+      <parent link="${parent_link}" />
+      <child link="${tf_prefix_ext}velodyne_puck_link" />
+    </joint>
     <link name="${tf_prefix_ext}velodyne_puck_link">
       <visual>
@@ -39,21 +44,12 @@
       </inertial>
     </link>
-    <link name="${tf_prefix_ext}${frame_id}"></link>
-    <joint name="${parent_link}_to_${tf_prefix_ext}velodyne_puck_link_joint" type="fixed">
-      <origin xyz="${xyz}" rpy="${rpy}" />
-      <parent link="${parent_link}" />
-      <child link="${tf_prefix_ext}velodyne_puck_link" />
-    </joint>
-    <joint name="${tf_prefix_ext}velodyne_puck_link_joint_to_${tf_prefix_ext}${frame_id}_joint" type="fixed">
+    <joint name="${tf_prefix_ext}velodyne_puck_link_to_${tf_prefix_ext}${frame_id}_joint" type="fixed">
       <origin xyz="0.0 0.0 0.0378" rpy="0.0 0.0 0.0" />
       <parent link="${tf_prefix_ext}velodyne_puck_link" />
       <child link="${tf_prefix_ext}${frame_id}" />
     </joint>
-    <gazebo reference="${tf_prefix_ext}velodyne_puck_link">
-      <material>Gazebo/DarkGrey</material>
-    </gazebo>
+    <link name="${tf_prefix_ext}${frame_id}"></link>
     <gazebo reference="${tf_prefix_ext}${frame_id}">
       <sensor type="ray" name="${tf_prefix_ext}velodyne_puck_sensor">
-        <pose>0 0 0.0378 0 0 0</pose>
         <visualize>false</visualize>
         <update_rate>10</update_rate>
@@ -61,5 +57,5 @@
           <scan>
             <horizontal>
-              <samples>3600</samples>
+              <samples>1024</samples>
               <resolution>1</resolution>
               <min_angle>-${pi}</min_angle>
@@ -74,7 +70,7 @@
           </scan>
           <range>
-            <min>0.061</min>
+            <min>${0.051+0.01}</min>
             <max>100.0</max>
-            <resolution>0.005</resolution>
+            <resolution>0.003</resolution>
           </range>
           <noise>
@@ -84,5 +80,5 @@
           </noise>
         </ray>
-        <plugin name="gazebo_ros_block_laser_controller" filename="libgazebo_ros_block_laser.so">
+        <plugin name="ray" filename="libgazebo_ros_block_laser.so">
           <topicName>${topic}</topicName>
           <frameName>${tf_prefix_ext}${frame_id}</frameName>
@@ -92,4 +88,7 @@
       </sensor>
     </gazebo>
+    <gazebo reference="${tf_prefix_ext}velodyne_puck_link">
+      <material>Gazebo/DarkGrey</material>
+    </gazebo>
   </xacro:macro>
 </robot>

Commit message: compliance with the coding style

File: urdf/orbbec_astra.gazebo.xacro (robot description, xacro)
@@ -14,8 +14,13 @@
       <xacro:property name="tf_prefix_ext" value="${tf_prefix}_" />
     </xacro:unless>
+    <joint name="${parent_link}_to_${tf_prefix_ext}orbbec_astra_link_joint" type="fixed">
+      <origin xyz="${xyz}" rpy="${rpy}" />
+      <parent link="${parent_link}" />
+      <child link="${tf_prefix_ext}orbbec_astra_link" />
+    </joint>
     <link name="${tf_prefix_ext}orbbec_astra_link">
       <visual>
         <geometry>
-            <mesh filename="file://$(find ros_components_description)/meshes/orbbec_astra.stl" scale="0.001 0.001 0.001" />
+          <mesh filename="file://$(find ros_components_description)/meshes/orbbec_astra.stl" scale="0.001 0.001 0.001" />
         </geometry>
         <origin xyz="-0.01 0.0 0.025" rpy="${pi/2} 0.0 ${pi/2}"/>
@@ -29,41 +34,19 @@
       </collision>
       <inertial>
-          <mass value="0.105" />
-          <inertia ixx="1" ixy="0" ixz="0" iyy="1" iyz="0" izz="1" />
+        <mass value="0.105" />
+        <inertia ixx="1.0" ixy="0.0" ixz="0.0" iyy="1.0" iyz="0.0" izz="1.0" />
       </inertial>
     </link>
-    <link name="${tf_prefix_ext}orbbec_astra_depth_link"></link>
-    <link name="${tf_prefix_ext}${frame_id}"></link>
-    <joint name="${parent_link}_to_${tf_prefix_ext}orbbec_astra_link_joint" type="fixed">
-      <origin xyz="${xyz}" rpy="${rpy}" />
-      <parent link="${parent_link}" />
-      <child link="${tf_prefix_ext}orbbec_astra_link" />
-    </joint>
-    <joint name="${tf_prefix_ext}orbbec_astra_depth_link_joint" type="fixed">
-      <origin xyz="0.01 0.0 0.035" rpy="0.0 ${pi/2} 0.0" />
+    <joint name="${tf_prefix_ext}${frame_id}_link_joint" type="fixed">
+      <origin xyz="0.01 0.0 0.035" rpy="${-pi/2.0} 0.0 ${-pi/2.0}" />
       <parent link="${tf_prefix_ext}orbbec_astra_link" />
-      <child link="${tf_prefix_ext}orbbec_astra_depth_link" />
-    </joint>
-    <joint name="${tf_prefix_ext}orbbec_astra_depth_link_refference_joint" type="fixed">
-      <origin xyz="0.0 0.0 0.0" rpy="${pi/2} ${-pi/2} 0.0" />
-      <parent link="${tf_prefix_ext}orbbec_astra_depth_link" />
       <child link="${tf_prefix_ext}${frame_id}" />
     </joint>
+    <link name="${tf_prefix_ext}${frame_id}"></link>
     <gazebo reference="${tf_prefix_ext}orbbec_astra_link">
-      <material>Gazebo/DarkGrey</material>
-    </gazebo>
-    <gazebo reference="${tf_prefix_ext}${frame_id}">
       <sensor type="depth" name="${tf_prefix_ext}orbbec_astra_camera">
         <always_on>1</always_on>
         <update_rate>10</update_rate>
         <camera name="${tf_prefix_ext}camera">
-          <distortion>
-            <k1>0.07</k1>
-            <k2>0.00</k2>
-            <k3>0.00</k3>
-            <p1>0.00</p1>
-            <p2>0.00</p2>
-            <center>0.0 0.0</center>
-          </distortion>
         </camera>
         <plugin name="plugin_name" filename="libgazebo_ros_camera.so">
@@ -84,4 +67,7 @@
       </sensor>
     </gazebo>
+    <gazebo reference="${tf_prefix_ext}orbbec_astra_link">
+      <material>Gazebo/DarkGrey</material>
+    </gazebo>
   </xacro:macro>
 </robot>

File: urdf/ouster_os1_32.gazebo.xacro (robot description, xacro)
@@ -10,9 +10,7 @@
     <xacro:if value="${use_gpu}">
       <xacro:property name="ray_type" value="gpu_ray" />
-      <xacro:property name="plugin_file_name" value="libgazebo_ros_gpu_ray_sensor.so" />
     </xacro:if>
     <xacro:unless value="${use_gpu}">
       <xacro:property name="ray_type" value="ray" />
-      <xacro:property name="plugin_file_name" value="libgazebo_ros_ray_sensor.so" />
     </xacro:unless>
     <xacro:if value="${tf_prefix == 'None'}">
@@ -22,8 +20,13 @@
       <xacro:property name="tf_prefix_ext" value="${tf_prefix}" />
     </xacro:unless>
+    <joint name="${parent_link}_to_${tf_prefix_ext}ouster_os1_32_link_joint" type="fixed">
+      <origin xyz="${xyz}" rpy="${rpy}" />
+      <parent link="${parent_link}" />
+      <child link="${tf_prefix_ext}ouster_os1_32_link" />
+    </joint>
     <link name="${tf_prefix_ext}ouster_os1_32_link">
       <visual>
         <geometry>
-          <mesh filename="file://$(find ros_components_description)/meshes/ouster_os1_32.stl" scale="1 1 0.65" />
+          <mesh filename="file://$(find ros_components_description)/meshes/ouster_os1_32.stl" scale="1.0 1.0 0.65" />
         </geometry>
         <origin xyz="0.0 0.0 0.0" rpy="0.0 0.0 ${pi/2.0}"/>
@@ -38,21 +41,13 @@
       <inertial>
           <mass value="0.447" />
-          <inertia ixx="1" ixy="0" ixz="0" iyy="1" iyz="0" izz="1" />
+          <inertia ixx="1.0" ixy="0.0" ixz="0.0" iyy="1.0" iyz="0.0" izz="1.0" />
       </inertial>
     </link>
-    <link name="${tf_prefix_ext}${frame_id}"></link>
-    <joint name="${parent_link}_to_${tf_prefix_ext}ouster_os1_32_link_joint" type="fixed">
-      <origin xyz="${xyz}" rpy="${rpy}" />
-      <parent link="${parent_link}" />
-      <child link="${tf_prefix_ext}ouster_os1_32_link" />
-    </joint>
     <joint name="${tf_prefix_ext}ouster_os1_32_link_to_${tf_prefix_ext}${frame_id}_joint" type="fixed">
-      <origin xyz="0 0 0.023" rpy="0 0 0" />
+      <origin xyz="0.0 0.0 0.023" rpy="0.0 0.0 0.0" />
       <parent link="${tf_prefix_ext}ouster_os1_32_link" />
       <child link="${tf_prefix_ext}${frame_id}" />
     </joint>
-    <gazebo reference="${tf_prefix_ext}ouster_os1_32_link">
-      <material>Gazebo/Grey</material>
-    </gazebo>
+    <link name="${tf_prefix_ext}${frame_id}"></link>
     <gazebo reference="${tf_prefix_ext}${frame_id}">
       <sensor type="${ray_type}" name="${tf_prefix_ext}ouster_os1_32_sensor">
@@ -95,4 +90,7 @@
       </sensor>
     </gazebo>
+    <gazebo reference="${tf_prefix_ext}ouster_os1_32_link">
+      <material>Gazebo/Grey</material>
+    </gazebo>
   </xacro:macro>
 </robot>

File: urdf/rplidar_s1.gazebo.xacro (robot description, xacro)
@@ -20,4 +20,9 @@
       <xacro:property name="tf_prefix_ext" value="${tf_prefix}_" />
     </xacro:unless>
+    <joint name="${parent_link}_to_${tf_prefix_ext}rplidar_s1_link_joint" type="fixed">
+      <origin xyz="${xyz}" rpy="${rpy}" />
+      <parent link="${parent_link}" />
+      <child link="${tf_prefix_ext}rplidar_s1_link" />
+    </joint>
     <link name="${tf_prefix_ext}rplidar_s1_link">
       <visual>
@@ -25,5 +30,5 @@
           <mesh filename="file://$(find ros_components_description)/meshes/rplidar_s1.stl" scale="0.0001 0.0001 0.0001" />
         </geometry>
-        <origin xyz="0.0 0.0 ${0.051/2.0}" rpy="0 0 -${pi/2.0}"/>
+        <origin xyz="0.0 0.0 ${0.051/2.0}" rpy="0.0 0.0 -${pi/2.0}"/>
         <material name="DarkGrey"/>
       </visual>
@@ -36,21 +41,13 @@
       <inertial>
         <mass value="0.105" />
-        <inertia ixx="1" ixy="0" ixz="0" iyy="1" iyz="0" izz="1" />
+        <inertia ixx="1.0" ixy="0.0" ixz="0.0" iyy="1.0" iyz="0.0" izz="1.0" />
       </inertial>
     </link>
-    <link name="${tf_prefix_ext}${frame_id}"></link>
-    <joint name="${parent_link}_to_${tf_prefix_ext}rplidar_s1_link_joint" type="fixed">
-      <origin xyz="${xyz}" rpy="${rpy}" />
-      <parent link="${parent_link}" />
-      <child link="${tf_prefix_ext}rplidar_s1_link" />
-    </joint>
     <joint name="${tf_prefix_ext}${frame_id}_joint" type="fixed">
-      <origin xyz="0 0 0.04" rpy="0.0 0.0 0.0" />
+      <origin xyz="0.0 0.0 0.04" rpy="0.0 0.0 0.0" />
       <parent link="${tf_prefix_ext}rplidar_s1_link" />
       <child link="${tf_prefix_ext}${frame_id}" />
     </joint>
-    <gazebo reference="${tf_prefix_ext}rplidar_s1_link">
-      <material>Gazebo/DarkGrey</material>
-    </gazebo>
+    <link name="${tf_prefix_ext}${frame_id}"></link>
     <gazebo reference="${tf_prefix_ext}${frame_id}">
       <sensor type="${ray_type}" name="${tf_prefix_ext}rplidar_s1_sensor">
@@ -87,4 +84,7 @@
       </sensor>
     </gazebo>
+    <gazebo reference="${tf_prefix_ext}rplidar_s1_link">
+      <material>Gazebo/DarkGrey</material>
+    </gazebo>
   </xacro:macro>
 </robot>

File: urdf/velodyne_puck.gazebo.xacro (robot description, xacro)
@@ -20,4 +20,9 @@
       <xacro:property name="tf_prefix_ext" value="${tf_prefix}_" />
     </xacro:unless>
+    <joint name="${parent_link}_to_${tf_prefix_ext}velodyne_puck_link_joint" type="fixed">
+      <origin xyz="${xyz}" rpy="${rpy}" />
+      <parent link="${parent_link}" />
+      <child link="${tf_prefix_ext}velodyne_puck_link" />
+    </joint>
     <link name="${tf_prefix_ext}velodyne_puck_link">
       <visual>
@@ -39,10 +44,4 @@
       </inertial>
     </link>
-    <link name="${tf_prefix_ext}${frame_id}"></link>
-    <joint name="${parent_link}_to_${tf_prefix_ext}velodyne_puck_link_joint" type="fixed">
-      <origin xyz="${xyz}" rpy="${rpy}" />
-      <parent link="${parent_link}" />
-      <child link="${tf_prefix_ext}velodyne_puck_link" />
-    </joint>
     <joint name="${tf_prefix_ext}velodyne_puck_link_joint_to_${tf_prefix_ext}${frame_id}_joint" type="fixed">
       <origin xyz="0.0 0.0 0.0378" rpy="0.0 0.0 0.0" />
@@ -50,7 +49,5 @@
       <child link="${tf_prefix_ext}${frame_id}" />
     </joint>
-    <gazebo reference="${tf_prefix_ext}velodyne_puck_link">
-      <material>Gazebo/DarkGrey</material>
-    </gazebo>
+    <link name="${tf_prefix_ext}${frame_id}"></link>
     <gazebo reference="${tf_prefix_ext}${frame_id}">
       <sensor type="${ray_type}" name="${tf_prefix_ext}velodyne_puck_sensor">
@@ -59,5 +56,5 @@
           <scan>
             <horizontal>
-              <samples>3600</samples>
+              <samples>1024</samples>
               <resolution>1</resolution>
               <min_angle>-${pi}</min_angle>
@@ -93,4 +90,7 @@
       </sensor>
     </gazebo>
+    <gazebo reference="${tf_prefix_ext}velodyne_puck_link">
+      <material>Gazebo/DarkGrey</material>
+    </gazebo>
   </xacro:macro>
 </robot>

Commit message: Update urdf/orbbec_astra.gazebo.xacro
Co-authored-by: Dawid Kmak <73443304+KmakD@users.noreply.github.com>

File: urdf/orbbec_astra.gazebo.xacro (robot description, xacro)
@@ -34,5 +34,5 @@
       <inertial>
           <mass value="0.105" />
-          <inertia ixx="1" ixy="0" ixz="0" iyy="1" iyz="0" izz="1" />
+          <inertia ixx="1.0" ixy="0.0" ixz="0.0" iyy="1.0" iyz="0.0" izz="1.0" />
       </inertial>
     </link>

Commit message: Update urdf/orbbec_astra.gazebo.xacro
Co-authored-by: Dawid Kmak <73443304+KmakD@users.noreply.github.com>

File: urdf/orbbec_astra.gazebo.xacro (robot description, xacro)
@@ -42,5 +42,5 @@
       <child link="${tf_prefix_ext}${frame_id}" />
     </joint>
-    <link name="${tf_prefix_ext}${frame_id}"></link>
+    <link name="${tf_prefix_ext}${frame_id}" />
     <gazebo reference="${tf_prefix_ext}orbbec_astra_link">
       <sensor type="depth" name="${tf_prefix_ext}orbbec_astra_camera">
