Commit message: Update urdf/velodyne_puck.gazebo.xacro
Co-authored-by: Dawid Kmak <73443304+KmakD@users.noreply.github.com>

File: urdf/velodyne_puck.gazebo.xacro (robot description, xacro)
@@ -34,5 +34,5 @@
       <inertial>
         <mass value="0.830" />
-        <inertia ixx="1" ixy="0" ixz="0" iyy="1" iyz="0" izz="1" />
+        <inertia ixx="1.0" ixy="0.0" ixz="0.0" iyy="1.0" iyz="0.0" izz="1.0" />
       </inertial>
     </link>

Commit message: Update urdf/velodyne_puck.gazebo.xacro
Co-authored-by: Krzysztof Wojciechowski <49921081+Kotochleb@users.noreply.github.com>

File: urdf/velodyne_puck.gazebo.xacro (robot description, xacro)
@@ -41,5 +41,5 @@
       <inertial>
         <mass value="0.830" />
-        <inertia ixx="1" ixy="0" ixz="0" iyy="1" iyz="0" izz="1" />
+        <inertia ixx="1.0" ixy="0.0" ixz="0.0" iyy="1.0" iyz="0.0" izz="1.0" />
       </inertial>
     </link>
