Commit message: Update urdf/ouster_os1_32.gazebo.xacro
Co-authored-by: Dawid Kmak <73443304+KmakD@users.noreply.github.com>

File: urdf/ouster_os1_32.gazebo.xacro (robot description, xacro)
@@ -21,5 +21,5 @@
       <visual>
         <geometry>
-          <mesh filename="file://$(find ros_components_description)/meshes/ouster_os1_32.stl" scale="1 1 0.65" />
+          <mesh filename="file://$(find ros_components_description)/meshes/ouster_os1_32.stl" scale="1.0 1.0 0.65" />
         </geometry>
         <origin xyz="0.0 0.0 0.0" rpy="0.0 0.0 ${pi/2.0}"/>

Commit message: Update urdf/ouster_os1_32.gazebo.xacro
Co-authored-by: Dawid Kmak <73443304+KmakD@users.noreply.github.com>

File: urdf/ouster_os1_32.gazebo.xacro (robot description, xacro)
@@ -34,5 +34,5 @@
       <inertial>
           <mass value="0.447" />
-          <inertia ixx="1" ixy="0" ixz="0" iyy="1" iyz="0" izz="1" />
+          <inertia ixx="1.0" ixy="0.0" ixz="0.0" iyy="1.0" iyz="0.0" izz="1.0" />
       </inertial>
     </link>

Commit message: Update urdf/ouster_os1_32.gazebo.xacro
Co-authored-by: Dawid Kmak <73443304+KmakD@users.noreply.github.com>

File: urdf/ouster_os1_32.gazebo.xacro (robot description, xacro)
@@ -38,5 +38,5 @@
     </link>
     <joint name="${tf_prefix_ext}ouster_os1_32_link_to_${tf_prefix_ext}${frame_id}_joint" type="fixed">
-      <origin xyz="0 0 0.023" rpy="0 0 0" />
+      <origin xyz="0.0 0.0 0.023" rpy="0.0 0.0 0.0" />
       <parent link="${tf_prefix_ext}ouster_os1_32_link" />
       <child link="${tf_prefix_ext}${frame_id}" />

Commit message: Update urdf/ouster_os1_32.gazebo.xacro
Co-authored-by: Dawid Kmak <73443304+KmakD@users.noreply.github.com>

File: urdf/ouster_os1_32.gazebo.xacro (robot description, xacro)
@@ -42,5 +42,5 @@
       <child link="${tf_prefix_ext}${frame_id}" />
     </joint>
-    <link name="${tf_prefix_ext}${frame_id}"></link>
+    <link name="${tf_prefix_ext}${frame_id}" />
     <gazebo reference="${tf_prefix_ext}${frame_id}">
       <sensor type="ray" name="${tf_prefix_ext}ouster_os1_32_sensor">

Commit message: Update ouster_os1_32.gazebo.xacro

File: urdf/ouster_os1_32.gazebo.xacro (robot description, xacro)
@@ -28,5 +28,5 @@
       <visual>
         <geometry>
-          <mesh filename="file://$(find ros_components_description)/meshes/ouster_os1_32.stl" scale="1.0 1.0 0.65" />
+          <mesh filename="file://$(find ros_components_description)/meshes/ouster_os1_32.stl" scale="1.0 1.0 1.0" />
         </geometry>
         <origin xyz="0.0 0.0 0.0" rpy="0.0 0.0 ${pi/2.0}"/>

Commit message: Update urdf/ouster_os1_32.gazebo.xacro
Co-authored-by: Dawid Kmak <73443304+KmakD@users.noreply.github.com>

File: urdf/ouster_os1_32.gazebo.xacro (robot description, xacro)
@@ -21,5 +21,5 @@
       <visual>
         <geometry>
-          <mesh filename="file://$(find ros_components_description)/meshes/ouster_os1_32.stl" scale="1.0 1.0 0.65" />
+          <mesh filename="file://$(find ros_components_description)/meshes/ouster_os1_32.stl" scale="1.0 1.0 1.0" />
         </geometry>
         <origin xyz="0.0 0.0 0.0" rpy="0.0 0.0 ${pi/2.0}"/>
