Commit message: fix gpu usage

File: urdf/rplidar_s1.gazebo.xacro (robot description, xacro)
@@ -5,6 +5,6 @@
                        use_gpu:=false
                        tf_prefix:=None
-                       topic:=rp_scan
-                       frame_id:=rp_laser
+                       topic:=scan
+                       frame_id:=laser
                        simulation_engine:=gazebo-classic">
     <xacro:if value="${use_gpu}">

File: urdf/velodyne_puck.gazebo.xacro (robot description, xacro)
@@ -8,10 +8,4 @@
                        frame_id:=velodyne
                        simulation_engine:=gazebo-classic">
-    <xacro:if value="${use_gpu}">
-      <xacro:property name="ray_type" value="gpu_ray" />
-    </xacro:if>
-    <xacro:unless value="${use_gpu}">
-      <xacro:property name="ray_type" value="ray" />
-    </xacro:unless>
     <xacro:if value="${tf_prefix == 'None'}">
       <xacro:property name="tf_prefix_ext" value="" />

Commit message: Update urdf/rplidar_s1.gazebo.xacro
Co-authored-by: Dawid Kmak <73443304+KmakD@users.noreply.github.com>

File: urdf/rplidar_s1.gazebo.xacro (robot description, xacro)
@@ -32,5 +32,5 @@
           <mesh filename="file://$(find ros_components_description)/meshes/rplidar_s1.stl" scale="0.0001 0.0001 0.0001" />
         </geometry>
-        <origin xyz="0.0 0.0 ${0.051/2.0}" rpy="0 0 -${pi/2.0}"/>
+        <origin xyz="0.0 0.0 ${0.051/2.0}" rpy="0.0 0.0 -${pi/2.0}"/>
         <material name="DarkGrey"/>
       </visual>

Commit message: Update urdf/rplidar_s1.gazebo.xacro
Co-authored-by: Dawid Kmak <73443304+KmakD@users.noreply.github.com>

File: urdf/rplidar_s1.gazebo.xacro (robot description, xacro)
@@ -43,5 +43,5 @@
       <inertial>
         <mass value="0.105" />
-        <inertia ixx="1" ixy="0" ixz="0" iyy="1" iyz="0" izz="1" />
+        <inertia ixx="1.0" ixy="0.0" ixz="0.0" iyy="1.0" iyz="0.0" izz="1.0" />
       </inertial>
     </link>

Commit message: Update urdf/rplidar_s1.gazebo.xacro
Co-authored-by: Dawid Kmak <73443304+KmakD@users.noreply.github.com>

File: urdf/rplidar_s1.gazebo.xacro (robot description, xacro)
@@ -51,5 +51,5 @@
       <child link="${tf_prefix_ext}${frame_id}" />
     </joint>
-    <link name="${tf_prefix_ext}${frame_id}"></link>
+    <link name="${tf_prefix_ext}${frame_id}" />
     <gazebo reference="${tf_prefix_ext}${frame_id}">
       <sensor type="${ray_type}" name="${tf_prefix_ext}rplidar_s1_sensor">

Commit message: Fix s1 lidar simulation in gazebo ignition

File: urdf/rplidar_s1.gazebo.xacro (robot description, xacro)
@@ -2,5 +2,5 @@
 <robot xmlns:xacro="http://www.ros.org/wiki/xacro">
   <xacro:macro name="rplidar_s1"
-               params="parent_link xyz rpy
+    params="parent_link xyz rpy
                        use_gpu:=false
                        tf_prefix:=None
@@ -30,6 +30,6 @@
           <mesh filename="file://$(find ros_components_description)/meshes/rplidar_s1.stl" scale="0.0001 0.0001 0.0001" />
         </geometry>
-        <origin xyz="0.0 0.0 ${0.051/2.0}" rpy="0.0 0.0 -${pi/2.0}"/>
-        <material name="DarkGrey"/>
+        <origin xyz="0.0 0.0 ${0.051/2.0}" rpy="0.0 0.0 -${pi/2.0}" />
+        <material name="DarkGrey" />
       </visual>
       <collision>
@@ -37,5 +37,5 @@
           <cylinder radius="${0.0555/2.0}" length="0.051" />
         </geometry>
-        <origin xyz="0.0 0.0 ${0.051/2.0}" rpy="0.0 0.0 0.0"/>
+        <origin xyz="0.0 0.0 ${0.051/2.0}" rpy="0.0 0.0 0.0" />
       </collision>
       <inertial>
@@ -52,5 +52,8 @@
     <gazebo reference="${tf_prefix_ext}${frame_id}">
       <sensor type="${ray_type}" name="${tf_prefix_ext}rplidar_s1_sensor">
-        <visualize>false</visualize>
+        <topic>/scan</topic>
+        <frame_id>${tf_prefix_ext}${frame_id}</frame_id>
+        <ignition_frame_id>${tf_prefix_ext}${frame_id}</ignition_frame_id>
+        <update_rate>10.0</update_rate>
         <ray>
           <scan>
@@ -63,5 +66,5 @@
           </scan>
           <range>
-            <min>0.2</min>
+            <min>0.04</min>
             <max>40.0</max>
             <resolution>0.03</resolution>
@@ -73,5 +76,15 @@
           </noise>
         </ray>
-        <update_rate>10.0</update_rate>
+        <always_on>1</always_on>
+        <visualize>true</visualize>
+      </sensor>
+    </gazebo>
+    <gazebo>
+      <xacro:if value="${simulation_engine == 'ignition-gazebo'}">
+        <plugin filename="libignition-gazebo-sensors-system.so" name="ignition::gazebo::systems::Sensors">
+          <render_engine>ogre2</render_engine>
+        </plugin>
+      </xacro:if>
+      <xacro:if value="${simulation_engine == 'gazebo-classic'}">
         <plugin name="scan" filename="libgazebo_ros_ray_sensor.so">
           <ros>
@@ -82,5 +95,5 @@
           <frame_name>${tf_prefix_ext}${frame_id}</frame_name>
         </plugin>
-      </sensor>
+      </xacro:if>
     </gazebo>
     <gazebo reference="${tf_prefix_ext}rplidar_s1_link">

Commit message: Add material color to s1 lidar

File: urdf/rplidar_s1.gazebo.xacro (robot description, xacro)
@@ -31,5 +31,7 @@
         </geometry>
         <origin xyz="0.0 0.0 ${0.051/2.0}" rpy="0.0 0.0 -${pi/2.0}" />
-        <material name="DarkGrey" />
+        <material name="DarkGrey">
+          <color rgba="0.05 0.05 0.05 1.0" />
+        </material>
       </visual>
       <collision>
