Commit message: Fix Velodyne name

File: urdf/velodyne_puck.urdf.xacro (robot description, xacro)
@@ -1,5 +1,5 @@
 <?xml version="1.0"?>
 <robot xmlns:xacro="http://www.ros.org/wiki/xacro">
-  <xacro:macro name="velodyne_vlp_16"
+  <xacro:macro name="velodyne_puck"
                params="parent_link xyz rpy
                        use_gpu:=false
@@ -22,14 +22,14 @@
       <xacro:property name="tf_prefix_ext" value="${tf_prefix}_" />
     </xacro:unless>
-    <joint name="${parent_link.rstrip('_link')}_to_${tf_prefix_ext}velodyne_vlp_16_joint" type="fixed">
+    <joint name="${parent_link.rstrip('_link')}_to_${tf_prefix_ext}velodyne_puck_joint" type="fixed">
       <origin xyz="${xyz}" rpy="${rpy}" />
       <parent link="${parent_link}" />
-      <child link="${tf_prefix_ext}velodyne_vlp_16_link" />
+      <child link="${tf_prefix_ext}velodyne_puck_link" />
     </joint>
-    <link name="${tf_prefix_ext}velodyne_vlp_16_link">
+    <link name="${tf_prefix_ext}velodyne_puck_link">
       <visual>
         <origin xyz="0.0 0.0 0.0" rpy="0.0 0.0 0.0"/>
         <geometry>
-          <mesh filename="file://$(find ros_components_description)/meshes/velodyne_vlp_16.dae" />
+          <mesh filename="file://$(find ros_components_description)/meshes/velodyne_puck.dae" />
         </geometry>
       </visual>
@@ -48,7 +48,7 @@
       </inertial>
     </link>
-    <joint name="${tf_prefix_ext}velodyne_vlp_16_to_${tf_prefix_ext}${frame_id.rstrip('_link')}_joint" type="fixed">
+    <joint name="${tf_prefix_ext}velodyne_puck_to_${tf_prefix_ext}${frame_id.rstrip('_link')}_joint" type="fixed">
       <origin xyz="0.0 0.0 0.0378" rpy="0.0 0.0 0.0" />
-      <parent link="${tf_prefix_ext}velodyne_vlp_16_link" />
+      <parent link="${tf_prefix_ext}velodyne_puck_link" />
       <child link="${tf_prefix_ext}${frame_id}" />
     </joint>
@@ -84,5 +84,5 @@
         </ray>
         <update_rate>10.0</update_rate>
-        <plugin name="${tf_prefix_ext}velodyne_vlp_16_${ray_type}" filename="libgazebo_ros_ray_sensor.so">
+        <plugin name="${tf_prefix_ext}velodyne_puck_${ray_type}" filename="libgazebo_ros_ray_sensor.so">
           <ros>
             <namespace>/</namespace>

Commit message: Add support for ignition gazebo in velodyne puck and change horizontal samples

File: urdf/velodyne_puck.urdf.xacro (robot description, xacro)
@@ -48,5 +48,6 @@
       </inertial>
     </link>
-    <joint name="${tf_prefix_ext}velodyne_puck_to_${tf_prefix_ext}${frame_id.rstrip('_link')}_joint" type="fixed">
+    <joint name="${tf_prefix_ext}velodyne_puck_to_${tf_prefix_ext}${frame_id.rstrip('_link')}_joint"
+      type="fixed">
       <origin xyz="0.0 0.0 0.0378" rpy="0.0 0.0 0.0" />
       <parent link="${tf_prefix_ext}velodyne_puck_link" />
@@ -57,8 +58,10 @@
       <sensor type="${ray_type}" name="${tf_prefix_ext}velodyne_puck_sensor">
         <visualize>false</visualize>
+        <update_rate>10.0</update_rate>
         <ray>
           <scan>
             <horizontal>
-              <samples>900</samples>
+              <!-- 0.2 angular resolution for 10Hz -->
+              <samples>1800</samples>
               <resolution>1</resolution>
               <min_angle>-${pi}</min_angle>
@@ -83,13 +86,25 @@
           </noise>
         </ray>
-        <update_rate>10.0</update_rate>
-        <plugin name="${tf_prefix_ext}velodyne_puck_${ray_type}" filename="libgazebo_ros_ray_sensor.so">
-          <ros>
-            <namespace></namespace>
-            <remapping>~/out:=${topic}</remapping>
-          </ros>
-          <output_type>sensor_msgs/PointCloud2</output_type>
-          <frame_name>${tf_prefix_ext}${frame_id}</frame_name>
-        </plugin>
+        <xacro:if value="${simulation_engine == 'ignition-gazebo'}">
+          <topic>${topic}</topic>
+          <frame_id>${tf_prefix_ext}${frame_id}</frame_id>
+          <ignition_frame_id>${tf_prefix_ext}${frame_id}</ignition_frame_id>
+          <always_on>1</always_on>
+          <plugin filename="libignition-gazebo-sensors-system.so"
+            name="ignition::gazebo::systems::Sensors">
+            <render_engine>ogre2</render_engine>
+          </plugin>
+        </xacro:if>
+        <xacro:if value="${simulation_engine == 'gazebo-classic'}">
+          <plugin name="${tf_prefix_ext}velodyne_puck_${ray_type}"
+            filename="libgazebo_ros_ray_sensor.so">
+            <ros>
+              <namespace></namespace>
+              <remapping>~/out:=${topic}</remapping>
+            </ros>
+            <output_type>sensor_msgs/PointCloud2</output_type>
+            <frame_name>${tf_prefix_ext}${frame_id}</frame_name>
+          </plugin>
+        </xacro:if>
       </sensor>
     </gazebo>

Commit message: Add support for ignition gazebo in velodyne puck (#19)
* Add support for ignition gazebo in velodyne puck and change horizontal samples

* Revert samples change

* Change always_on value to true

---------

Co-authored-by: Maciej Stępień <maciej.stepien@husarion.com>

File: urdf/velodyne_puck.urdf.xacro (robot description, xacro)
@@ -48,5 +48,6 @@
       </inertial>
     </link>
-    <joint name="${tf_prefix_ext}velodyne_puck_to_${tf_prefix_ext}${frame_id.rstrip('_link')}_joint" type="fixed">
+    <joint name="${tf_prefix_ext}velodyne_puck_to_${tf_prefix_ext}${frame_id.rstrip('_link')}_joint"
+      type="fixed">
       <origin xyz="0.0 0.0 0.0378" rpy="0.0 0.0 0.0" />
       <parent link="${tf_prefix_ext}velodyne_puck_link" />
@@ -57,4 +58,5 @@
       <sensor type="${ray_type}" name="${tf_prefix_ext}velodyne_puck_sensor">
         <visualize>false</visualize>
+        <update_rate>10.0</update_rate>
         <ray>
           <scan>
@@ -83,13 +85,25 @@
           </noise>
         </ray>
-        <update_rate>10.0</update_rate>
-        <plugin name="${tf_prefix_ext}velodyne_puck_${ray_type}" filename="libgazebo_ros_ray_sensor.so">
-          <ros>
-            <namespace></namespace>
-            <remapping>~/out:=${topic}</remapping>
-          </ros>
-          <output_type>sensor_msgs/PointCloud2</output_type>
-          <frame_name>${tf_prefix_ext}${frame_id}</frame_name>
-        </plugin>
+        <xacro:if value="${simulation_engine == 'ignition-gazebo'}">
+          <topic>${topic}</topic>
+          <frame_id>${tf_prefix_ext}${frame_id}</frame_id>
+          <ignition_frame_id>${tf_prefix_ext}${frame_id}</ignition_frame_id>
+          <always_on>true</always_on>
+          <plugin filename="libignition-gazebo-sensors-system.so"
+            name="ignition::gazebo::systems::Sensors">
+            <render_engine>ogre2</render_engine>
+          </plugin>
+        </xacro:if>
+        <xacro:if value="${simulation_engine == 'gazebo-classic'}">
+          <plugin name="${tf_prefix_ext}velodyne_puck_${ray_type}"
+            filename="libgazebo_ros_ray_sensor.so">
+            <ros>
+              <namespace></namespace>
+              <remapping>~/out:=${topic}</remapping>
+            </ros>
+            <output_type>sensor_msgs/PointCloud2</output_type>
+            <frame_name>${tf_prefix_ext}${frame_id}</frame_name>
+          </plugin>
+        </xacro:if>
       </sensor>
     </gazebo>
