Commit message: Update urdf/slamtec_rplidar_a2.urdf.xacro
Co-authored-by: Dawid Kmak <73443304+KmakD@users.noreply.github.com>

File: urdf/slamtec_rplidar_a2.urdf.xacro (robot description, xacro)
@@ -76,5 +76,5 @@
       <child link="${tf_prefix_ext}${frame_id}" />
     </joint>
-    <link name="${tf_prefix_ext}${frame_id}" />10
+    <link name="${tf_prefix_ext}${frame_id}" />
     <gazebo reference="${tf_prefix_ext}${frame_id}">
       <sensor type="${ray_type}" name="${tf_prefix_ext}slamtec_rplidar_a2_sensor">

Commit message: RPlidar A2 ranfe as float

File: urdf/slamtec_rplidar_a2.urdf.xacro (robot description, xacro)
@@ -30,15 +30,15 @@
     <xacro:if value="${model == 'A2M7'}">
       <xacro:property name="samples" value="1600" />
-      <xacro:property name="max_distance" value="14" />
+      <xacro:property name="max_distance" value="14.0" />
       <xacro:property name="mesh" value="slamtec_rplidar_ax.dae" />
     </xacro:if>
     <xacro:if value="${model == 'A2M8'}">
       <xacro:property name="samples" value="800" />
-      <xacro:property name="max_distance" value="10" />
+      <xacro:property name="max_distance" value="10.0" />
       <xacro:property name="mesh" value="slamtec_rplidar_a2m8.dae" />
     </xacro:if>
     <xacro:if value="${model == 'A2M12'}">
       <xacro:property name="samples" value="1600" />
-      <xacro:property name="max_distance" value="10" />
+      <xacro:property name="max_distance" value="10.0" />
       <xacro:property name="mesh" value="slamtec_rplidar_ax.dae" />
     </xacro:if>

Commit message: Change gpu_lidar to lidar in cpu-default for ignition

File: urdf/slamtec_rplidar_a2.urdf.xacro (robot description, xacro)
@@ -27,6 +27,7 @@
       </xacro:if>
       <xacro:if value="${simulation_engine == 'ignition-gazebo'}">
-        <!-- this is king of awkward, but it seems like cpu lidar does not work -->
-        <xacro:property name="ray_type" value="gpu_lidar" />
+        <!-- use_gpu has to be set to true, CPU lidar doesn't work in ignition -
+          https://github.com/gazebosim/gz-sensors/issues/26 -->
+        <xacro:property name="ray_type" value="lidar" />
       </xacro:if>
     </xacro:unless>

File: urdf/slamtec_rplidar_a3.urdf.xacro (robot description, xacro)
@@ -21,6 +21,7 @@
       </xacro:if>
       <xacro:if value="${simulation_engine == 'ignition-gazebo'}">
-        <!-- this is king of awkward, but it seems like cpu lidar does not work -->
-        <xacro:property name="ray_type" value="gpu_lidar" />
+        <!-- use_gpu has to be set to true, CPU lidar doesn't work in ignition -
+          https://github.com/gazebosim/gz-sensors/issues/26 -->
+        <xacro:property name="ray_type" value="lidar" />
       </xacro:if>
     </xacro:unless>

File: urdf/slamtec_rplidar_s1.urdf.xacro (robot description, xacro)
@@ -21,6 +21,7 @@
       </xacro:if>
       <xacro:if value="${simulation_engine == 'ignition-gazebo'}">
-        <!-- this is king of awkward, but it seems like cpu lidar does not work -->
-        <xacro:property name="ray_type" value="gpu_lidar" />
+        <!-- use_gpu has to be set to true, CPU lidar doesn't work in ignition -
+          https://github.com/gazebosim/gz-sensors/issues/26 -->
+        <xacro:property name="ray_type" value="lidar" />
       </xacro:if>
     </xacro:unless>

Commit message: Added rplidars s2 and s3 (#35)
* Added rplidars s2 and s3

Signed-off-by: Jakub Delicat <jakub.delicat@husarion.com>

* small fixes

---------

Signed-off-by: Jakub Delicat <jakub.delicat@husarion.com>
Co-authored-by: rafal-gorecki <rafal.gorecki@husarion.com>

File: urdf/slamtec_rplidar_a2.urdf.xacro (robot description, xacro)
@@ -145,5 +145,5 @@
               <type>gaussian</type>
               <mean>0.0</mean>
-              <stddev>0.001</stddev>
+              <stddev>0.03</stddev>
             </noise>
           </ray>

File: urdf/slamtec_rplidar_s1.urdf.xacro (robot description, xacro)
@@ -130,5 +130,5 @@
               <type>gaussian</type>
               <mean>0.0</mean>
-              <stddev>0.001</stddev>
+              <stddev>0.03</stddev>
             </noise>
           </ray>

File: urdf/slamtec_rplidar_s2.urdf.xacro (robot description, xacro)
@@ -1,5 +1,5 @@
 <?xml version="1.0"?>
 <robot xmlns:xacro="http://www.ros.org/wiki/xacro">
-  <xacro:macro name="slamtec_rplidar_a3"
+  <xacro:macro name="slamtec_rplidar_s2"
                params="parent_link xyz rpy
                        use_gpu:=false
@@ -27,53 +27,53 @@
     </xacro:unless>
     <xacro:if value="${tf_prefix == 'None'}">
-      <xacro:property name="tf_prefix_ext" value="" />
+      <xacro:property name="prefix" value="" />
     </xacro:if>
     <xacro:unless value="${tf_prefix == 'None'}">
-      <xacro:property name="tf_prefix_ext" value="${tf_prefix}_" />
+      <xacro:property name="prefix" value="${tf_prefix}_" />
     </xacro:unless>
-    <joint name="${parent_link.rstrip('_link')}_to_${tf_prefix_ext}slamtec_rplidar_a3_joint" type="fixed">
+    <joint name="${parent_link.rstrip('_link')}_to_${prefix}slamtec_rplidar_s2_joint" type="fixed">
       <origin xyz="${xyz}" rpy="${rpy}" />
       <parent link="${parent_link}" />
-      <child link="${tf_prefix_ext}slamtec_rplidar_a3_link" />
+      <child link="${prefix}slamtec_rplidar_s2_link" />
     </joint>
-    <link name="${tf_prefix_ext}slamtec_rplidar_a3_link">
+    <link name="${prefix}slamtec_rplidar_s2_link">
       <visual>
         <origin xyz="0.0 0.0 0.0" rpy="0.0 0.0 0.0" />
         <geometry>
-          <!-- slamtec_rplidar_ax.dae is used as a shared mesh for A2 and A3 rplidars -->
-          <mesh filename="package://ros_components_description/meshes/slamtec_rplidar_ax.dae" />
+          <mesh filename="file://$(find ros_components_description)/meshes/slamtec_rplidar_s2.dae" />
         </geometry>
       </visual>
+      <!-- base and head collision -->
       <collision>
-        <origin xyz="0.0 0.0 ${0.041/2.0}" rpy="0.0 0.0 0.0" />
+        <origin xyz="0.0 0.0 ${0.038857/2.0}" rpy="0.0 0.0 0.0" />
         <geometry>
-          <cylinder radius="${0.076/2.0}" length="0.041" />
+          <box size="0.077 0.076856 0.038857" />
         </geometry>
       </collision>
       <inertial>
-        <origin xyz="0.0 0.0 ${0.041/2.0}" rpy="0.0 0.0 0.0" />
-        <mass value="0.190" />
-        <inertia ixx="0.000095206" ixy="0.0"         ixz="0.0"
-                                   iyy="0.000095206" iyz="0.0"
-                                                     izz="0.00013718" />
+        <origin xyz="0.0 -0.000021 ${0.038857/2.0 + 0.0017953}" rpy="0.0 0.0 0.0" />
+        <mass value="0.104949" />
+        <inertia ixx="0.00005071491" ixy="0.0"            ixz="0.0"
+                                     iyy="0.00005064080"  iyz="0.0"
+                                                          izz="0.000075682018" />
       </inertial>
     </link>
-    <joint name="${tf_prefix_ext}slamtec_rplidar_a3_to_${tf_prefix_ext}${frame_id.rstrip('_link')}_joint" type="fixed">
-      <origin xyz="0.0 0.0 0.031" rpy="0.0 0.0 ${pi}" />
-      <parent link="${tf_prefix_ext}slamtec_rplidar_a3_link" />
-      <child link="${tf_prefix_ext}${frame_id}" />
+    <joint name="${prefix}slamtec_rplidar_s2_to_${prefix}${frame_id.rstrip('_link')}_joint" type="fixed">
+      <origin xyz="0.0 0.0 0.0285" rpy="0.0 0.0 ${pi}" />
+      <parent link="${prefix}slamtec_rplidar_s2_link" />
+      <child link="${prefix}${frame_id}" />
     </joint>
-    <link name="${tf_prefix_ext}${frame_id}" />
+    <link name="${prefix}${frame_id}" />
     <xacro:if value="${simulation_engine == 'ignition-gazebo'}">
-      <gazebo reference="${tf_prefix_ext}${frame_id}">
-        <sensor type="${ray_type}" name="${tf_prefix_ext}rplidar_a3_sensor">
+      <gazebo reference="${prefix}${frame_id}">
+        <sensor type="${ray_type}" name="${prefix}rplidar_s2_sensor">
           <topic>${topic}</topic>
-          <frame_id>${tf_prefix_ext}${frame_id}</frame_id>
-          <ignition_frame_id>${tf_prefix_ext}${frame_id}</ignition_frame_id>
+          <frame_id>${prefix}${frame_id}</frame_id>
+          <ignition_frame_id>${prefix}${frame_id}</ignition_frame_id>
           <update_rate>10.0</update_rate>
           <ray>
             <scan>
               <horizontal>
-                <samples>1600</samples>
+                <samples>3000</samples>
                 <resolution>1</resolution>
                 <min_angle>-${pi}</min_angle>
@@ -82,8 +82,7 @@
             </scan>
             <range>
-              <min>0.2</min>
-              <!-- as an tradeoff between white and black object range -->
-              <max>16.0</max>
-              <resolution>0.05</resolution>
+              <min>0.05</min>
+              <max>30.0</max>
+              <resolution>0.03</resolution>
             </range>
             <noise>
@@ -93,22 +92,22 @@
             </noise>
           </ray>
-          <always_on>true</always_on>
+          <always_on>1</always_on>
           <visualize>false</visualize>
         </sensor>
       </gazebo>
       <gazebo>
-          <plugin filename="libignition-gazebo-sensors-system.so" name="ignition::gazebo::systems::Sensors">
-            <render_engine>ogre2</render_engine>
-          </plugin>
-        </gazebo>
+        <plugin filename="libignition-gazebo-sensors-system.so" name="ignition::gazebo::systems::Sensors">
+          <render_engine>ogre2</render_engine>
+        </plugin>
+      </gazebo>
     </xacro:if>
     <xacro:if value="${simulation_engine == 'gazebo-classic'}">
-      <gazebo reference="${tf_prefix_ext}${frame_id}">
-        <sensor type="${ray_type}" name="${tf_prefix_ext}slamtec_rplidar_a3_sensor">
+      <gazebo reference="${prefix}${frame_id}">
+        <sensor type="${ray_type}" name="${prefix}slamtec_rplidar_s2_sensor">
           <visualize>false</visualize>
           <ray>
             <scan>
               <horizontal>
-                <samples>1600</samples>
+                <samples>3000</samples>
                 <resolution>1</resolution>
                 <min_angle>-${pi}</min_angle>
@@ -117,8 +116,7 @@
             </scan>
             <range>
-              <min>0.2</min>
-              <!-- as an tradeoff between white and black object range -->
-              <max>20.0</max>
-              <resolution>0.05</resolution>
+              <min>0.05</min>
+              <max>30.0</max>
+              <resolution>0.013</resolution>
             </range>
             <noise>
@@ -135,5 +133,5 @@
             </ros>
             <output_type>sensor_msgs/LaserScan</output_type>
-            <frame_name>${tf_prefix_ext}${frame_id}</frame_name>
+            <frame_name>${prefix}${frame_id}</frame_name>
           </plugin>
         </sensor>

File: urdf/slamtec_rplidar_s3.urdf.xacro (robot description, xacro)
@@ -1,5 +1,5 @@
 <?xml version="1.0"?>
 <robot xmlns:xacro="http://www.ros.org/wiki/xacro">
-  <xacro:macro name="slamtec_rplidar_a3"
+  <xacro:macro name="slamtec_rplidar_s3"
                params="parent_link xyz rpy
                        use_gpu:=false
@@ -27,53 +27,53 @@
     </xacro:unless>
     <xacro:if value="${tf_prefix == 'None'}">
-      <xacro:property name="tf_prefix_ext" value="" />
+      <xacro:property name="prefix" value="" />
     </xacro:if>
     <xacro:unless value="${tf_prefix == 'None'}">
-      <xacro:property name="tf_prefix_ext" value="${tf_prefix}_" />
+      <xacro:property name="prefix" value="${tf_prefix}_" />
     </xacro:unless>
-    <joint name="${parent_link.rstrip('_link')}_to_${tf_prefix_ext}slamtec_rplidar_a3_joint" type="fixed">
+    <joint name="${parent_link.rstrip('_link')}_to_${prefix}slamtec_rplidar_s3_joint" type="fixed">
       <origin xyz="${xyz}" rpy="${rpy}" />
       <parent link="${parent_link}" />
-      <child link="${tf_prefix_ext}slamtec_rplidar_a3_link" />
+      <child link="${prefix}slamtec_rplidar_s3_link" />
     </joint>
-    <link name="${tf_prefix_ext}slamtec_rplidar_a3_link">
+    <link name="${prefix}slamtec_rplidar_s3_link">
       <visual>
         <origin xyz="0.0 0.0 0.0" rpy="0.0 0.0 0.0" />
         <geometry>
-          <!-- slamtec_rplidar_ax.dae is used as a shared mesh for A2 and A3 rplidars -->
-          <mesh filename="package://ros_components_description/meshes/slamtec_rplidar_ax.dae" />
+          <mesh filename="file://$(find ros_components_description)/meshes/slamtec_rplidar_s3.dae" />
         </geometry>
       </visual>
+      <!-- base and head collision -->
       <collision>
-        <origin xyz="0.0 0.0 ${0.041/2.0}" rpy="0.0 0.0 0.0" />
+        <origin xyz="0.0 0.0 ${0.0413/2.0}" rpy="0.0 0.0 0.0" />
         <geometry>
-          <cylinder radius="${0.076/2.0}" length="0.041" />
+          <box size="0.0556 0.0556 0.0413" />
         </geometry>
       </collision>
       <inertial>
-        <origin xyz="0.0 0.0 ${0.041/2.0}" rpy="0.0 0.0 0.0" />
-        <mass value="0.190" />
-        <inertia ixx="0.000095206" ixy="0.0"         ixz="0.0"
-                                   iyy="0.000095206" iyz="0.0"
-                                                     izz="0.00013718" />
+        <origin xyz="0.0 0.0 ${0.0413/2.0 + 0.0018237}" rpy="0.0 0.0 0.0" />
+        <mass value="0.115033" />
+        <inertia ixx="0.00004115765" ixy="0.0"            ixz="0.0"
+                                     iyy="0.00004115765"  iyz="0.0"
+                                                          izz="0.00004956023" />
       </inertial>
     </link>
-    <joint name="${tf_prefix_ext}slamtec_rplidar_a3_to_${tf_prefix_ext}${frame_id.rstrip('_link')}_joint" type="fixed">
-      <origin xyz="0.0 0.0 0.031" rpy="0.0 0.0 ${pi}" />
-      <parent link="${tf_prefix_ext}slamtec_rplidar_a3_link" />
-      <child link="${tf_prefix_ext}${frame_id}" />
+    <joint name="${prefix}slamtec_rplidar_s3_to_${prefix}${frame_id.rstrip('_link')}_joint" type="fixed">
+      <origin xyz="0.0 0.0 0.0305" rpy="0.0 0.0 ${pi}" />
+      <parent link="${prefix}slamtec_rplidar_s3_link" />
+      <child link="${prefix}${frame_id}" />
     </joint>
-    <link name="${tf_prefix_ext}${frame_id}" />
+    <link name="${prefix}${frame_id}" />
     <xacro:if value="${simulation_engine == 'ignition-gazebo'}">
-      <gazebo reference="${tf_prefix_ext}${frame_id}">
-        <sensor type="${ray_type}" name="${tf_prefix_ext}rplidar_a3_sensor">
+      <gazebo reference="${prefix}${frame_id}">
+        <sensor type="${ray_type}" name="${prefix}rplidar_s3_sensor">
           <topic>${topic}</topic>
-          <frame_id>${tf_prefix_ext}${frame_id}</frame_id>
-          <ignition_frame_id>${tf_prefix_ext}${frame_id}</ignition_frame_id>
+          <frame_id>${prefix}${frame_id}</frame_id>
+          <ignition_frame_id>${prefix}${frame_id}</ignition_frame_id>
           <update_rate>10.0</update_rate>
           <ray>
             <scan>
               <horizontal>
-                <samples>1600</samples>
+                <samples>3000</samples>
                 <resolution>1</resolution>
                 <min_angle>-${pi}</min_angle>
@@ -82,33 +82,32 @@
             </scan>
             <range>
-              <min>0.2</min>
-              <!-- as an tradeoff between white and black object range -->
-              <max>16.0</max>
-              <resolution>0.05</resolution>
+              <min>0.05</min>
+              <max>40.0</max>
+              <resolution>0.01</resolution>
             </range>
             <noise>
               <type>gaussian</type>
               <mean>0.0</mean>
-              <stddev>0.001</stddev>
+              <stddev>0.03</stddev>
             </noise>
           </ray>
-          <always_on>true</always_on>
+          <always_on>1</always_on>
           <visualize>false</visualize>
         </sensor>
       </gazebo>
       <gazebo>
-          <plugin filename="libignition-gazebo-sensors-system.so" name="ignition::gazebo::systems::Sensors">
-            <render_engine>ogre2</render_engine>
-          </plugin>
-        </gazebo>
+        <plugin filename="libignition-gazebo-sensors-system.so" name="ignition::gazebo::systems::Sensors">
+          <render_engine>ogre2</render_engine>
+        </plugin>
+      </gazebo>
     </xacro:if>
     <xacro:if value="${simulation_engine == 'gazebo-classic'}">
-      <gazebo reference="${tf_prefix_ext}${frame_id}">
-        <sensor type="${ray_type}" name="${tf_prefix_ext}slamtec_rplidar_a3_sensor">
+      <gazebo reference="${prefix}${frame_id}">
+        <sensor type="${ray_type}" name="${prefix}slamtec_rplidar_s3_sensor">
           <visualize>false</visualize>
           <ray>
             <scan>
               <horizontal>
-                <samples>1600</samples>
+                <samples>3200</samples>
                 <resolution>1</resolution>
                 <min_angle>-${pi}</min_angle>
@@ -117,13 +116,12 @@
             </scan>
             <range>
-              <min>0.2</min>
-              <!-- as an tradeoff between white and black object range -->
-              <max>20.0</max>
-              <resolution>0.05</resolution>
+              <min>0.05</min>
+              <max>40.0</max>
+              <resolution>0.01</resolution>
             </range>
             <noise>
               <type>gaussian</type>
               <mean>0.0</mean>
-              <stddev>0.03</stddev>
+              <stddev>0.001</stddev>
             </noise>
           </ray>
@@ -135,5 +133,5 @@
             </ros>
             <output_type>sensor_msgs/LaserScan</output_type>
-            <frame_name>${tf_prefix_ext}${frame_id}</frame_name>
+            <frame_name>${prefix}${frame_id}</frame_name>
           </plugin>
         </sensor>
