Commit message: file -> package

File: urdf/slamtec_rplidar_s2.urdf.xacro (robot description, xacro)
@@ -41,5 +41,5 @@
         <origin xyz="0.0 0.0 0.0" rpy="0.0 0.0 0.0" />
         <geometry>
-          <mesh filename="file://$(find ros_components_description)/meshes/slamtec_rplidar_s2.dae" />
+          <mesh filename="package://ros_components_description/meshes/slamtec_rplidar_s2.dae" />
         </geometry>
       </visual>

File: urdf/slamtec_rplidar_s3.urdf.xacro (robot description, xacro)
@@ -41,5 +41,5 @@
         <origin xyz="0.0 0.0 0.0" rpy="0.0 0.0 0.0" />
         <geometry>
-          <mesh filename="file://$(find ros_components_description)/meshes/slamtec_rplidar_s3.dae" />
+          <mesh filename="package://ros_components_description/meshes/slamtec_rplidar_s3.dae" />
         </geometry>
       </visual>

Commit message: added namespace gazebo to other rplidars
Signed-off-by: Jakub Delicat <jakub.delicat@husarion.com>

File: urdf/slamtec_rplidar_s2.urdf.xacro (robot description, xacro)
@@ -7,5 +7,12 @@
                        topic:=scan
                        frame_id:=laser
+                       namespace=None
                        simulation_engine:=gazebo-classic">
+    <xacro:if value="${namespace == 'None'}">
+      <xacro:property name="namespace_ext" value="" />
+    </xacro:if>
+    <xacro:unless value="${namespace == 'None'}">
+        <xacro:property name="namespace_ext" value="${namespace}/" />
+    </xacro:unless>
     <xacro:if value="${use_gpu}">
       <xacro:if value="${simulation_engine == 'gazebo-classic'}">
@@ -67,6 +74,6 @@
     <xacro:if value="${simulation_engine == 'ignition-gazebo'}">
       <gazebo reference="${prefix}${frame_id}">
-        <sensor type="${ray_type}" name="${prefix}rplidar_s2_sensor">
-          <topic>${topic}</topic>
+        <sensor type="${ray_type}" name="${namespace_ext}${prefix}rplidar_s2_sensor">
+          <topic>${namespace_ext}${topic}</topic>
           <frame_id>${prefix}${frame_id}</frame_id>
           <ignition_frame_id>${prefix}${frame_id}</ignition_frame_id>
@@ -94,10 +101,8 @@
           <always_on>1</always_on>
           <visualize>false</visualize>
+          <ros>
+            <namespace>${namespace_ext}</namespace>
+          </ros>
         </sensor>
-      </gazebo>
-      <gazebo>
-        <plugin filename="libignition-gazebo-sensors-system.so" name="ignition::gazebo::systems::Sensors">
-          <render_engine>ogre2</render_engine>
-        </plugin>
       </gazebo>
     </xacro:if>

File: urdf/slamtec_rplidar_s3.urdf.xacro (robot description, xacro)
@@ -7,5 +7,12 @@
                        topic:=scan
                        frame_id:=laser
+                       namespace=None
                        simulation_engine:=gazebo-classic">
+    <xacro:if value="${namespace == 'None'}">
+      <xacro:property name="namespace_ext" value="" />
+    </xacro:if>
+    <xacro:unless value="${namespace == 'None'}">
+        <xacro:property name="namespace_ext" value="${namespace}/" />
+    </xacro:unless>
     <xacro:if value="${use_gpu}">
       <xacro:if value="${simulation_engine == 'gazebo-classic'}">
@@ -67,6 +74,6 @@
     <xacro:if value="${simulation_engine == 'ignition-gazebo'}">
       <gazebo reference="${prefix}${frame_id}">
-        <sensor type="${ray_type}" name="${prefix}rplidar_s3_sensor">
-          <topic>${topic}</topic>
+        <sensor type="${ray_type}" name="${namespace_ext}${prefix}rplidar_s3_sensor">
+          <topic>${namespace_ext}${topic}</topic>
           <frame_id>${prefix}${frame_id}</frame_id>
           <ignition_frame_id>${prefix}${frame_id}</ignition_frame_id>
@@ -95,9 +102,7 @@
           <visualize>false</visualize>
         </sensor>
-      </gazebo>
-      <gazebo>
-        <plugin filename="libignition-gazebo-sensors-system.so" name="ignition::gazebo::systems::Sensors">
-          <render_engine>ogre2</render_engine>
-        </plugin>
+        <ros>
+          <namespace>${namespace_ext}</namespace>
+        </ros>
       </gazebo>
     </xacro:if>
