Commit message: Update sensor definitions to standard from guide

File: urdf/orbbec_astra.urdf.xacro (robot description, xacro)
@@ -13,5 +13,5 @@
       <xacro:property name="tf_prefix_ext" value="${tf_prefix}_" />
     </xacro:unless>
-    <joint name="${parent_link}_to_${tf_prefix_ext}orbbec_astra_link_joint" type="fixed">
+    <joint name="${parent_link.rstrip('_link')}_to_${tf_prefix_ext}orbbec_astra_joint" type="fixed">
       <origin xyz="${xyz}" rpy="${rpy}" />
       <parent link="${parent_link}" />
@@ -20,22 +20,32 @@
     <link name="${tf_prefix_ext}orbbec_astra_link">
       <visual>
+        <origin xyz="0.0 0.0 0.0" rpy="0.0 0.0 0.0"/>
         <geometry>
-          <mesh filename="file://$(find ros_components_description)/meshes/orbbec_astra.stl" scale="0.001 0.001 0.001" />
+          <mesh filename="file://$(find ros_components_description)/meshes/orbbec_astra.dae" />
         </geometry>
-        <origin xyz="-0.01 0 0.025" rpy="${pi/2} 0 ${pi/2}"/>
-        <material name="DarkGrey"/>
       </visual>
+      <!-- camera module collision -->
       <collision>
+        <origin xyz="${0.0225-0.04/2.0} 0.0 ${0.019+0.03/2.0}" rpy="0.0 0.0 0.0"/>
         <geometry>
-          <box size="0.165 0.04 0.05" />
+          <box size="0.04 0.165 0.03" />
         </geometry>
-        <origin xyz="-0.01 0 0.025" rpy="0 0 ${pi/2}"/>
+      </collision>
+      <!-- mounting base model collision -->
+      <collision>
+        <origin xyz="${0.0235-0.06/2.0} 0.0 ${0.019/2.0}" rpy="0.0 0.0 0.0"/>
+        <geometry>
+          <box size="0.06 0.06 0.019" />
+        </geometry>
       </collision>
       <inertial>
-          <mass value="0.105" />
-          <inertia ixx="1.0" ixy="0.0" ixz="0.0" iyy="1.0" iyz="0.0" izz="1.0" />
+        <origin xyz="0.0 0.0 ${0.019+0.01}" rpy="0.0 0.0 0.0" />
+        <mass value="0.300" />
+        <inertia ixx="0.00073916" ixy="0.0"        ixz="0.0"
+                                  iyy="0.00015435" iyz="0.0"
+                                                   izz="0.00077395" />
       </inertial>
     </link>
-    <joint name="${tf_prefix_ext}${frame_id}_link_joint" type="fixed">
+    <joint name="${tf_prefix_ext}orbbec_astra_to_${tf_prefix_ext}${frame_id.rstrip('_link')}_joint" type="fixed">
       <origin xyz="0.01 0 0.035" rpy="${-pi/2} 0 ${-pi/2}" />
       <parent link="${tf_prefix_ext}orbbec_astra_link" />
@@ -85,7 +95,4 @@
       </sensor>
     </gazebo>
-    <gazebo reference="${tf_prefix_ext}orbbec_astra_link">
-      <material>Gazebo/DarkGrey</material>
-    </gazebo>
   </xacro:macro>
 </robot>

File: urdf/ouster_os1_32.urdf.xacro (robot description, xacro)
@@ -3,8 +3,17 @@
     <xacro:macro name="ouster_os1_32"
                params="parent_link xyz rpy
+                       use_gpu:=false
                        tf_prefix:=None
                        topic:=os_lidar
                        frame_id:=os_lidar
-                       simulation_engine:=gazebo-classic">
+                       simulation_engine:=gazebo-classic" >
+    <xacro:if value="${use_gpu}">
+      <xacro:property name="ray_type" value="gpu_ray" />
+      <xacro:property name="plugin_file_name" value="libgazebo_ros_velodyne_gpu_laser.so" />
+    </xacro:if>
+    <xacro:unless value="${use_gpu}">
+      <xacro:property name="ray_type" value="ray" />
+      <xacro:property name="plugin_file_name" value="libgazebo_ros_velodyne_laser.so" />
+    </xacro:unless>
     <xacro:if value="${tf_prefix == 'None'}">
       <xacro:property name="tf_prefix_ext" value="" />
@@ -13,5 +22,5 @@
       <xacro:property name="tf_prefix_ext" value="${tf_prefix}" />
     </xacro:unless>
-    <joint name="${parent_link}_to_${tf_prefix_ext}ouster_os1_32_link_joint" type="fixed">
+    <joint name="${parent_link.rstrip('_link')}_to_${tf_prefix_ext}ouster_os1_32_joint" type="fixed">
       <origin xyz="${xyz}" rpy="${rpy}" />
       <parent link="${parent_link}" />
@@ -20,22 +29,24 @@
     <link name="${tf_prefix_ext}ouster_os1_32_link">
       <visual>
+        <origin xyz="0.0 0.0 0.0" rpy="0.0 0.0 0.0"/>
         <geometry>
-          <mesh filename="file://$(find ros_components_description)/meshes/ouster_os1_32.stl" scale="1.0 1.0 1.0" />
+          <mesh filename="file://$(find ros_components_description)/meshes/ouster_os1_32.dae" />
         </geometry>
-        <origin xyz="0.0 0.0 0.0" rpy="0.0 0.0 ${pi/2.0}"/>
-        <material name="Grey"/>
       </visual>
       <collision>
+        <origin xyz="0.0 0.0 ${0.072/2.0}" rpy="0.0 0.0 0.0"/>
         <geometry>
-          <cylinder radius="${0.0753/2.0}" length="0.0435" />
+          <cylinder radius="${0.085/2.0}" length="0.073" />
         </geometry>
-        <origin xyz="0.0 0.0 ${0.0435/2.0}" rpy="0.0 0.0 0.0"/>
       </collision>
       <inertial>
-          <mass value="0.447" />
-          <inertia ixx="1.0" ixy="0.0" ixz="0.0" iyy="1.0" iyz="0.0" izz="1.0" />
+        <origin xyz="0.0 0.0 ${0.072/2.0}" rpy="0.0 0.0 0.0" />
+        <mass value="0.447" />
+        <inertia ixx="0.00047706" ixy="0.0"        ixz="0.0"
+                                  iyy="0.00047706" iyz="0.0"
+                                                   izz="0.00053722" />
       </inertial>
     </link>
-    <joint name="${tf_prefix_ext}ouster_os1_32_link_to_${tf_prefix_ext}${frame_id}_joint" type="fixed">
+    <joint name="${tf_prefix_ext}ouster_os1_32_to_${tf_prefix_ext}${frame_id.rstrip('_link')}_joint" type="fixed">
       <origin xyz="0.0 0.0 0.023" rpy="0.0 0.0 0.0" />
       <parent link="${tf_prefix_ext}ouster_os1_32_link" />
@@ -44,5 +55,5 @@
     <link name="${tf_prefix_ext}${frame_id}" />
     <gazebo reference="${tf_prefix_ext}${frame_id}">
-      <sensor type="ray" name="${tf_prefix_ext}ouster_os1_32_sensor">
+      <sensor type="${ray_type}" name="${tf_prefix_ext}ouster_os1_32_sensor">
         <visualize>false</visualize>
         <update_rate>10</update_rate>
@@ -63,6 +74,6 @@
           </scan>
           <range>
-            <min>${0.0753/2+0.01}</min>
-            <max>100.0</max>
+            <min>${0.085/2.0+0.01}</min>
+            <max>120.0</max>
             <resolution>0.003</resolution>
           </range>
@@ -73,15 +84,14 @@
           </noise>
         </ray>
-        <plugin name="ray" filename="libgazebo_ros_block_laser.so">
+        <plugin name="${tf_prefix_ext}ouster_os1_32_${ray_type}" filename="${plugin_file_name}">
           <topicName>${topic}</topicName>
           <frameName>${tf_prefix_ext}${frame_id}</frameName>
+          <organize_cloud>true</organize_cloud>
+          <min_range>0.5</min_range>
+          <max_range>120.0</max_range>
           <gaussianNoise>0.0008</gaussianNoise>
-          <updateRate>10</updateRate>
         </plugin>
       </sensor>
     </gazebo>
-    <gazebo reference="${tf_prefix_ext}ouster_os1_32_link">
-      <material>Gazebo/Grey</material>
-    </gazebo>
   </xacro:macro>
 </robot>

File: urdf/slamtec_rplidar_s1.urdf.xacro (robot description, xacro)
@@ -1,5 +1,5 @@
 <?xml version="1.0"?>
 <robot xmlns:xacro="http://www.ros.org/wiki/xacro">
-  <xacro:macro name="rplidar_s1"
+  <xacro:macro name="slamtec_rplidar_s1"
                params="parent_link xyz rpy
                        use_gpu:=false
@@ -7,5 +7,5 @@
                        topic:=scan
                        frame_id:=laser
-                       simulation_engine:=gazebo-classic">
+                       simulation_engine:=gazebo-classic" >
     <xacro:if value="${use_gpu}">
       <xacro:property name="ray_type" value="gpu_ray" />
@@ -22,36 +22,46 @@
       <xacro:property name="tf_prefix_ext" value="${tf_prefix}_" />
     </xacro:unless>
-    <joint name="${parent_link}_to_${tf_prefix_ext}rplidar_s1_link_joint" type="fixed">
+    <joint name="${parent_link.rstrip('_link')}_to_${tf_prefix_ext}slamtec_rplidar_s1_joint" type="fixed">
       <origin xyz="${xyz}" rpy="${rpy}" />
       <parent link="${parent_link}" />
-      <child link="${tf_prefix_ext}rplidar_s1_link" />
+      <child link="${tf_prefix_ext}slamtec_rplidar_s1_link" />
     </joint>
-    <link name="${tf_prefix_ext}rplidar_s1_link">
+    <link name="${tf_prefix_ext}slamtec_rplidar_s1_link">
       <visual>
+        <origin xyz="0.0 0.0 0.0" rpy="0.0 0.0 0.0"/>
         <geometry>
-          <mesh filename="file://$(find ros_components_description)/meshes/rplidar_s1.stl" scale="0.0001 0.0001 0.0001" />
+          <mesh filename="file://$(find ros_components_description)/meshes/slamtec_rplidar_s1.dae" />
         </geometry>
-        <origin xyz="0.0 0.0 ${0.051/2.0}" rpy="0.0 0.0 -${pi/2.0}"/>
-        <material name="DarkGrey"/>
       </visual>
+      <!-- spinning head collision -->
       <collision>
+        <origin xyz="0.0 0.0 ${0.051/2.0}" rpy="0.0 0.0 0.0"/>
         <geometry>
           <cylinder radius="${0.0555/2.0}" length="0.051" />
         </geometry>
-        <origin xyz="0.0 0.0 ${0.051/2.0}" rpy="0.0 0.0 0.0"/>
+      </collision>
+      <!-- base collision -->
+      <collision>
+        <origin xyz="0.0 0.0 ${0.0195/2.0}" rpy="0.0 0.0 0.0"/>
+        <geometry>
+          <box size="0.0555 0.0555 0.0195" />
+        </geometry>
       </collision>
       <inertial>
+        <origin xyz="0.0 0.0 ${0.0555/2.0}" rpy="0.0 0.0 0.0" />
         <mass value="0.105" />
-        <inertia ixx="1.0" ixy="0.0" ixz="0.0" iyy="1.0" iyz="0.0" izz="1.0" />
+        <inertia ixx="0.000049654" ixy="0.0"         ixz="0.0"
+                                   iyy="0.000049654" iyz="0.0"
+                                                     izz="0.000053884" />
       </inertial>
     </link>
-    <joint name="${tf_prefix_ext}rplidar_s1_to_${tf_prefix_ext}${frame_id}_joint" type="fixed">
-      <origin xyz="0 0 0.04" rpy="0.0 0.0 0.0" />
-      <parent link="${tf_prefix_ext}rplidar_s1_link" />
+    <joint name="${tf_prefix_ext}slamtec_rplidar_s1_to_${tf_prefix_ext}${frame_id.rstrip('_link')}_joint" type="fixed">
+      <origin xyz="0 0 0.04" rpy="0.0 0.0 ${pi}" />
+      <parent link="${tf_prefix_ext}slamtec_rplidar_s1_link" />
       <child link="${tf_prefix_ext}${frame_id}" />
     </joint>
     <link name="${tf_prefix_ext}${frame_id}" />
     <gazebo reference="${tf_prefix_ext}${frame_id}">
-      <sensor type="${ray_type}" name="${tf_prefix_ext}rplidar_s1_sensor">
+      <sensor type="${ray_type}" name="${tf_prefix_ext}slamtec_rplidar_s1_sensor">
         <pose>0 0 0.04 0 0 0</pose>
         <visualize>false</visualize>
@@ -67,5 +77,5 @@
           </scan>
           <range>
-            <min>${0.051/2+0.03}</min>
+            <min>${0.0555/2.0+0.01}</min>
             <max>40.0</max>
             <resolution>0.03</resolution>
@@ -83,7 +93,4 @@
       </sensor>
     </gazebo>
-    <gazebo reference="${tf_prefix_ext}rplidar_s1_link">
-      <material>Gazebo/DarkGrey</material>
-    </gazebo>
   </xacro:macro>
 </robot>

File: urdf/velodyne_vlp_16.urdf.xacro (robot description, xacro)
@@ -1,10 +1,19 @@
 <?xml version="1.0"?>
 <robot xmlns:xacro="http://www.ros.org/wiki/xacro">
-  <xacro:macro name="velodyne_puck"
+  <xacro:macro name="velodyne_vlp_16"
                params="parent_link xyz rpy
+                       use_gpu:=false
                        tf_prefix:=None
                        topic:=scan
                        frame_id:=velodyne
-                       simulation_engine:=gazebo-classic">
+                       simulation_engine:=gazebo-classic" >
+    <xacro:if value="${use_gpu}">
+      <xacro:property name="ray_type" value="gpu_ray" />
+      <xacro:property name="plugin_file_name" value="libgazebo_ros_velodyne_gpu_laser.so" />
+    </xacro:if>
+    <xacro:unless value="${use_gpu}">
+      <xacro:property name="ray_type" value="ray" />
+      <xacro:property name="plugin_file_name" value="libgazebo_ros_velodyne_laser.so" />
+    </xacro:unless>
     <xacro:if value="${tf_prefix == 'None'}">
       <xacro:property name="tf_prefix_ext" value="" />
@@ -13,36 +22,38 @@
       <xacro:property name="tf_prefix_ext" value="${tf_prefix}_" />
     </xacro:unless>
-    <joint name="${parent_link}_to_${tf_prefix_ext}velodyne_puck_link_joint" type="fixed">
+    <joint name="${parent_link.rstrip('_link')}_to_${tf_prefix_ext}velodyne_vlp_16_joint" type="fixed">
       <origin xyz="${xyz}" rpy="${rpy}" />
       <parent link="${parent_link}" />
-      <child link="${tf_prefix_ext}velodyne_puck_link" />
+      <child link="${tf_prefix_ext}velodyne_vlp_16_link" />
     </joint>
-    <link name="${tf_prefix_ext}velodyne_puck_link">
+    <link name="${tf_prefix_ext}velodyne_vlp_16_link">
       <visual>
+        <origin xyz="0.0 0.0 0.0" rpy="0.0 0.0 0.0"/>
         <geometry>
-          <mesh filename="file://$(find ros_components_description)/meshes/velodyne_puck.stl" scale="0.025035 0.025035 0.025035" />
+          <mesh filename="file://$(find ros_components_description)/meshes/velodyne_vlp_16.dae" />
         </geometry>
-        <origin xyz="0.0 0.0 0.0" rpy="${pi/2.0} 0.0 ${pi}"/>
-        <material name="DarkGrey"/>
       </visual>
       <collision>
+        <origin xyz="0.0 0.0 ${0.072/2.0}" rpy="0.0 0.0 0.0"/>
         <geometry>
-          <cylinder radius="${0.090/2.0}" length="0.0717" />
+          <cylinder radius="${0.103/2.0}" length="0.072" />
         </geometry>
-        <origin xyz="0.0 0.0 ${0.0717/2.0}" rpy="0.0 0.0 0.0"/>
       </collision>
       <inertial>
+        <origin xyz="0.0 0.0 ${0.072/2.0}" rpy="0.0 0.0 0.0" />
         <mass value="0.830" />
-        <inertia ixx="1.0" ixy="0.0" ixz="0.0" iyy="1.0" iyz="0.0" izz="1.0" />
+        <inertia ixx="0.001111" ixy="0.0"      ixz="0.0"
+                                iyy="0.001109" iyz="0.0"
+                                               izz="0.001493" />
       </inertial>
     </link>
-    <joint name="${tf_prefix_ext}velodyne_puck_link_to_${tf_prefix_ext}${frame_id}_joint" type="fixed">
+    <joint name="${tf_prefix_ext}velodyne_vlp_16_to_${tf_prefix_ext}${frame_id.rstrip('_link')}_joint" type="fixed">
       <origin xyz="0.0 0.0 0.0378" rpy="0.0 0.0 0.0" />
-      <parent link="${tf_prefix_ext}velodyne_puck_link" />
+      <parent link="${tf_prefix_ext}velodyne_vlp_16_link" />
       <child link="${tf_prefix_ext}${frame_id}" />
     </joint>
-    <link name="${tf_prefix_ext}${frame_id}"></link>
+    <link name="${tf_prefix_ext}${frame_id}" />
     <gazebo reference="${tf_prefix_ext}${frame_id}">
-      <sensor type="ray" name="${tf_prefix_ext}velodyne_puck_sensor">
+      <sensor type="${ray_type}" name="${tf_prefix_ext}velodyne_vlp_16_sensor">
         <visualize>false</visualize>
         <update_rate>10</update_rate>
@@ -63,5 +74,5 @@
           </scan>
           <range>
-            <min>${0.051+0.01}</min>
+            <min>${0.103/2.0+0.01}</min>
             <max>100.0</max>
             <resolution>0.003</resolution>
@@ -73,15 +84,14 @@
           </noise>
         </ray>
-        <plugin name="ray" filename="libgazebo_ros_block_laser.so">
+        <plugin name="${tf_prefix_ext}velodyne_vlp_16_${ray_type}" filename="${plugin_file_name}">
           <topicName>${topic}</topicName>
           <frameName>${tf_prefix_ext}${frame_id}</frameName>
+          <organize_cloud>true</organize_cloud>
+          <min_range>0.4</min_range>
+          <max_range>100.0</max_range>
           <gaussianNoise>0.0008</gaussianNoise>
-          <updateRate>10</updateRate>
         </plugin>
       </sensor>
     </gazebo>
-    <gazebo reference="${tf_prefix_ext}velodyne_puck_link">
-      <material>Gazebo/DarkGrey</material>
-    </gazebo>
   </xacro:macro>
 </robot>
