Commit message: Update components with URDF guide

File: urdf/orbbec_astra.urdf.xacro (robot description, xacro)
@@ -13,5 +13,5 @@
       <xacro:property name="tf_prefix_ext" value="${tf_prefix}_" />
     </xacro:unless>
-    <joint name="${parent_link}_to_${tf_prefix_ext}orbbec_astra_link_joint" type="fixed">
+    <joint name="${parent_link.rstrip('_link')}_to_${tf_prefix_ext}orbbec_astra_joint" type="fixed">
       <origin xyz="${xyz}" rpy="${rpy}" />
       <parent link="${parent_link}" />
@@ -20,23 +20,33 @@
     <link name="${tf_prefix_ext}orbbec_astra_link">
       <visual>
+        <origin xyz="0.0 0.0 0.0" rpy="0.0 0.0 0.0"/>
         <geometry>
-          <mesh filename="file://$(find ros_components_description)/meshes/orbbec_astra.stl" scale="0.001 0.001 0.001" />
+          <mesh filename="file://$(find ros_components_description)/meshes/orbbec_astra.dae" />
         </geometry>
-        <origin xyz="-0.01 0.0 0.025" rpy="${pi/2} 0.0 ${pi/2}"/>
-        <material name="DarkGrey"/>
       </visual>
+      <!-- camera module collision -->
       <collision>
+        <origin xyz="${0.0225-0.04/2.0} 0.0 ${0.019+0.03/2.0}" rpy="0.0 0.0 0.0"/>
         <geometry>
-          <box size="0.165 0.04 0.05" />
+          <box size="0.04 0.165 0.03" />
         </geometry>
-        <origin xyz="-0.01 0.0 0.025" rpy="0.0 0.0 ${pi/2}"/>
+      </collision>
+      <!-- mounting base model collision -->
+      <collision>
+        <origin xyz="${0.0235-0.06/2.0} 0.0 ${0.019/2.0}" rpy="0.0 0.0 0.0"/>
+        <geometry>
+          <box size="0.06 0.06 0.019" />
+        </geometry>
       </collision>
       <inertial>
-        <mass value="0.105" />
-        <inertia ixx="1.0" ixy="0.0" ixz="0.0" iyy="1.0" iyz="0.0" izz="1.0" />
+        <origin xyz="0.0 0.0 ${0.019+0.01}" rpy="0.0 0.0 0.0" />
+        <mass value="0.300" />
+        <inertia ixx="0.00073916" ixy="0.0"        ixz="0.0"
+                                  iyy="0.00015435" iyz="0.0"
+                                                   izz="0.00077395" />
       </inertial>
     </link>
-    <joint name="${tf_prefix_ext}${frame_id}_link_joint" type="fixed">
-      <origin xyz="0.01 0.0 0.035" rpy="${-pi/2.0} 0.0 ${-pi/2.0}" />
+    <joint name="${tf_prefix_ext}orbbec_astra_to_${tf_prefix_ext}${frame_id.rstrip('_link')}_joint" type="fixed">
+      <origin xyz="0.01 0 0.035" rpy="${-pi/2} 0 ${-pi/2}" />
       <parent link="${tf_prefix_ext}orbbec_astra_link" />
       <child link="${tf_prefix_ext}${frame_id}" />
@@ -49,5 +59,5 @@
         <camera name="${tf_prefix_ext}camera">
         </camera>
-        <plugin name="plugin_name" filename="libgazebo_ros_camera.so">
+        <plugin name="${tf_prefix_ext}orbbec_astra_camera" filename="libgazebo_ros_camera.so">
           <ros>
             <namespace>${tf_prefix_ext}orbbec_astra_camera</namespace>
@@ -66,7 +76,4 @@
       </sensor>
     </gazebo>
-    <gazebo reference="${tf_prefix_ext}orbbec_astra_link">
-      <material>Gazebo/DarkGrey</material>
-    </gazebo>
   </xacro:macro>
 </robot>

File: urdf/ouster_os1_32.urdf.xacro (robot description, xacro)
@@ -7,10 +7,12 @@
                        topic:=os_lidar
                        frame_id:=os_lidar
-                       simulation_engine:=gazebo-classic">
+                       simulation_engine:=gazebo-classic" >
     <xacro:if value="${use_gpu}">
       <xacro:property name="ray_type" value="gpu_ray" />
+      <xacro:property name="plugin_file_name" value="libgazebo_ros_velodyne_gpu_laser.so" />
     </xacro:if>
     <xacro:unless value="${use_gpu}">
       <xacro:property name="ray_type" value="ray" />
+      <xacro:property name="plugin_file_name" value="libgazebo_ros_velodyne_laser.so" />
     </xacro:unless>
     <xacro:if value="${tf_prefix == 'None'}">
@@ -20,5 +22,5 @@
       <xacro:property name="tf_prefix_ext" value="${tf_prefix}" />
     </xacro:unless>
-    <joint name="${parent_link}_to_${tf_prefix_ext}ouster_os1_32_link_joint" type="fixed">
+    <joint name="${parent_link.rstrip('_link')}_to_${tf_prefix_ext}ouster_os1_32_joint" type="fixed">
       <origin xyz="${xyz}" rpy="${rpy}" />
       <parent link="${parent_link}" />
@@ -27,27 +29,29 @@
     <link name="${tf_prefix_ext}ouster_os1_32_link">
       <visual>
+        <origin xyz="0.0 0.0 0.0" rpy="0.0 0.0 0.0"/>
         <geometry>
-          <mesh filename="file://$(find ros_components_description)/meshes/ouster_os1_32.stl" scale="1.0 1.0 1.0" />
+          <mesh filename="file://$(find ros_components_description)/meshes/ouster_os1_32.dae" />
         </geometry>
-        <origin xyz="0.0 0.0 0.0" rpy="0.0 0.0 ${pi/2.0}"/>
-        <material name="Grey"/>
       </visual>
       <collision>
+        <origin xyz="0.0 0.0 ${0.072/2.0}" rpy="0.0 0.0 0.0"/>
         <geometry>
-          <cylinder radius="${0.0753/2.0}" length="0.0435" />
+          <cylinder radius="${0.085/2.0}" length="0.073" />
         </geometry>
-        <origin xyz="0.0 0.0 ${0.0435/2.0}" rpy="0.0 0.0 0.0"/>
       </collision>
       <inertial>
-          <mass value="0.447" />
-          <inertia ixx="1.0" ixy="0.0" ixz="0.0" iyy="1.0" iyz="0.0" izz="1.0" />
+        <origin xyz="0.0 0.0 ${0.072/2.0}" rpy="0.0 0.0 0.0" />
+        <mass value="0.447" />
+        <inertia ixx="0.00047706" ixy="0.0"        ixz="0.0"
+                                  iyy="0.00047706" iyz="0.0"
+                                                   izz="0.00053722" />
       </inertial>
     </link>
-    <joint name="${tf_prefix_ext}ouster_os1_32_link_to_${tf_prefix_ext}${frame_id}_joint" type="fixed">
-      <origin xyz="0.0 0.0 0.023" rpy="0.0 0.0 0.0" />
+    <joint name="${tf_prefix_ext}ouster_os1_32_to_${tf_prefix_ext}${frame_id.rstrip('_link')}_joint" type="fixed">
+      <origin xyz="0.0 0.0 0.03618" rpy="0.0 0.0 0.0" />
       <parent link="${tf_prefix_ext}ouster_os1_32_link" />
       <child link="${tf_prefix_ext}${frame_id}" />
     </joint>
-    <link name="${tf_prefix_ext}${frame_id}"></link>
+    <link name="${tf_prefix_ext}${frame_id}" />
     <gazebo reference="${tf_prefix_ext}${frame_id}">
       <sensor type="${ray_type}" name="${tf_prefix_ext}ouster_os1_32_sensor">
@@ -69,6 +73,6 @@
           </scan>
           <range>
-            <min>${0.0753/2.0+0.01}</min>
-            <max>100.0</max>
+            <min>${0.085/2.0+0.01}</min>
+            <max>120.0</max>
             <resolution>0.003</resolution>
           </range>
@@ -80,5 +84,5 @@
         </ray>
         <update_rate>10.0</update_rate>
-        <plugin name="scan" filename="libgazebo_ros_ray_sensor.so">
+        <plugin name="${tf_prefix_ext}ouster_os1_32_${ray_type}" filename="libgazebo_ros_ray_sensor.so">
           <ros>
             <namespace>/</namespace>
@@ -90,7 +94,4 @@
       </sensor>
     </gazebo>
-    <gazebo reference="${tf_prefix_ext}ouster_os1_32_link">
-      <material>Gazebo/Grey</material>
-    </gazebo>
   </xacro:macro>
 </robot>

File: urdf/velodyne_vlp_16.urdf.xacro (robot description, xacro)
@@ -1,5 +1,5 @@
 <?xml version="1.0"?>
 <robot xmlns:xacro="http://www.ros.org/wiki/xacro">
-  <xacro:macro name="velodyne_puck"
+  <xacro:macro name="velodyne_vlp_16"
                params="parent_link xyz rpy
                        use_gpu:=false
@@ -7,10 +7,12 @@
                        topic:=scan
                        frame_id:=velodyne
-                       simulation_engine:=gazebo-classic">
+                       simulation_engine:=gazebo-classic" >
     <xacro:if value="${use_gpu}">
       <xacro:property name="ray_type" value="gpu_ray" />
+      <xacro:property name="plugin_file_name" value="libgazebo_ros_velodyne_gpu_laser.so" />
     </xacro:if>
     <xacro:unless value="${use_gpu}">
       <xacro:property name="ray_type" value="ray" />
+      <xacro:property name="plugin_file_name" value="libgazebo_ros_velodyne_laser.so" />
     </xacro:unless>
     <xacro:if value="${tf_prefix == 'None'}">
@@ -20,34 +22,36 @@
       <xacro:property name="tf_prefix_ext" value="${tf_prefix}_" />
     </xacro:unless>
-    <joint name="${parent_link}_to_${tf_prefix_ext}velodyne_puck_link_joint" type="fixed">
+    <joint name="${parent_link.rstrip('_link')}_to_${tf_prefix_ext}velodyne_vlp_16_joint" type="fixed">
       <origin xyz="${xyz}" rpy="${rpy}" />
       <parent link="${parent_link}" />
-      <child link="${tf_prefix_ext}velodyne_puck_link" />
+      <child link="${tf_prefix_ext}velodyne_vlp_16_link" />
     </joint>
-    <link name="${tf_prefix_ext}velodyne_puck_link">
+    <link name="${tf_prefix_ext}velodyne_vlp_16_link">
       <visual>
+        <origin xyz="0.0 0.0 0.0" rpy="0.0 0.0 0.0"/>
         <geometry>
-          <mesh filename="file://$(find ros_components_description)/meshes/velodyne_puck.stl" scale="0.025035 0.025035 0.025035" />
+          <mesh filename="file://$(find ros_components_description)/meshes/velodyne_vlp_16.dae" />
         </geometry>
-        <origin xyz="0.0 0.0 0.0" rpy="${pi/2.0} 0.0 ${pi}"/>
-        <material name="DarkGrey"/>
       </visual>
       <collision>
+        <origin xyz="0.0 0.0 ${0.072/2.0}" rpy="0.0 0.0 0.0"/>
         <geometry>
-          <cylinder radius="${0.090/2.0}" length="0.0717" />
+          <cylinder radius="${0.103/2.0}" length="0.072" />
         </geometry>
-        <origin xyz="0.0 0.0 ${0.0717/2.0}" rpy="0.0 0.0 0.0"/>
       </collision>
       <inertial>
+        <origin xyz="0.0 0.0 ${0.072/2.0}" rpy="0.0 0.0 0.0" />
         <mass value="0.830" />
-        <inertia ixx="1.0" ixy="0.0" ixz="0.0" iyy="1.0" iyz="0.0" izz="1.0" />
+        <inertia ixx="0.001111" ixy="0.0"      ixz="0.0"
+                                iyy="0.001109" iyz="0.0"
+                                               izz="0.001493" />
       </inertial>
     </link>
-    <joint name="${tf_prefix_ext}velodyne_puck_link_joint_to_${tf_prefix_ext}${frame_id}_joint" type="fixed">
+    <joint name="${tf_prefix_ext}velodyne_vlp_16_to_${tf_prefix_ext}${frame_id.rstrip('_link')}_joint" type="fixed">
       <origin xyz="0.0 0.0 0.0378" rpy="0.0 0.0 0.0" />
-      <parent link="${tf_prefix_ext}velodyne_puck_link" />
+      <parent link="${tf_prefix_ext}velodyne_vlp_16_link" />
       <child link="${tf_prefix_ext}${frame_id}" />
     </joint>
-    <link name="${tf_prefix_ext}${frame_id}"></link>
+    <link name="${tf_prefix_ext}${frame_id}" />
     <gazebo reference="${tf_prefix_ext}${frame_id}">
       <sensor type="${ray_type}" name="${tf_prefix_ext}velodyne_puck_sensor">
@@ -69,7 +73,7 @@
           </scan>
           <range>
-            <min>${0.051+0.01}</min>
+            <min>${0.103/2.0+0.01}</min>
             <max>100.0</max>
-            <resolution>0.005</resolution>
+            <resolution>0.003</resolution>
           </range>
           <noise>
@@ -80,5 +84,5 @@
         </ray>
         <update_rate>10.0</update_rate>
-        <plugin name="scan" filename="libgazebo_ros_ray_sensor.so">
+        <plugin name="${tf_prefix_ext}velodyne_vlp_16_${ray_type}" filename="libgazebo_ros_ray_sensor.so">
           <ros>
             <namespace>/</namespace>
@@ -90,7 +94,4 @@
       </sensor>
     </gazebo>
-    <gazebo reference="${tf_prefix_ext}velodyne_puck_link">
-      <material>Gazebo/DarkGrey</material>
-    </gazebo>
   </xacro:macro>
 </robot>

Commit message: FIx velodyne name, ouser link and astra plugin

File: urdf/orbbec_astra.urdf.xacro (robot description, xacro)
@@ -71,5 +71,5 @@
           </clip>
         </camera>
-        <plugin name="kinect_controller" filename="libgazebo_ros_openni_kinect.so">
+        <plugin name="${tf_prefix_ext}orbbec_astra_camera" filename="libgazebo_ros_openni_kinect.so">
           <alwaysOn>true</alwaysOn>
           <updateRate>10.0</updateRate>

File: urdf/ouster_os1_32.urdf.xacro (robot description, xacro)
@@ -49,5 +49,5 @@
     </link>
     <joint name="${tf_prefix_ext}ouster_os1_32_to_${tf_prefix_ext}${frame_id.rstrip('_link')}_joint" type="fixed">
-      <origin xyz="0.0 0.0 0.023" rpy="0.0 0.0 0.0" />
+      <origin xyz="0.0 0.0 0.03618" rpy="0.0 0.0 0.0" />
       <parent link="${tf_prefix_ext}ouster_os1_32_link" />
       <child link="${tf_prefix_ext}${frame_id}" />

File: urdf/velodyne_puck.urdf.xacro (robot description, xacro)
@@ -1,5 +1,5 @@
 <?xml version="1.0"?>
 <robot xmlns:xacro="http://www.ros.org/wiki/xacro">
-  <xacro:macro name="velodyne_vlp_16"
+  <xacro:macro name="velodyne_puck"
                params="parent_link xyz rpy
                        use_gpu:=false
@@ -22,14 +22,14 @@
       <xacro:property name="tf_prefix_ext" value="${tf_prefix}_" />
     </xacro:unless>
-    <joint name="${parent_link.rstrip('_link')}_to_${tf_prefix_ext}velodyne_vlp_16_joint" type="fixed">
+    <joint name="${parent_link.rstrip('_link')}_to_${tf_prefix_ext}velodyne_puck_joint" type="fixed">
       <origin xyz="${xyz}" rpy="${rpy}" />
       <parent link="${parent_link}" />
-      <child link="${tf_prefix_ext}velodyne_vlp_16_link" />
+      <child link="${tf_prefix_ext}velodyne_puck_link" />
     </joint>
-    <link name="${tf_prefix_ext}velodyne_vlp_16_link">
+    <link name="${tf_prefix_ext}velodyne_puck_link">
       <visual>
         <origin xyz="0.0 0.0 0.0" rpy="0.0 0.0 0.0"/>
         <geometry>
-          <mesh filename="file://$(find ros_components_description)/meshes/velodyne_vlp_16.dae" />
+          <mesh filename="file://$(find ros_components_description)/meshes/velodyne_puck.dae" />
         </geometry>
       </visual>
@@ -48,12 +48,12 @@
       </inertial>
     </link>
-    <joint name="${tf_prefix_ext}velodyne_vlp_16_to_${tf_prefix_ext}${frame_id.rstrip('_link')}_joint" type="fixed">
+    <joint name="${tf_prefix_ext}velodyne_puck_to_${tf_prefix_ext}${frame_id.rstrip('_link')}_joint" type="fixed">
       <origin xyz="0.0 0.0 0.0378" rpy="0.0 0.0 0.0" />
-      <parent link="${tf_prefix_ext}velodyne_vlp_16_link" />
+      <parent link="${tf_prefix_ext}velodyne_puck_link" />
       <child link="${tf_prefix_ext}${frame_id}" />
     </joint>
     <link name="${tf_prefix_ext}${frame_id}" />
     <gazebo reference="${tf_prefix_ext}${frame_id}">
-      <sensor type="${ray_type}" name="${tf_prefix_ext}velodyne_vlp_16_sensor">
+      <sensor type="${ray_type}" name="${tf_prefix_ext}velodyne_puck_sensor">
         <visualize>false</visualize>
         <update_rate>10</update_rate>
@@ -84,5 +84,5 @@
           </noise>
         </ray>
-        <plugin name="${tf_prefix_ext}velodyne_vlp_16_${ray_type}" filename="${plugin_file_name}">
+        <plugin name="${tf_prefix_ext}velodyne_puck_${ray_type}" filename="${plugin_file_name}">
           <topicName>${topic}</topicName>
           <frameName>${tf_prefix_ext}${frame_id}</frameName>
