Commit message: Update components with URDF guide (#9)
* Update components with URDF guide

* Update readme

* Update env variable name

* Fix Velodyne name

* Change env name, add ignition dependency and fix namespace

* Apply remapping to all sensors

* Change namespaces

* Fix namespace for ignition

File: urdf/orbbec_astra.urdf.xacro (robot description, xacro)
@@ -13,5 +13,5 @@
       <xacro:property name="tf_prefix_ext" value="${tf_prefix}_" />
     </xacro:unless>
-    <joint name="${parent_link}_to_${tf_prefix_ext}orbbec_astra_link_joint" type="fixed">
+    <joint name="${parent_link.rstrip('_link')}_to_${tf_prefix_ext}orbbec_astra_joint" type="fixed">
       <origin xyz="${xyz}" rpy="${rpy}" />
       <parent link="${parent_link}" />
@@ -20,23 +20,33 @@
     <link name="${tf_prefix_ext}orbbec_astra_link">
       <visual>
+        <origin xyz="0.0 0.0 0.0" rpy="0.0 0.0 0.0"/>
         <geometry>
-          <mesh filename="file://$(find ros_components_description)/meshes/orbbec_astra.stl" scale="0.001 0.001 0.001" />
+          <mesh filename="file://$(find ros_components_description)/meshes/orbbec_astra.dae" />
         </geometry>
-        <origin xyz="-0.01 0.0 0.025" rpy="${pi/2} 0.0 ${pi/2}"/>
-        <material name="DarkGrey"/>
       </visual>
+      <!-- camera module collision -->
       <collision>
+        <origin xyz="${0.0225-0.04/2.0} 0.0 ${0.019+0.03/2.0}" rpy="0.0 0.0 0.0"/>
         <geometry>
-          <box size="0.165 0.04 0.05" />
+          <box size="0.04 0.165 0.03" />
         </geometry>
-        <origin xyz="-0.01 0.0 0.025" rpy="0.0 0.0 ${pi/2}"/>
+      </collision>
+      <!-- mounting base model collision -->
+      <collision>
+        <origin xyz="${0.0235-0.06/2.0} 0.0 ${0.019/2.0}" rpy="0.0 0.0 0.0"/>
+        <geometry>
+          <box size="0.06 0.06 0.019" />
+        </geometry>
       </collision>
       <inertial>
-        <mass value="0.105" />
-        <inertia ixx="1.0" ixy="0.0" ixz="0.0" iyy="1.0" iyz="0.0" izz="1.0" />
+        <origin xyz="0.0 0.0 ${0.019+0.01}" rpy="0.0 0.0 0.0" />
+        <mass value="0.300" />
+        <inertia ixx="0.00073916" ixy="0.0"        ixz="0.0"
+                                  iyy="0.00015435" iyz="0.0"
+                                                   izz="0.00077395" />
       </inertial>
     </link>
-    <joint name="${tf_prefix_ext}${frame_id}_link_joint" type="fixed">
-      <origin xyz="0.01 0.0 0.035" rpy="${-pi/2.0} 0.0 ${-pi/2.0}" />
+    <joint name="${tf_prefix_ext}orbbec_astra_to_${tf_prefix_ext}${frame_id.rstrip('_link')}_joint" type="fixed">
+      <origin xyz="0.01 0 0.035" rpy="${-pi/2} 0 ${-pi/2}" />
       <parent link="${tf_prefix_ext}orbbec_astra_link" />
       <child link="${tf_prefix_ext}${frame_id}" />
@@ -49,12 +59,12 @@
         <camera name="${tf_prefix_ext}camera">
         </camera>
-        <plugin name="plugin_name" filename="libgazebo_ros_camera.so">
+        <plugin name="${tf_prefix_ext}orbbec_astra_camera" filename="libgazebo_ros_camera.so">
           <ros>
-            <namespace>${tf_prefix_ext}orbbec_astra_camera</namespace>
-            <argument>custom_camera/image_raw:=rgb/image_raw</argument>
-            <argument>custom_camera/image_depth:=depth/image_raw</argument>
-            <argument>custom_camera/camera_info:=rgb/camera_info</argument>
-            <argument>custom_camera/camera_info_depth:=depth/camera_info</argument>
-            <argument>custom_camera/points:=depth/points</argument>
+            <namespace>orbbec_astra_camera</namespace>
+            <remapping>custom_camera/image_raw:=rgb/image_raw</remapping>
+            <remapping>custom_camera/image_depth:=depth/image_raw</remapping>
+            <remapping>custom_camera/camera_info:=rgb/camera_info</remapping>
+            <remapping>custom_camera/camera_info_depth:=depth/camera_info</remapping>
+            <remapping>custom_camera/points:=depth/points</remapping>
           </ros>
           <camera_name>${tf_prefix_ext}camera</camera_name>
@@ -66,7 +76,4 @@
       </sensor>
     </gazebo>
-    <gazebo reference="${tf_prefix_ext}orbbec_astra_link">
-      <material>Gazebo/DarkGrey</material>
-    </gazebo>
   </xacro:macro>
 </robot>

File: urdf/ouster_os1_32.urdf.xacro (robot description, xacro)
@@ -7,10 +7,12 @@
                        topic:=os_lidar
                        frame_id:=os_lidar
-                       simulation_engine:=gazebo-classic">
+                       simulation_engine:=gazebo-classic" >
     <xacro:if value="${use_gpu}">
       <xacro:property name="ray_type" value="gpu_ray" />
+      <xacro:property name="plugin_file_name" value="libgazebo_ros_velodyne_gpu_laser.so" />
     </xacro:if>
     <xacro:unless value="${use_gpu}">
       <xacro:property name="ray_type" value="ray" />
+      <xacro:property name="plugin_file_name" value="libgazebo_ros_velodyne_laser.so" />
     </xacro:unless>
     <xacro:if value="${tf_prefix == 'None'}">
@@ -20,5 +22,5 @@
       <xacro:property name="tf_prefix_ext" value="${tf_prefix}" />
     </xacro:unless>
-    <joint name="${parent_link}_to_${tf_prefix_ext}ouster_os1_32_link_joint" type="fixed">
+    <joint name="${parent_link.rstrip('_link')}_to_${tf_prefix_ext}ouster_os1_32_joint" type="fixed">
       <origin xyz="${xyz}" rpy="${rpy}" />
       <parent link="${parent_link}" />
@@ -27,27 +29,29 @@
     <link name="${tf_prefix_ext}ouster_os1_32_link">
       <visual>
+        <origin xyz="0.0 0.0 0.0" rpy="0.0 0.0 0.0"/>
         <geometry>
-          <mesh filename="file://$(find ros_components_description)/meshes/ouster_os1_32.stl" scale="1.0 1.0 1.0" />
+          <mesh filename="file://$(find ros_components_description)/meshes/ouster_os1_32.dae" />
         </geometry>
-        <origin xyz="0.0 0.0 0.0" rpy="0.0 0.0 ${pi/2.0}"/>
-        <material name="Grey"/>
       </visual>
       <collision>
+        <origin xyz="0.0 0.0 ${0.072/2.0}" rpy="0.0 0.0 0.0"/>
         <geometry>
-          <cylinder radius="${0.0753/2.0}" length="0.0435" />
+          <cylinder radius="${0.085/2.0}" length="0.073" />
         </geometry>
-        <origin xyz="0.0 0.0 ${0.0435/2.0}" rpy="0.0 0.0 0.0"/>
       </collision>
       <inertial>
-          <mass value="0.447" />
-          <inertia ixx="1.0" ixy="0.0" ixz="0.0" iyy="1.0" iyz="0.0" izz="1.0" />
+        <origin xyz="0.0 0.0 ${0.072/2.0}" rpy="0.0 0.0 0.0" />
+        <mass value="0.447" />
+        <inertia ixx="0.00047706" ixy="0.0"        ixz="0.0"
+                                  iyy="0.00047706" iyz="0.0"
+                                                   izz="0.00053722" />
       </inertial>
     </link>
-    <joint name="${tf_prefix_ext}ouster_os1_32_link_to_${tf_prefix_ext}${frame_id}_joint" type="fixed">
-      <origin xyz="0.0 0.0 0.023" rpy="0.0 0.0 0.0" />
+    <joint name="${tf_prefix_ext}ouster_os1_32_to_${tf_prefix_ext}${frame_id.rstrip('_link')}_joint" type="fixed">
+      <origin xyz="0.0 0.0 0.03618" rpy="0.0 0.0 0.0" />
       <parent link="${tf_prefix_ext}ouster_os1_32_link" />
       <child link="${tf_prefix_ext}${frame_id}" />
     </joint>
-    <link name="${tf_prefix_ext}${frame_id}"></link>
+    <link name="${tf_prefix_ext}${frame_id}" />
     <gazebo reference="${tf_prefix_ext}${frame_id}">
       <sensor type="${ray_type}" name="${tf_prefix_ext}ouster_os1_32_sensor">
@@ -69,6 +73,6 @@
           </scan>
           <range>
-            <min>${0.0753/2.0+0.01}</min>
-            <max>100.0</max>
+            <min>${0.085/2.0+0.01}</min>
+            <max>120.0</max>
             <resolution>0.003</resolution>
           </range>
@@ -80,8 +84,8 @@
         </ray>
         <update_rate>10.0</update_rate>
-        <plugin name="scan" filename="libgazebo_ros_ray_sensor.so">
+        <plugin name="${tf_prefix_ext}ouster_os1_32_${ray_type}" filename="libgazebo_ros_ray_sensor.so">
           <ros>
-            <namespace>/</namespace>
-            <argument>~/out:=${topic}</argument>
+            <namespace></namespace>
+            <remapping>~/out:=${topic}</remapping>
           </ros>
           <output_type>sensor_msgs/PointCloud2</output_type>
@@ -90,7 +94,4 @@
       </sensor>
     </gazebo>
-    <gazebo reference="${tf_prefix_ext}ouster_os1_32_link">
-      <material>Gazebo/Grey</material>
-    </gazebo>
   </xacro:macro>
 </robot>

File: urdf/velodyne_puck.urdf.xacro (robot description, xacro)
@@ -7,10 +7,12 @@
                        topic:=scan
                        frame_id:=velodyne
-                       simulation_engine:=gazebo-classic">
+                       simulation_engine:=gazebo-classic" >
     <xacro:if value="${use_gpu}">
       <xacro:property name="ray_type" value="gpu_ray" />
+      <xacro:property name="plugin_file_name" value="libgazebo_ros_velodyne_gpu_laser.so" />
     </xacro:if>
     <xacro:unless value="${use_gpu}">
       <xacro:property name="ray_type" value="ray" />
+      <xacro:property name="plugin_file_name" value="libgazebo_ros_velodyne_laser.so" />
     </xacro:unless>
     <xacro:if value="${tf_prefix == 'None'}">
@@ -20,5 +22,5 @@
       <xacro:property name="tf_prefix_ext" value="${tf_prefix}_" />
     </xacro:unless>
-    <joint name="${parent_link}_to_${tf_prefix_ext}velodyne_puck_link_joint" type="fixed">
+    <joint name="${parent_link.rstrip('_link')}_to_${tf_prefix_ext}velodyne_puck_joint" type="fixed">
       <origin xyz="${xyz}" rpy="${rpy}" />
       <parent link="${parent_link}" />
@@ -27,27 +29,29 @@
     <link name="${tf_prefix_ext}velodyne_puck_link">
       <visual>
+        <origin xyz="0.0 0.0 0.0" rpy="0.0 0.0 0.0"/>
         <geometry>
-          <mesh filename="file://$(find ros_components_description)/meshes/velodyne_puck.stl" scale="0.025035 0.025035 0.025035" />
+          <mesh filename="file://$(find ros_components_description)/meshes/velodyne_puck.dae" />
         </geometry>
-        <origin xyz="0.0 0.0 0.0" rpy="${pi/2.0} 0.0 ${pi}"/>
-        <material name="DarkGrey"/>
       </visual>
       <collision>
+        <origin xyz="0.0 0.0 ${0.072/2.0}" rpy="0.0 0.0 0.0"/>
         <geometry>
-          <cylinder radius="${0.090/2.0}" length="0.0717" />
+          <cylinder radius="${0.103/2.0}" length="0.072" />
         </geometry>
-        <origin xyz="0.0 0.0 ${0.0717/2.0}" rpy="0.0 0.0 0.0"/>
       </collision>
       <inertial>
+        <origin xyz="0.0 0.0 ${0.072/2.0}" rpy="0.0 0.0 0.0" />
         <mass value="0.830" />
-        <inertia ixx="1.0" ixy="0.0" ixz="0.0" iyy="1.0" iyz="0.0" izz="1.0" />
+        <inertia ixx="0.001111" ixy="0.0"      ixz="0.0"
+                                iyy="0.001109" iyz="0.0"
+                                               izz="0.001493" />
       </inertial>
     </link>
-    <joint name="${tf_prefix_ext}velodyne_puck_link_joint_to_${tf_prefix_ext}${frame_id}_joint" type="fixed">
+    <joint name="${tf_prefix_ext}velodyne_puck_to_${tf_prefix_ext}${frame_id.rstrip('_link')}_joint" type="fixed">
       <origin xyz="0.0 0.0 0.0378" rpy="0.0 0.0 0.0" />
       <parent link="${tf_prefix_ext}velodyne_puck_link" />
       <child link="${tf_prefix_ext}${frame_id}" />
     </joint>
-    <link name="${tf_prefix_ext}${frame_id}"></link>
+    <link name="${tf_prefix_ext}${frame_id}" />
     <gazebo reference="${tf_prefix_ext}${frame_id}">
       <sensor type="${ray_type}" name="${tf_prefix_ext}velodyne_puck_sensor">
@@ -69,7 +73,7 @@
           </scan>
           <range>
-            <min>${0.051+0.01}</min>
+            <min>${0.103/2.0+0.01}</min>
             <max>100.0</max>
-            <resolution>0.005</resolution>
+            <resolution>0.003</resolution>
           </range>
           <noise>
@@ -80,8 +84,8 @@
         </ray>
         <update_rate>10.0</update_rate>
-        <plugin name="scan" filename="libgazebo_ros_ray_sensor.so">
+        <plugin name="${tf_prefix_ext}velodyne_puck_${ray_type}" filename="libgazebo_ros_ray_sensor.so">
           <ros>
-            <namespace>/</namespace>
-            <argument>~/out:=${topic}</argument>
+            <namespace></namespace>
+            <remapping>~/out:=${topic}</remapping>
           </ros>
           <output_type>sensor_msgs/PointCloud2</output_type>
@@ -90,7 +94,4 @@
       </sensor>
     </gazebo>
-    <gazebo reference="${tf_prefix_ext}velodyne_puck_link">
-      <material>Gazebo/DarkGrey</material>
-    </gazebo>
   </xacro:macro>
 </robot>

Commit message: Fix formatting

File: urdf/orbbec_astra.urdf.xacro (robot description, xacro)
@@ -20,5 +20,5 @@
     <link name="${tf_prefix_ext}orbbec_astra_link">
       <visual>
-        <origin xyz="0.0 0.0 0.0" rpy="0.0 0.0 0.0"/>
+        <origin xyz="0.0 0.0 0.0" rpy="0.0 0.0 0.0" />
         <geometry>
           <mesh filename="file://$(find ros_components_description)/meshes/orbbec_astra.dae" />
@@ -27,5 +27,5 @@
       <!-- camera module collision -->
       <collision>
-        <origin xyz="${0.0225-0.04/2.0} 0.0 ${0.019+0.03/2.0}" rpy="0.0 0.0 0.0"/>
+        <origin xyz="${0.0225-0.04/2.0} 0.0 ${0.019+0.03/2.0}" rpy="0.0 0.0 0.0" />
         <geometry>
           <box size="0.04 0.165 0.03" />
@@ -34,5 +34,5 @@
       <!-- mounting base model collision -->
       <collision>
-        <origin xyz="${0.0235-0.06/2.0} 0.0 ${0.019/2.0}" rpy="0.0 0.0 0.0"/>
+        <origin xyz="${0.0235-0.06/2.0} 0.0 ${0.019/2.0}" rpy="0.0 0.0 0.0" />
         <geometry>
           <box size="0.06 0.06 0.019" />
@@ -48,5 +48,5 @@
     </link>
     <joint name="${tf_prefix_ext}orbbec_astra_to_${tf_prefix_ext}${frame_id.rstrip('_link')}_joint" type="fixed">
-      <origin xyz="0.01 0 0.035" rpy="${-pi/2} 0 ${-pi/2}" />
+      <origin xyz="0.01 0.0 0.035" rpy="${-pi/2} 0.0 ${-pi/2}" />
       <parent link="${tf_prefix_ext}orbbec_astra_link" />
       <child link="${tf_prefix_ext}${frame_id}" />
@@ -55,6 +55,6 @@
     <gazebo reference="${tf_prefix_ext}orbbec_astra_link">
       <sensor type="depth" name="${tf_prefix_ext}orbbec_astra_camera">
-        <always_on>1</always_on>
-        <update_rate>20</update_rate>
+        <always_on>true</always_on>
+        <update_rate>20.0</update_rate>
         <camera name="${tf_prefix_ext}camera">
           <horizontal_fov>${60/180*pi}</horizontal_fov>

File: urdf/ouster_os1_32.urdf.xacro (robot description, xacro)
@@ -7,5 +7,5 @@
                        topic:=os_lidar
                        frame_id:=os_lidar
-                       simulation_engine:=gazebo-classic" >
+                       simulation_engine:=gazebo-classic">
     <xacro:if value="${use_gpu}">
       <xacro:property name="ray_type" value="gpu_ray" />
@@ -29,5 +29,5 @@
     <link name="${tf_prefix_ext}ouster_os1_32_link">
       <visual>
-        <origin xyz="0.0 0.0 0.0" rpy="0.0 0.0 0.0"/>
+        <origin xyz="0.0 0.0 0.0" rpy="0.0 0.0 0.0" />
         <geometry>
           <mesh filename="file://$(find ros_components_description)/meshes/ouster_os1_32.dae" />
@@ -35,5 +35,5 @@
       </visual>
       <collision>
-        <origin xyz="0.0 0.0 ${0.072/2.0}" rpy="0.0 0.0 0.0"/>
+        <origin xyz="0.0 0.0 ${0.072/2.0}" rpy="0.0 0.0 0.0" />
         <geometry>
           <cylinder radius="${0.085/2.0}" length="0.073" />

File: urdf/slamtec_rplidar_a2.urdf.xacro (robot description, xacro)
@@ -13,5 +13,5 @@
                        frame_id:=laser
                        model:=A2M12
-                       simulation_engine:=gazebo-classic" >
+                       simulation_engine:=gazebo-classic">
     <xacro:if value="${use_gpu}">
       <xacro:property name="ray_type" value="gpu_ray" />
@@ -50,5 +50,5 @@
     <link name="${tf_prefix_ext}slamtec_rplidar_a2_link">
       <visual>
-        <origin xyz="0.0 0.0 0.0" rpy="0.0 0.0 0.0"/>
+        <origin xyz="0.0 0.0 0.0" rpy="0.0 0.0 0.0" />
         <geometry>
           <mesh filename="file://$(find ros_components_description)/meshes/${mesh}" />
@@ -56,5 +56,5 @@
       </visual>
       <collision>
-        <origin xyz="0.0 0.0 ${0.041/2.0}" rpy="0.0 0.0 0.0"/>
+        <origin xyz="0.0 0.0 ${0.041/2.0}" rpy="0.0 0.0 0.0" />
         <geometry>
           <cylinder radius="${0.076/2.0}" length="0.041" />
@@ -70,5 +70,5 @@
     </link>
     <joint name="${tf_prefix_ext}slamtec_rplidar_a2_to_${tf_prefix_ext}${frame_id.rstrip('_link')}_joint" type="fixed">
-      <origin xyz="0 0 0.031" rpy="0.0 0.0 ${pi}" />
+      <origin xyz="0.0 0.0 0.031" rpy="0.0 0.0 ${pi}" />
       <parent link="${tf_prefix_ext}slamtec_rplidar_a2_link" />
       <child link="${tf_prefix_ext}${frame_id}" />
@@ -115,5 +115,4 @@
       <gazebo reference="${tf_prefix_ext}${frame_id}">
         <sensor type="${ray_type}" name="${tf_prefix_ext}slamtec_rplidar_a2_sensor">
-          <pose>0 0 0.04 0 0 0</pose>
           <visualize>false</visualize>
           <ray>
@@ -137,5 +136,5 @@
             </noise>
           </ray>
-          <update_rate>10</update_rate>
+          <update_rate>10.0</update_rate>
           <plugin name="scan" filename="libgazebo_ros_ray_sensor.so">
             <ros>

File: urdf/slamtec_rplidar_a3.urdf.xacro (robot description, xacro)
@@ -7,5 +7,5 @@
                        topic:=scan
                        frame_id:=laser
-                       simulation_engine:=gazebo-classic" >
+                       simulation_engine:=gazebo-classic">
     <xacro:if value="${use_gpu}">
       <xacro:property name="ray_type" value="gpu_ray" />
@@ -27,5 +27,5 @@
     <link name="${tf_prefix_ext}slamtec_rplidar_a3_link">
       <visual>
-        <origin xyz="0.0 0.0 0.0" rpy="0.0 0.0 0.0"/>
+        <origin xyz="0.0 0.0 0.0" rpy="0.0 0.0 0.0" />
         <geometry>
           <!-- slamtec_rplidar_ax.dae is used as a shared mesh for A2 and A3 rplidars -->
@@ -34,5 +34,5 @@
       </visual>
       <collision>
-        <origin xyz="0.0 0.0 ${0.041/2.0}" rpy="0.0 0.0 0.0"/>
+        <origin xyz="0.0 0.0 ${0.041/2.0}" rpy="0.0 0.0 0.0" />
         <geometry>
           <cylinder radius="${0.076/2.0}" length="0.041" />
@@ -48,5 +48,5 @@
     </link>
     <joint name="${tf_prefix_ext}slamtec_rplidar_a3_to_${tf_prefix_ext}${frame_id.rstrip('_link')}_joint" type="fixed">
-      <origin xyz="0 0 0.031" rpy="0.0 0.0 ${pi}" />
+      <origin xyz="0.0 0.0 0.031" rpy="0.0 0.0 ${pi}" />
       <parent link="${tf_prefix_ext}slamtec_rplidar_a3_link" />
       <child link="${tf_prefix_ext}${frame_id}" />
@@ -94,5 +94,4 @@
       <gazebo reference="${tf_prefix_ext}${frame_id}">
         <sensor type="${ray_type}" name="${tf_prefix_ext}slamtec_rplidar_a3_sensor">
-          <pose>0 0 0.04 0 0 0</pose>
           <visualize>false</visualize>
           <ray>
@@ -107,5 +106,5 @@
             <range>
               <min>0.2</min>
-              <!-- as an tradoff between white and black object range -->
+              <!-- as an tradeoff between white and black object range -->
               <max>16.0</max>
               <resolution>0.05</resolution>
@@ -117,5 +116,5 @@
             </noise>
           </ray>
-          <update_rate>10</update_rate>
+          <update_rate>10.0</update_rate>
           <plugin name="scan" filename="libgazebo_ros_ray_sensor.so">
             <ros>

File: urdf/slamtec_rplidar_s1.urdf.xacro (robot description, xacro)
@@ -7,5 +7,5 @@
                        topic:=scan
                        frame_id:=laser
-                       simulation_engine:=gazebo-classic" >
+                       simulation_engine:=gazebo-classic">
     <xacro:if value="${use_gpu}">
       <xacro:property name="ray_type" value="gpu_ray" />
@@ -27,5 +27,5 @@
     <link name="${tf_prefix_ext}slamtec_rplidar_s1_link">
       <visual>
-        <origin xyz="0.0 0.0 0.0" rpy="0.0 0.0 0.0"/>
+        <origin xyz="0.0 0.0 0.0" rpy="0.0 0.0 0.0" />
         <geometry>
           <mesh filename="file://$(find ros_components_description)/meshes/slamtec_rplidar_s1.dae" />
@@ -34,5 +34,5 @@
       <!-- spinning head collision -->
       <collision>
-        <origin xyz="0.0 0.0 ${0.051/2.0}" rpy="0.0 0.0 0.0"/>
+        <origin xyz="0.0 0.0 ${0.051/2.0}" rpy="0.0 0.0 0.0" />
         <geometry>
           <cylinder radius="${0.0555/2.0}" length="0.051" />
@@ -41,5 +41,5 @@
       <!-- base collision -->
       <collision>
-        <origin xyz="0.0 0.0 ${0.0195/2.0}" rpy="0.0 0.0 0.0"/>
+        <origin xyz="0.0 0.0 ${0.0195/2.0}" rpy="0.0 0.0 0.0" />
         <geometry>
           <box size="0.0555 0.0555 0.0195" />
@@ -55,5 +55,5 @@
     </link>
     <joint name="${tf_prefix_ext}slamtec_rplidar_s1_to_${tf_prefix_ext}${frame_id.rstrip('_link')}_joint" type="fixed">
-      <origin xyz="0 0 0.04" rpy="0.0 0.0 ${pi}" />
+      <origin xyz="0.0 0.0 0.04" rpy="0.0 0.0 ${pi}" />
       <parent link="${tf_prefix_ext}slamtec_rplidar_s1_link" />
       <child link="${tf_prefix_ext}${frame_id}" />
@@ -100,5 +100,4 @@
       <gazebo reference="${tf_prefix_ext}${frame_id}">
         <sensor type="${ray_type}" name="${tf_prefix_ext}slamtec_rplidar_s1_sensor">
-          <pose>0 0 0.04 0 0 0</pose>
           <visualize>false</visualize>
           <ray>
@@ -122,5 +121,5 @@
             </noise>
           </ray>
-          <update_rate>10</update_rate>
+          <update_rate>10.0</update_rate>
           <plugin name="scan" filename="libgazebo_ros_ray_sensor.so">
             <ros>

File: urdf/velodyne_puck.urdf.xacro (robot description, xacro)
@@ -7,5 +7,5 @@
                        topic:=scan
                        frame_id:=velodyne
-                       simulation_engine:=gazebo-classic" >
+                       simulation_engine:=gazebo-classic">
     <xacro:if value="${use_gpu}">
       <xacro:property name="ray_type" value="gpu_ray" />
@@ -29,5 +29,5 @@
     <link name="${tf_prefix_ext}velodyne_puck_link">
       <visual>
-        <origin xyz="0.0 0.0 0.0" rpy="0.0 0.0 0.0"/>
+        <origin xyz="0.0 0.0 0.0" rpy="0.0 0.0 0.0" />
         <geometry>
           <mesh filename="file://$(find ros_components_description)/meshes/velodyne_puck.dae" />
@@ -35,5 +35,5 @@
       </visual>
       <collision>
-        <origin xyz="0.0 0.0 ${0.072/2.0}" rpy="0.0 0.0 0.0"/>
+        <origin xyz="0.0 0.0 ${0.072/2.0}" rpy="0.0 0.0 0.0" />
         <geometry>
           <cylinder radius="${0.103/2.0}" length="0.072" />
