Commit message: Fix formatting

File: urdf/orbbec_astra.urdf.xacro (robot description, xacro)
@@ -20,5 +20,5 @@
     <link name="${tf_prefix_ext}orbbec_astra_link">
       <visual>
-        <origin xyz="0.0 0.0 0.0" rpy="0.0 0.0 0.0"/>
+        <origin xyz="0.0 0.0 0.0" rpy="0.0 0.0 0.0" />
         <geometry>
           <mesh filename="file://$(find ros_components_description)/meshes/orbbec_astra.dae" />
@@ -27,5 +27,5 @@
       <!-- camera module collision -->
       <collision>
-        <origin xyz="${0.0225-0.04/2.0} 0.0 ${0.019+0.03/2.0}" rpy="0.0 0.0 0.0"/>
+        <origin xyz="${0.0225-0.04/2.0} 0.0 ${0.019+0.03/2.0}" rpy="0.0 0.0 0.0" />
         <geometry>
           <box size="0.04 0.165 0.03" />
@@ -34,5 +34,5 @@
       <!-- mounting base model collision -->
       <collision>
-        <origin xyz="${0.0235-0.06/2.0} 0.0 ${0.019/2.0}" rpy="0.0 0.0 0.0"/>
+        <origin xyz="${0.0235-0.06/2.0} 0.0 ${0.019/2.0}" rpy="0.0 0.0 0.0" />
         <geometry>
           <box size="0.06 0.06 0.019" />
@@ -48,5 +48,5 @@
     </link>
     <joint name="${tf_prefix_ext}orbbec_astra_to_${tf_prefix_ext}${frame_id.rstrip('_link')}_joint" type="fixed">
-      <origin xyz="0.01 0 0.035" rpy="${-pi/2} 0 ${-pi/2}" />
+      <origin xyz="0.01 0.0 0.035" rpy="${-pi/2} 0.0 ${-pi/2}" />
       <parent link="${tf_prefix_ext}orbbec_astra_link" />
       <child link="${tf_prefix_ext}${frame_id}" />
@@ -55,6 +55,5 @@
     <gazebo reference="${tf_prefix_ext}orbbec_astra_link">
       <sensor type="depth" name="${tf_prefix_ext}orbbec_astra_camera">
-        <always_on>1</always_on>
-        <visualize>true</visualize>
+        <always_on>true</always_on>
         <camera>
           <horizontal_fov>${60/180*pi}</horizontal_fov>

File: urdf/ouster_os1_32.urdf.xacro (robot description, xacro)
@@ -7,5 +7,5 @@
                        topic:=os_lidar
                        frame_id:=os_lidar
-                       simulation_engine:=gazebo-classic" >
+                       simulation_engine:=gazebo-classic">
     <xacro:if value="${use_gpu}">
       <xacro:property name="ray_type" value="gpu_ray" />
@@ -29,5 +29,5 @@
     <link name="${tf_prefix_ext}ouster_os1_32_link">
       <visual>
-        <origin xyz="0.0 0.0 0.0" rpy="0.0 0.0 0.0"/>
+        <origin xyz="0.0 0.0 0.0" rpy="0.0 0.0 0.0" />
         <geometry>
           <mesh filename="file://$(find ros_components_description)/meshes/ouster_os1_32.dae" />
@@ -35,5 +35,5 @@
       </visual>
       <collision>
-        <origin xyz="0.0 0.0 ${0.072/2.0}" rpy="0.0 0.0 0.0"/>
+        <origin xyz="0.0 0.0 ${0.072/2.0}" rpy="0.0 0.0 0.0" />
         <geometry>
           <cylinder radius="${0.085/2.0}" length="0.073" />
@@ -57,5 +57,5 @@
       <sensor type="${ray_type}" name="${tf_prefix_ext}ouster_os1_32_sensor">
         <visualize>false</visualize>
-        <update_rate>20</update_rate>
+        <update_rate>20.0</update_rate>
         <ray>
           <scan>

File: urdf/slamtec_rplidar_a2.urdf.xacro (robot description, xacro)
@@ -13,5 +13,5 @@
                        frame_id:=laser
                        model:=A2M12
-                       simulation_engine:=gazebo-classic" >
+                       simulation_engine:=gazebo-classic">
     <xacro:if value="${use_gpu}">
       <xacro:property name="ray_type" value="gpu_ray" />
@@ -32,15 +32,15 @@
     <xacro:if value="${model == 'A2M7'}">
       <xacro:property name="samples" value="1600" />
-      <xacro:property name="max_distance" value="14" />
+      <xacro:property name="max_distance" value="14.0" />
       <xacro:property name="mesh" value="slamtec_rplidar_ax.dae" />
     </xacro:if>
     <xacro:if value="${model == 'A2M8'}">
       <xacro:property name="samples" value="800" />
-      <xacro:property name="max_distance" value="10" />
+      <xacro:property name="max_distance" value="10.0" />
       <xacro:property name="mesh" value="slamtec_rplidar_a2m8.dae" />
     </xacro:if>
     <xacro:if value="${model == 'A2M12'}">
       <xacro:property name="samples" value="1600" />
-      <xacro:property name="max_distance" value="10" />
+      <xacro:property name="max_distance" value="10.0" />
       <xacro:property name="mesh" value="slamtec_rplidar_ax.dae" />
     </xacro:if>
@@ -52,5 +52,5 @@
     <link name="${tf_prefix_ext}slamtec_rplidar_a2_link">
       <visual>
-        <origin xyz="0.0 0.0 0.0" rpy="0.0 0.0 0.0"/>
+        <origin xyz="0.0 0.0 0.0" rpy="0.0 0.0 0.0" />
         <geometry>
           <mesh filename="file://$(find ros_components_description)/meshes/${mesh}" />
@@ -58,5 +58,5 @@
       </visual>
       <collision>
-        <origin xyz="0.0 0.0 ${0.041/2.0}" rpy="0.0 0.0 0.0"/>
+        <origin xyz="0.0 0.0 ${0.041/2.0}" rpy="0.0 0.0 0.0" />
         <geometry>
           <cylinder radius="${0.076/2.0}" length="0.041" />
@@ -72,5 +72,5 @@
     </link>
     <joint name="${tf_prefix_ext}slamtec_rplidar_a2_to_${tf_prefix_ext}${frame_id.rstrip('_link')}_joint" type="fixed">
-      <origin xyz="0 0 0.031" rpy="0.0 0.0 ${pi}" />
+      <origin xyz="0.0 0.0 0.031" rpy="0.0 0.0 ${pi}" />
       <parent link="${tf_prefix_ext}slamtec_rplidar_a2_link" />
       <child link="${tf_prefix_ext}${frame_id}" />
@@ -80,5 +80,5 @@
       <sensor type="${ray_type}" name="${tf_prefix_ext}slamtec_rplidar_a2_sensor">
         <visualize>false</visualize>
-        <update_rate>10</update_rate>
+        <update_rate>10.0</update_rate>
         <ray>
           <scan>
@@ -97,5 +97,5 @@
           <noise>
             <type>gaussian</type>
-            <mean>0</mean>
+            <mean>0.0</mean>
             <stddev>0.001</stddev>
           </noise>

File: urdf/slamtec_rplidar_a3.urdf.xacro (robot description, xacro)
@@ -7,5 +7,5 @@
                        topic:=scan
                        frame_id:=laser
-                       simulation_engine:=gazebo-classic" >
+                       simulation_engine:=gazebo-classic">
     <xacro:if value="${use_gpu}">
       <xacro:property name="ray_type" value="gpu_ray" />
@@ -29,5 +29,5 @@
     <link name="${tf_prefix_ext}slamtec_rplidar_a3_link">
       <visual>
-        <origin xyz="0.0 0.0 0.0" rpy="0.0 0.0 0.0"/>
+        <origin xyz="0.0 0.0 0.0" rpy="0.0 0.0 0.0" />
         <geometry>
           <!-- slamtec_rplidar_ax.dae is used as a shared mesh for A2 and A3 rplidars -->
@@ -36,5 +36,5 @@
       </visual>
       <collision>
-        <origin xyz="0.0 0.0 ${0.041/2.0}" rpy="0.0 0.0 0.0"/>
+        <origin xyz="0.0 0.0 ${0.041/2.0}" rpy="0.0 0.0 0.0" />
         <geometry>
           <cylinder radius="${0.076/2.0}" length="0.041" />
@@ -50,5 +50,5 @@
     </link>
     <joint name="${tf_prefix_ext}slamtec_rplidar_a3_to_${tf_prefix_ext}${frame_id.rstrip('_link')}_joint" type="fixed">
-      <origin xyz="0 0 0.031" rpy="0.0 0.0 ${pi}" />
+      <origin xyz="0.0 0.0 0.031" rpy="0.0 0.0 ${pi}" />
       <parent link="${tf_prefix_ext}slamtec_rplidar_a3_link" />
       <child link="${tf_prefix_ext}${frame_id}" />
@@ -58,5 +58,5 @@
       <sensor type="${ray_type}" name="${tf_prefix_ext}slamtec_rplidar_a3_sensor">
         <visualize>false</visualize>
-        <update_rate>10</update_rate>
+        <update_rate>10.0</update_rate>
         <ray>
           <scan>
@@ -76,5 +76,5 @@
           <noise>
             <type>gaussian</type>
-            <mean>0</mean>
+            <mean>0.0</mean>
             <stddev>0.001</stddev>
           </noise>

File: urdf/slamtec_rplidar_s1.urdf.xacro (robot description, xacro)
@@ -7,5 +7,5 @@
                        topic:=scan
                        frame_id:=laser
-                       simulation_engine:=gazebo-classic" >
+                       simulation_engine:=gazebo-classic">
     <xacro:if value="${use_gpu}">
       <xacro:property name="ray_type" value="gpu_ray" />
@@ -29,5 +29,5 @@
     <link name="${tf_prefix_ext}slamtec_rplidar_s1_link">
       <visual>
-        <origin xyz="0.0 0.0 0.0" rpy="0.0 0.0 0.0"/>
+        <origin xyz="0.0 0.0 0.0" rpy="0.0 0.0 0.0" />
         <geometry>
           <mesh filename="file://$(find ros_components_description)/meshes/slamtec_rplidar_s1.dae" />
@@ -36,5 +36,5 @@
       <!-- spinning head collision -->
       <collision>
-        <origin xyz="0.0 0.0 ${0.051/2.0}" rpy="0.0 0.0 0.0"/>
+        <origin xyz="0.0 0.0 ${0.051/2.0}" rpy="0.0 0.0 0.0" />
         <geometry>
           <cylinder radius="${0.0555/2.0}" length="0.051" />
@@ -43,5 +43,5 @@
       <!-- base collision -->
       <collision>
-        <origin xyz="0.0 0.0 ${0.0195/2.0}" rpy="0.0 0.0 0.0"/>
+        <origin xyz="0.0 0.0 ${0.0195/2.0}" rpy="0.0 0.0 0.0" />
         <geometry>
           <box size="0.0555 0.0555 0.0195" />
@@ -57,5 +57,5 @@
     </link>
     <joint name="${tf_prefix_ext}slamtec_rplidar_s1_to_${tf_prefix_ext}${frame_id.rstrip('_link')}_joint" type="fixed">
-      <origin xyz="0 0 0.04" rpy="0.0 0.0 ${pi}" />
+      <origin xyz="0.0 0.0 0.04" rpy="0.0 0.0 ${pi}" />
       <parent link="${tf_prefix_ext}slamtec_rplidar_s1_link" />
       <child link="${tf_prefix_ext}${frame_id}" />
@@ -64,7 +64,6 @@
     <gazebo reference="${tf_prefix_ext}${frame_id}">
       <sensor type="${ray_type}" name="${tf_prefix_ext}slamtec_rplidar_s1_sensor">
-        <pose>0 0 0.04 0 0 0</pose>
         <visualize>false</visualize>
-        <update_rate>10</update_rate>
+        <update_rate>10.0</update_rate>
         <ray>
           <scan>
@@ -83,5 +82,5 @@
           <noise>
             <type>gaussian</type>
-            <mean>0</mean>
+            <mean>0.0</mean>
             <stddev>0.001</stddev>
           </noise>

File: urdf/velodyne_puck.urdf.xacro (robot description, xacro)
@@ -7,5 +7,5 @@
                        topic:=scan
                        frame_id:=velodyne
-                       simulation_engine:=gazebo-classic" >
+                       simulation_engine:=gazebo-classic">
     <xacro:if value="${use_gpu}">
       <xacro:property name="ray_type" value="gpu_ray" />
@@ -29,5 +29,5 @@
     <link name="${tf_prefix_ext}velodyne_puck_link">
       <visual>
-        <origin xyz="0.0 0.0 0.0" rpy="0.0 0.0 0.0"/>
+        <origin xyz="0.0 0.0 0.0" rpy="0.0 0.0 0.0" />
         <geometry>
           <mesh filename="file://$(find ros_components_description)/meshes/velodyne_puck.dae" />
@@ -35,5 +35,5 @@
       </visual>
       <collision>
-        <origin xyz="0.0 0.0 ${0.072/2.0}" rpy="0.0 0.0 0.0"/>
+        <origin xyz="0.0 0.0 ${0.072/2.0}" rpy="0.0 0.0 0.0" />
         <geometry>
           <cylinder radius="${0.103/2.0}" length="0.072" />
@@ -57,5 +57,5 @@
       <sensor type="${ray_type}" name="${tf_prefix_ext}velodyne_puck_sensor">
         <visualize>false</visualize>
-        <update_rate>10</update_rate>
+        <update_rate>10.0</update_rate>
         <ray>
           <scan>

Commit message: Update floats

File: urdf/orbbec_astra.urdf.xacro (robot description, xacro)
@@ -48,5 +48,5 @@
     </link>
     <joint name="${tf_prefix_ext}orbbec_astra_to_${tf_prefix_ext}${frame_id.rstrip('_link')}_joint" type="fixed">
-      <origin xyz="0.01 0.0 0.035" rpy="${-pi/2} 0.0 ${-pi/2}" />
+      <origin xyz="0.01 0.0 0.035" rpy="${-pi/2.0} 0.0 ${-pi/2.0}" />
       <parent link="${tf_prefix_ext}orbbec_astra_link" />
       <child link="${tf_prefix_ext}${frame_id}" />
@@ -57,5 +57,5 @@
         <always_on>true</always_on>
         <camera>
-          <horizontal_fov>${60/180*pi}</horizontal_fov>
+          <horizontal_fov>${60.0/180.0*pi}</horizontal_fov>
           <image>
             <format>R8G8B8</format>

Commit message: Fix floating point precision

File: urdf/orbbec_astra.urdf.xacro (robot description, xacro)
@@ -48,5 +48,5 @@
     </link>
     <joint name="${tf_prefix_ext}orbbec_astra_to_${tf_prefix_ext}${frame_id.rstrip('_link')}_joint" type="fixed">
-      <origin xyz="0.01 0.0 0.035" rpy="${-pi/2} 0.0 ${-pi/2}" />
+      <origin xyz="0.01 0.0 0.035" rpy="${-pi/2.0} 0.0 ${-pi/2.0}" />
       <parent link="${tf_prefix_ext}orbbec_astra_link" />
       <child link="${tf_prefix_ext}${frame_id}" />
@@ -58,5 +58,5 @@
         <update_rate>20.0</update_rate>
         <camera name="${tf_prefix_ext}camera">
-          <horizontal_fov>${60/180*pi}</horizontal_fov>
+          <horizontal_fov>${60.0/180.0*pi}</horizontal_fov>
           <image>
             <format>R8G8B8</format>

File: urdf/ouster_os1_32.urdf.xacro (robot description, xacro)
@@ -68,6 +68,6 @@
               <samples>32</samples>
               <resolution>1</resolution>
-              <min_angle>-${22.5/180*pi}</min_angle>
-              <max_angle>${22.5/180*pi}</max_angle>
+              <min_angle>-${22.5/180.0*pi}</min_angle>
+              <max_angle>${22.5/180.0*pi}</max_angle>
             </vertical>
           </scan>

File: urdf/velodyne_puck.urdf.xacro (robot description, xacro)
@@ -68,6 +68,6 @@
               <samples>16</samples>
               <resolution>1</resolution>
-              <min_angle>-${15/180*pi}</min_angle>
-              <max_angle>${15/180*pi}</max_angle>
+              <min_angle>-${15.0/180.0*pi}</min_angle>
+              <max_angle>${15.0/180.0*pi}</max_angle>
             </vertical>
           </scan>

Commit message: Fix formatting (#17)
* Fix formatting

* Update floats

* Fix floating points

File: urdf/orbbec_astra.urdf.xacro (robot description, xacro)
@@ -20,5 +20,5 @@
     <link name="${tf_prefix_ext}orbbec_astra_link">
       <visual>
-        <origin xyz="0.0 0.0 0.0" rpy="0.0 0.0 0.0"/>
+        <origin xyz="0.0 0.0 0.0" rpy="0.0 0.0 0.0" />
         <geometry>
           <mesh filename="file://$(find ros_components_description)/meshes/orbbec_astra.dae" />
@@ -27,5 +27,5 @@
       <!-- camera module collision -->
       <collision>
-        <origin xyz="${0.0225-0.04/2.0} 0.0 ${0.019+0.03/2.0}" rpy="0.0 0.0 0.0"/>
+        <origin xyz="${0.0225-0.04/2.0} 0.0 ${0.019+0.03/2.0}" rpy="0.0 0.0 0.0" />
         <geometry>
           <box size="0.04 0.165 0.03" />
@@ -34,5 +34,5 @@
       <!-- mounting base model collision -->
       <collision>
-        <origin xyz="${0.0235-0.06/2.0} 0.0 ${0.019/2.0}" rpy="0.0 0.0 0.0"/>
+        <origin xyz="${0.0235-0.06/2.0} 0.0 ${0.019/2.0}" rpy="0.0 0.0 0.0" />
         <geometry>
           <box size="0.06 0.06 0.019" />
@@ -48,5 +48,5 @@
     </link>
     <joint name="${tf_prefix_ext}orbbec_astra_to_${tf_prefix_ext}${frame_id.rstrip('_link')}_joint" type="fixed">
-      <origin xyz="0.01 0 0.035" rpy="${-pi/2} 0 ${-pi/2}" />
+      <origin xyz="0.01 0.0 0.035" rpy="${-pi/2.0} 0.0 ${-pi/2.0}" />
       <parent link="${tf_prefix_ext}orbbec_astra_link" />
       <child link="${tf_prefix_ext}${frame_id}" />
@@ -55,8 +55,7 @@
     <gazebo reference="${tf_prefix_ext}orbbec_astra_link">
       <sensor type="depth" name="${tf_prefix_ext}orbbec_astra_camera">
-        <always_on>1</always_on>
-        <visualize>true</visualize>
+        <always_on>true</always_on>
         <camera>
-          <horizontal_fov>${60/180*pi}</horizontal_fov>
+          <horizontal_fov>${60.0/180.0*pi}</horizontal_fov>
           <image>
             <format>R8G8B8</format>

File: urdf/ouster_os1_32.urdf.xacro (robot description, xacro)
@@ -7,5 +7,5 @@
                        topic:=os_lidar
                        frame_id:=os_lidar
-                       simulation_engine:=gazebo-classic" >
+                       simulation_engine:=gazebo-classic">
     <xacro:if value="${use_gpu}">
       <xacro:property name="ray_type" value="gpu_ray" />
@@ -29,5 +29,5 @@
     <link name="${tf_prefix_ext}ouster_os1_32_link">
       <visual>
-        <origin xyz="0.0 0.0 0.0" rpy="0.0 0.0 0.0"/>
+        <origin xyz="0.0 0.0 0.0" rpy="0.0 0.0 0.0" />
         <geometry>
           <mesh filename="file://$(find ros_components_description)/meshes/ouster_os1_32.dae" />
@@ -35,5 +35,5 @@
       </visual>
       <collision>
-        <origin xyz="0.0 0.0 ${0.072/2.0}" rpy="0.0 0.0 0.0"/>
+        <origin xyz="0.0 0.0 ${0.072/2.0}" rpy="0.0 0.0 0.0" />
         <geometry>
           <cylinder radius="${0.085/2.0}" length="0.073" />
@@ -57,5 +57,5 @@
       <sensor type="${ray_type}" name="${tf_prefix_ext}ouster_os1_32_sensor">
         <visualize>false</visualize>
-        <update_rate>20</update_rate>
+        <update_rate>20.0</update_rate>
         <ray>
           <scan>
@@ -69,6 +69,6 @@
               <samples>32</samples>
               <resolution>1</resolution>
-              <min_angle>-${22.5/180*pi}</min_angle>
-              <max_angle>${22.5/180*pi}</max_angle>
+              <min_angle>-${22.5/180.0*pi}</min_angle>
+              <max_angle>${22.5/180.0*pi}</max_angle>
             </vertical>
           </scan>

File: urdf/velodyne_puck.urdf.xacro (robot description, xacro)
@@ -7,5 +7,5 @@
                        topic:=scan
                        frame_id:=velodyne
-                       simulation_engine:=gazebo-classic" >
+                       simulation_engine:=gazebo-classic">
     <xacro:if value="${use_gpu}">
       <xacro:property name="ray_type" value="gpu_ray" />
@@ -29,5 +29,5 @@
     <link name="${tf_prefix_ext}velodyne_puck_link">
       <visual>
-        <origin xyz="0.0 0.0 0.0" rpy="0.0 0.0 0.0"/>
+        <origin xyz="0.0 0.0 0.0" rpy="0.0 0.0 0.0" />
         <geometry>
           <mesh filename="file://$(find ros_components_description)/meshes/velodyne_puck.dae" />
@@ -35,5 +35,5 @@
       </visual>
       <collision>
-        <origin xyz="0.0 0.0 ${0.072/2.0}" rpy="0.0 0.0 0.0"/>
+        <origin xyz="0.0 0.0 ${0.072/2.0}" rpy="0.0 0.0 0.0" />
         <geometry>
           <cylinder radius="${0.103/2.0}" length="0.072" />
@@ -57,5 +57,5 @@
       <sensor type="${ray_type}" name="${tf_prefix_ext}velodyne_puck_sensor">
         <visualize>false</visualize>
-        <update_rate>10</update_rate>
+        <update_rate>10.0</update_rate>
         <ray>
           <scan>
@@ -69,6 +69,6 @@
               <samples>16</samples>
               <resolution>1</resolution>
-              <min_angle>-${15/180*pi}</min_angle>
-              <max_angle>${15/180*pi}</max_angle>
+              <min_angle>-${15.0/180.0*pi}</min_angle>
+              <max_angle>${15.0/180.0*pi}</max_angle>
             </vertical>
           </scan>
