Commit message: Fix lidars and astra to work with gz-ign Fortress

File: urdf/orbbec_astra.urdf.xacro (robot description, xacro)
@@ -4,5 +4,5 @@
                params="parent_link xyz rpy
                        tf_prefix:=None
-                       topic:=camera/depth/points
+                       topic:=camera
                        frame_id:=depth
                        simulation_engine:=gazebo-classic">
@@ -53,33 +53,63 @@
     </joint>
     <link name="${tf_prefix_ext}${frame_id}" />
-    <gazebo reference="${tf_prefix_ext}orbbec_astra_link">
-      <sensor type="depth" name="${tf_prefix_ext}orbbec_astra_camera">
-        <always_on>true</always_on>
-        <update_rate>20.0</update_rate>
-        <camera name="${tf_prefix_ext}camera">
-          <horizontal_fov>${60.0/180.0*pi}</horizontal_fov>
-          <image>
-            <format>R8G8B8</format>
-            <width>640</width>
-            <height>480</height>
-          </image>
-        </camera>
-        <plugin name="${tf_prefix_ext}orbbec_astra_camera" filename="libgazebo_ros_camera.so">
-          <ros>
-            <namespace>orbbec_astra_camera</namespace>
-            <remapping>custom_camera/image_raw:=rgb/image_raw</remapping>
-            <remapping>custom_camera/image_depth:=depth/image_raw</remapping>
-            <remapping>custom_camera/camera_info:=rgb/camera_info</remapping>
-            <remapping>custom_camera/camera_info_depth:=depth/camera_info</remapping>
-            <remapping>custom_camera/points:=depth/points</remapping>
-          </ros>
-          <camera_name>${tf_prefix_ext}camera</camera_name>
-          <frame_name>${tf_prefix_ext}${frame_id}</frame_name>
-          <hack_baseline>0.07</hack_baseline>
-          <min_depth>0.6</min_depth>
-          <max_depth>8.0</max_depth>
+    <xacro:if value="${simulation_engine == 'ignition-gazebo'}">
+      <gazebo reference="${tf_prefix_ext}orbbec_astra_link">
+        <sensor type="rgbd_camera" name="${tf_prefix_ext}orbbec_astra_camera">
+          <always_on>true</always_on>
+          <update_rate>20.0</update_rate>
+          <topic>${topic}</topic>
+          <!-- <frame_id>${tf_prefix_ext}${frame_id}</frame_id> -->
+          <optical_frame_id>${tf_prefix_ext}${frame_id}</optical_frame_id>
+          <ignition_frame_id>${tf_prefix_ext}${frame_id}</ignition_frame_id>
+          <camera name="${tf_prefix_ext}camera">
+            <horizontal_fov>${60.0/180.0*pi}</horizontal_fov>
+            <image>
+              <width>640</width>
+              <height>480</height>
+            </image>
+            <clip>
+              <near>0.6</near>
+              <far>8.0</far>
+            </clip>
+          </camera>
+        </sensor>
+      </gazebo>
+      <!-- <gazebo>
+        <plugin filename="libignition-gazebo-sensors-system.so" name="ignition::gazebo::systems::Sensors">
+          <render_engine>ogre2</render_engine>
         </plugin>
-      </sensor>
-    </gazebo>
+      </gazebo>  -->
+    </xacro:if>
+    <xacro:if value="${simulation_engine == 'gazebo-classic'}">
+      <gazebo reference="${tf_prefix_ext}orbbec_astra_link">
+        <sensor type="depth" name="${tf_prefix_ext}orbbec_astra_camera">
+          <always_on>true</always_on>
+          <update_rate>20.0</update_rate>
+          <camera name="${tf_prefix_ext}camera">
+            <horizontal_fov>${60.0/180.0*pi}</horizontal_fov>
+            <image>
+              <format>R8G8B8</format>
+              <width>640</width>
+              <height>480</height>
+            </image>
+          </camera>
+          <plugin name="${tf_prefix_ext}orbbec_astra_camera" filename="libgazebo_ros_camera.so">
+            <ros>
+              <namespace>orbbec_astra_camera</namespace>
+              <remapping>custom_camera/image_raw:=rgb/image_raw</remapping>
+              <remapping>custom_camera/image_depth:=depth/image_raw</remapping>
+              <remapping>custom_camera/camera_info:=rgb/camera_info</remapping>
+              <remapping>custom_camera/camera_info_depth:=depth/camera_info</remapping>
+              <remapping>custom_camera/points:=depth/points</remapping>
+            </ros>
+            <camera_name>${tf_prefix_ext}camera</camera_name>
+            <frame_name>${tf_prefix_ext}${frame_id}</frame_name>
+            <hack_baseline>0.07</hack_baseline>
+            <min_depth>0.6</min_depth>
+            <max_depth>8.0</max_depth>
+          </plugin>
+        </sensor>
+      </gazebo>
+    </xacro:if>
   </xacro:macro>
 </robot>

File: urdf/slamtec_rplidar_a2.urdf.xacro (robot description, xacro)
@@ -15,8 +15,19 @@
                        simulation_engine:=gazebo-classic">
     <xacro:if value="${use_gpu}">
-      <xacro:property name="ray_type" value="gpu_ray" />
+      <xacro:if value="${simulation_engine == 'gazebo-classic'}">
+        <xacro:property name="ray_type" value="gpu_ray" />
+      </xacro:if>
+      <xacro:if value="${simulation_engine == 'ignition-gazebo'}">
+        <xacro:property name="ray_type" value="gpu_lidar" />
+      </xacro:if>
     </xacro:if>
     <xacro:unless value="${use_gpu}">
-      <xacro:property name="ray_type" value="ray" />
+      <xacro:if value="${simulation_engine == 'gazebo-classic'}">
+        <xacro:property name="ray_type" value="ray" />
+      </xacro:if>
+      <xacro:if value="${simulation_engine == 'ignition-gazebo'}">
+        <!-- this is king of awkward, but it seems like cpu lidar does not work -->
+        <xacro:property name="ray_type" value="gpu_lidar" />
+      </xacro:if>
     </xacro:unless>
     <xacro:if value="${tf_prefix == 'None'}">
@@ -78,5 +89,5 @@
       <gazebo reference="${tf_prefix_ext}${frame_id}">
         <sensor type="${ray_type}" name="${tf_prefix_ext}rplidar_a2_sensor">
-          <topic>scan</topic>
+          <topic>${topic}</topic>
           <frame_id>${tf_prefix_ext}${frame_id}</frame_id>
           <ignition_frame_id>${tf_prefix_ext}${frame_id}</ignition_frame_id>

File: urdf/slamtec_rplidar_a3.urdf.xacro (robot description, xacro)
@@ -9,8 +9,19 @@
                        simulation_engine:=gazebo-classic">
     <xacro:if value="${use_gpu}">
-      <xacro:property name="ray_type" value="gpu_ray" />
+      <xacro:if value="${simulation_engine == 'gazebo-classic'}">
+        <xacro:property name="ray_type" value="gpu_ray" />
+      </xacro:if>
+      <xacro:if value="${simulation_engine == 'ignition-gazebo'}">
+        <xacro:property name="ray_type" value="gpu_lidar" />
+      </xacro:if>
     </xacro:if>
     <xacro:unless value="${use_gpu}">
-      <xacro:property name="ray_type" value="ray" />
+      <xacro:if value="${simulation_engine == 'gazebo-classic'}">
+        <xacro:property name="ray_type" value="ray" />
+      </xacro:if>
+      <xacro:if value="${simulation_engine == 'ignition-gazebo'}">
+        <!-- this is king of awkward, but it seems like cpu lidar does not work -->
+        <xacro:property name="ray_type" value="gpu_lidar" />
+      </xacro:if>
     </xacro:unless>
     <xacro:if value="${tf_prefix == 'None'}">
@@ -56,5 +67,5 @@
       <gazebo reference="${tf_prefix_ext}${frame_id}">
         <sensor type="${ray_type}" name="${tf_prefix_ext}rplidar_a3_sensor">
-          <topic>scan</topic>
+          <topic>${topic}</topic>
           <frame_id>${tf_prefix_ext}${frame_id}</frame_id>
           <ignition_frame_id>${tf_prefix_ext}${frame_id}</ignition_frame_id>

File: urdf/slamtec_rplidar_s1.urdf.xacro (robot description, xacro)
@@ -9,8 +9,19 @@
                        simulation_engine:=gazebo-classic">
     <xacro:if value="${use_gpu}">
-      <xacro:property name="ray_type" value="gpu_ray" />
+      <xacro:if value="${simulation_engine == 'gazebo-classic'}">
+        <xacro:property name="ray_type" value="gpu_ray" />
+      </xacro:if>
+      <xacro:if value="${simulation_engine == 'ignition-gazebo'}">
+        <xacro:property name="ray_type" value="gpu_lidar" />
+      </xacro:if>
     </xacro:if>
     <xacro:unless value="${use_gpu}">
-      <xacro:property name="ray_type" value="ray" />
+      <xacro:if value="${simulation_engine == 'gazebo-classic'}">
+        <xacro:property name="ray_type" value="ray" />
+      </xacro:if>
+      <xacro:if value="${simulation_engine == 'ignition-gazebo'}">
+        <!-- this is king of awkward, but it seems like cpu lidar does not work -->
+        <xacro:property name="ray_type" value="gpu_lidar" />
+      </xacro:if>
     </xacro:unless>
     <xacro:if value="${tf_prefix == 'None'}">
@@ -63,5 +74,5 @@
       <gazebo reference="${tf_prefix_ext}${frame_id}">
         <sensor type="${ray_type}" name="${tf_prefix_ext}rplidar_s1_sensor">
-          <topic>scan</topic>
+          <topic>${topic}</topic>
           <frame_id>${tf_prefix_ext}${frame_id}</frame_id>
           <ignition_frame_id>${tf_prefix_ext}${frame_id}</ignition_frame_id>
@@ -70,5 +81,5 @@
             <scan>
               <horizontal>
-                <samples>9200</samples>
+                <samples>920</samples>
                 <resolution>1</resolution>
                 <min_angle>-${pi}</min_angle>
@@ -92,8 +103,8 @@
       </gazebo>
       <gazebo>
-          <plugin filename="libignition-gazebo-sensors-system.so" name="ignition::gazebo::systems::Sensors">
-            <render_engine>ogre2</render_engine>
-          </plugin>
-        </gazebo>
+        <plugin filename="libignition-gazebo-sensors-system.so" name="ignition::gazebo::systems::Sensors">
+          <render_engine>ogre2</render_engine>
+        </plugin>
+      </gazebo>
     </xacro:if>
     <xacro:if value="${simulation_engine == 'gazebo-classic'}">

Commit message: unify astra description with real camera
Signed-off-by: Jakub Delicat <jakub.delicat@husarion.com>

File: urdf/orbbec_astra.urdf.xacro (robot description, xacro)
@@ -4,7 +4,7 @@
                params="parent_link xyz rpy
                        tf_prefix:=None
-                       topic:=camera
-                       frame_id:=depth
-                       simulation_engine:=gazebo-classic">
+                       camera_name:=camera
+                       simulation_engine:=gazebo-classic
+                       use_sim:=false">
     <xacro:if value="${tf_prefix == 'None'}">
       <xacro:property name="tf_prefix_ext" value="" />
@@ -13,10 +13,10 @@
       <xacro:property name="tf_prefix_ext" value="${tf_prefix}_" />
     </xacro:unless>
-    <joint name="${parent_link.rstrip('_link')}_to_${tf_prefix_ext}orbbec_astra_joint" type="fixed">
+    <joint name="${parent_link.rstrip('_link')}_to_${tf_prefix_ext}${camera_name}_orbbec_astra_joint" type="fixed">
       <origin xyz="${xyz}" rpy="${rpy}" />
       <parent link="${parent_link}" />
-      <child link="${tf_prefix_ext}orbbec_astra_link" />
+      <child link="${tf_prefix_ext}${camera_name}_orbbec_astra_link" />
     </joint>
-    <link name="${tf_prefix_ext}orbbec_astra_link">
+    <link name="${tf_prefix_ext}${camera_name}_orbbec_astra_link">
       <visual>
         <origin xyz="0.0 0.0 0.0" rpy="0.0 0.0 0.0" />
@@ -47,19 +47,39 @@
       </inertial>
     </link>
-    <joint name="${tf_prefix_ext}orbbec_astra_to_${tf_prefix_ext}${frame_id.rstrip('_link')}_joint" type="fixed">
-      <origin xyz="0.01 0.0 0.035" rpy="${-pi/2.0} 0.0 ${-pi/2.0}" />
-      <parent link="${tf_prefix_ext}orbbec_astra_link" />
-      <child link="${tf_prefix_ext}${frame_id}" />
-    </joint>
-    <link name="${tf_prefix_ext}${frame_id}" />
+    <xacro:if value="$(arg use_sim)">
+      <joint name="${parent_link.rstrip('_link')}_to_${tf_prefix_ext}${camera_name}_color_joint" type="fixed">
+        <origin xyz="-0.002 0.0125 0.03325" rpy="-0.003 0.0 -0.003" />
+        <parent link="${parent_link}" />
+        <child link="${tf_prefix_ext}${camera_name}_color_frame" />
+      </joint>
+      <link name="${tf_prefix_ext}${camera_name}_depth_frame" />
+      <joint name="${parent_link.rstrip('_link')}_to_${tf_prefix_ext}${camera_name}_depth_joint" type="fixed">
+        <origin xyz="0.0 0.0 0.03325" rpy="0.0 0.0 0.0" />
+        <parent link="${parent_link}" />
+        <child link="${tf_prefix_ext}${camera_name}_depth_frame" />
+      </joint>
+      <link name="${tf_prefix_ext}${camera_name}_color_frame" />
+      <joint name="${tf_prefix_ext}${camera_name}_color_to_${tf_prefix_ext}${camera_name}_color_optical_joint" type="fixed">
+        <origin xyz="0.0 0.0 0.0" rpy="${-pi/2} 0.0 ${-pi/2}" />
+        <parent link="${tf_prefix_ext}${camera_name}_color_frame" />
+        <child link="${tf_prefix_ext}${camera_name}_color_optical_frame" />
+      </joint>
+      <link name="${tf_prefix_ext}${camera_name}_depth_optical_frame" />
+      <joint name="${tf_prefix_ext}${camera_name}_depth_to_${tf_prefix_ext}${camera_name}_depth_optical_joint" type="fixed">
+        <origin xyz="0.1 0.0 0.0" rpy="${-pi/2} 0.0 ${-pi/2}" />
+        <parent link="${tf_prefix_ext}${camera_name}_depth_frame" />
+        <child link="${tf_prefix_ext}${camera_name}_depth_optical_frame" />
+      </joint>
+      <link name="${tf_prefix_ext}${camera_name}_color_optical_frame" />
+    </xacro:if>
     <xacro:if value="${simulation_engine == 'ignition-gazebo'}">
-      <gazebo reference="${tf_prefix_ext}orbbec_astra_link">
-        <sensor type="rgbd_camera" name="${tf_prefix_ext}orbbec_astra_camera">
+      <gazebo reference="${tf_prefix_ext}${camera_name}_orbbec_astra_link">
+        <sensor type="rgbd_camera" name="${tf_prefix_ext}${camera_name}_orbbec_astra_camera">
           <always_on>true</always_on>
           <update_rate>20.0</update_rate>
-          <topic>${topic}</topic>
-          <!-- <frame_id>${tf_prefix_ext}${frame_id}</frame_id> -->
-          <optical_frame_id>${tf_prefix_ext}${frame_id}</optical_frame_id>
-          <ignition_frame_id>${tf_prefix_ext}${frame_id}</ignition_frame_id>
+          <topic>${camera_name}</topic>
+          <!-- It is not possible to split the frame of the color and the depth stream.
+               The frame of color stream should be ${tf_prefix_ext}${camera_name}_color_optical_frame -->
+          <ignition_frame_id>${tf_prefix_ext}${camera_name}_depth_optical_frame</ignition_frame_id>
           <camera name="${tf_prefix_ext}camera">
             <horizontal_fov>${60.0/180.0*pi}</horizontal_fov>

Commit message: apply transform for real astra
Signed-off-by: Jakub Delicat <jakub.delicat@husarion.com>

File: urdf/orbbec_astra.urdf.xacro (robot description, xacro)
@@ -47,30 +47,28 @@
       </inertial>
     </link>
-    <xacro:if value="$(arg use_sim)">
-      <joint name="${parent_link.rstrip('_link')}_to_${tf_prefix_ext}${camera_name}_color_joint" type="fixed">
-        <origin xyz="-0.002 0.0125 0.03325" rpy="-0.003 0.0 -0.003" />
-        <parent link="${parent_link}" />
-        <child link="${tf_prefix_ext}${camera_name}_color_frame" />
-      </joint>
-      <link name="${tf_prefix_ext}${camera_name}_depth_frame" />
-      <joint name="${parent_link.rstrip('_link')}_to_${tf_prefix_ext}${camera_name}_depth_joint" type="fixed">
-        <origin xyz="0.0 0.0 0.03325" rpy="0.0 0.0 0.0" />
-        <parent link="${parent_link}" />
-        <child link="${tf_prefix_ext}${camera_name}_depth_frame" />
-      </joint>
-      <link name="${tf_prefix_ext}${camera_name}_color_frame" />
-      <joint name="${tf_prefix_ext}${camera_name}_color_to_${tf_prefix_ext}${camera_name}_color_optical_joint" type="fixed">
-        <origin xyz="0.0 0.0 0.0" rpy="${-pi/2} 0.0 ${-pi/2}" />
-        <parent link="${tf_prefix_ext}${camera_name}_color_frame" />
-        <child link="${tf_prefix_ext}${camera_name}_color_optical_frame" />
-      </joint>
-      <link name="${tf_prefix_ext}${camera_name}_depth_optical_frame" />
-      <joint name="${tf_prefix_ext}${camera_name}_depth_to_${tf_prefix_ext}${camera_name}_depth_optical_joint" type="fixed">
-        <origin xyz="0.1 0.0 0.0" rpy="${-pi/2} 0.0 ${-pi/2}" />
-        <parent link="${tf_prefix_ext}${camera_name}_depth_frame" />
-        <child link="${tf_prefix_ext}${camera_name}_depth_optical_frame" />
-      </joint>
-      <link name="${tf_prefix_ext}${camera_name}_color_optical_frame" />
-    </xacro:if>
+    <joint name="${parent_link.rstrip('_link')}_to_${tf_prefix_ext}${camera_name}_color_joint" type="fixed">
+      <origin xyz="-0.002 0.0125 0.03325" rpy="-0.003 0.0 -0.003" />
+      <parent link="${parent_link}" />
+      <child link="${tf_prefix_ext}${camera_name}_color_frame" />
+    </joint>
+    <link name="${tf_prefix_ext}${camera_name}_depth_frame" />
+    <joint name="${parent_link.rstrip('_link')}_to_${tf_prefix_ext}${camera_name}_depth_joint" type="fixed">
+      <origin xyz="0.0 0.0 0.03325" rpy="0.0 0.0 0.0" />
+      <parent link="${parent_link}" />
+      <child link="${tf_prefix_ext}${camera_name}_depth_frame" />
+    </joint>
+    <link name="${tf_prefix_ext}${camera_name}_color_frame" />
+    <joint name="${tf_prefix_ext}${camera_name}_color_to_${tf_prefix_ext}${camera_name}_color_optical_joint" type="fixed">
+      <origin xyz="0.0 0.0 0.0" rpy="${-pi/2} 0.0 ${-pi/2}" />
+      <parent link="${tf_prefix_ext}${camera_name}_color_frame" />
+      <child link="${tf_prefix_ext}${camera_name}_color_optical_frame" />
+    </joint>
+    <link name="${tf_prefix_ext}${camera_name}_depth_optical_frame" />
+    <joint name="${tf_prefix_ext}${camera_name}_depth_to_${tf_prefix_ext}${camera_name}_depth_optical_joint" type="fixed">
+      <origin xyz="0.0 0.0 0.0" rpy="${-pi/2} 0.0 ${-pi/2}" />
+      <parent link="${tf_prefix_ext}${camera_name}_depth_frame" />
+      <child link="${tf_prefix_ext}${camera_name}_depth_optical_frame" />
+    </joint>
+    <link name="${tf_prefix_ext}${camera_name}_color_optical_frame" />
     <xacro:if value="${simulation_engine == 'ignition-gazebo'}">
       <gazebo reference="${tf_prefix_ext}${camera_name}_orbbec_astra_link">
