Commit message: add s2 and s3

File: urdf/orbbec_astra.urdf.xacro (robot description, xacro)
@@ -2,9 +2,9 @@
 <robot name="orbbec_astra" xmlns:xacro="http://www.ros.org/wiki/xacro">
   <xacro:macro name="orbbec_astra"
-               params="parent_link xyz rpy
-                       tf_prefix:=None
-                       name:=camera
-                       topic:=camera
-                       simulation_engine:=ignition-gazebo">
+    params="parent_link xyz rpy
+            tf_prefix:=None
+            name:=camera
+            topic:=camera
+            simulation_engine:=ignition-gazebo">
     <xacro:if value="${tf_prefix == 'None'}">
       <xacro:property name="prefix" value="" />

File: urdf/slamtec_rplidar_s2.urdf.xacro (robot description, xacro)
@@ -2,10 +2,11 @@
 <robot xmlns:xacro="http://www.ros.org/wiki/xacro">
   <xacro:macro name="slamtec_rplidar_s2"
-               params="parent_link xyz rpy
-                       use_gpu:=false
-                       tf_prefix:=None
-                       topic:=scan
-                       frame_id:=laser
-                       simulation_engine:=gazebo-classic">
+    params="parent_link xyz rpy
+            use_gpu:=false
+            tf_prefix:=None
+            name:=slamtec_rplidar_s2
+            topic:=scan
+            frame_id:=laser
+            simulation_engine:=ignition-gazebo">
     <xacro:if value="${use_gpu}">
       <xacro:if value="${simulation_engine == 'gazebo-classic'}">
@@ -32,10 +33,10 @@
       <xacro:property name="prefix" value="${tf_prefix}_" />
     </xacro:unless>
-    <joint name="${parent_link.rstrip('_link')}_to_${prefix}slamtec_rplidar_s2_joint" type="fixed">
+    <joint name="${parent_link.rstrip('_link')}_to_${prefix}${name}_joint" type="fixed">
       <origin xyz="${xyz}" rpy="${rpy}" />
       <parent link="${parent_link}" />
-      <child link="${prefix}slamtec_rplidar_s2_link" />
+      <child link="${prefix}${name}_link" />
     </joint>
-    <link name="${prefix}slamtec_rplidar_s2_link">
+    <link name="${prefix}${name}_link">
       <visual>
         <origin xyz="0.0 0.0 0.0" rpy="0.0 0.0 0.0" />
@@ -59,7 +60,7 @@
       </inertial>
     </link>
-    <joint name="${prefix}slamtec_rplidar_s2_to_${prefix}${frame_id.rstrip('_link')}_joint" type="fixed">
+    <joint name="${prefix}${name}_to_${prefix}${frame_id.rstrip('_link')}_joint" type="fixed">
       <origin xyz="0.0 0.0 0.0285" rpy="0.0 0.0 ${pi}" />
-      <parent link="${prefix}slamtec_rplidar_s2_link" />
+      <parent link="${prefix}${name}_link" />
       <child link="${prefix}${frame_id}" />
     </joint>
@@ -104,5 +105,5 @@
     <xacro:if value="${simulation_engine == 'gazebo-classic'}">
       <gazebo reference="${prefix}${frame_id}">
-        <sensor type="${ray_type}" name="${prefix}slamtec_rplidar_s2_sensor">
+        <sensor type="${ray_type}" name="${prefix}${name}_sensor">
           <visualize>false</visualize>
           <ray>

File: urdf/slamtec_rplidar_s3.urdf.xacro (robot description, xacro)
@@ -2,10 +2,11 @@
 <robot xmlns:xacro="http://www.ros.org/wiki/xacro">
   <xacro:macro name="slamtec_rplidar_s3"
-               params="parent_link xyz rpy
-                       use_gpu:=false
-                       tf_prefix:=None
-                       topic:=scan
-                       frame_id:=laser
-                       simulation_engine:=gazebo-classic">
+    params="parent_link xyz rpy
+            use_gpu:=false
+            tf_prefix:=None
+            name:=slamtec_rplidar_s3
+            topic:=scan
+            frame_id:=laser
+            simulation_engine:=ignition-gazebo">
     <xacro:if value="${use_gpu}">
       <xacro:if value="${simulation_engine == 'gazebo-classic'}">
@@ -32,10 +33,10 @@
       <xacro:property name="prefix" value="${tf_prefix}_" />
     </xacro:unless>
-    <joint name="${parent_link.rstrip('_link')}_to_${prefix}slamtec_rplidar_s3_joint" type="fixed">
+    <joint name="${parent_link.rstrip('_link')}_to_${prefix}${name}_joint" type="fixed">
       <origin xyz="${xyz}" rpy="${rpy}" />
       <parent link="${parent_link}" />
-      <child link="${prefix}slamtec_rplidar_s3_link" />
+      <child link="${prefix}${name}_link" />
     </joint>
-    <link name="${prefix}slamtec_rplidar_s3_link">
+    <link name="${prefix}${name}_link">
       <visual>
         <origin xyz="0.0 0.0 0.0" rpy="0.0 0.0 0.0" />
@@ -59,7 +60,7 @@
       </inertial>
     </link>
-    <joint name="${prefix}slamtec_rplidar_s3_to_${prefix}${frame_id.rstrip('_link')}_joint" type="fixed">
+    <joint name="${prefix}${name}_to_${prefix}${frame_id.rstrip('_link')}_joint" type="fixed">
       <origin xyz="0.0 0.0 0.0305" rpy="0.0 0.0 ${pi}" />
-      <parent link="${prefix}slamtec_rplidar_s3_link" />
+      <parent link="${prefix}${name}_link" />
       <child link="${prefix}${frame_id}" />
     </joint>
@@ -104,5 +105,5 @@
     <xacro:if value="${simulation_engine == 'gazebo-classic'}">
       <gazebo reference="${prefix}${frame_id}">
-        <sensor type="${ray_type}" name="${prefix}slamtec_rplidar_s3_sensor">
+        <sensor type="${ray_type}" name="${prefix}${name}_sensor">
           <visualize>false</visualize>
           <ray>

Commit message: added namespaces for astra rplidar
Signed-off-by: Jakub Delicat <jakub.delicat@husarion.com>

File: urdf/orbbec_astra.urdf.xacro (robot description, xacro)
@@ -5,5 +5,12 @@
                        tf_prefix:=None
                        camera_name:=camera
+                       namespace:=None
                        simulation_engine:=gazebo-classic">
+      <xacro:if value="${namespace == 'None'}">
+      <xacro:property name="namespace_ext" value="" />
+    </xacro:if>
+    <xacro:unless value="${namespace == 'None'}">
+        <xacro:property name="namespace_ext" value="${namespace}/" />
+    </xacro:unless>
     <xacro:if value="${tf_prefix == 'None'}">
       <xacro:property name="tf_prefix_ext" value="" />
@@ -65,5 +72,5 @@
     <link name="${tf_prefix_ext}${camera_name}_depth_optical_frame" />
     <joint name="${tf_prefix_ext}${camera_name}_depth_to_${tf_prefix_ext}${camera_name}_depth_optical_joint" type="fixed">
-      <origin xyz="0.0 0.0 0.0" rpy="${-pi/2} 0.0 ${-pi/2}" />
+      <origin xyz="0.0 0.0 0.0" rpy="0 0 0" />
       <parent link="${tf_prefix_ext}${camera_name}_depth_frame" />
       <child link="${tf_prefix_ext}${camera_name}_depth_optical_frame" />
@@ -75,5 +82,5 @@
           <always_on>true</always_on>
           <update_rate>20.0</update_rate>
-          <topic>${camera_name}</topic>
+          <topic>${namespace_ext}${camera_name}</topic>
           <!-- It is not possible to split the frame of the color and the depth stream.
                The frame of color stream should be ${tf_prefix_ext}${camera_name}_color_optical_frame -->
@@ -90,11 +97,9 @@
             </clip>
           </camera>
+          <ros>
+            <namespace>${namespace_ext}</namespace>
+          </ros>
         </sensor>
       </gazebo>
-      <!-- <gazebo>
-        <plugin filename="libignition-gazebo-sensors-system.so" name="ignition::gazebo::systems::Sensors">
-          <render_engine>ogre2</render_engine>
-        </plugin>
-      </gazebo>  -->
     </xacro:if>
     <xacro:if value="${simulation_engine == 'gazebo-classic'}">

File: urdf/slamtec_rplidar_a2.urdf.xacro (robot description, xacro)
@@ -13,5 +13,12 @@
                        frame_id:=laser
                        model:=A2M12
+                       namespace:=None
                        simulation_engine:=gazebo-classic">
+    <xacro:if value="${namespace == 'None'}">
+      <xacro:property name="namespace_ext" value="" />
+    </xacro:if>
+    <xacro:unless value="${namespace == 'None'}">
+        <xacro:property name="namespace_ext" value="${namespace}/" />
+    </xacro:unless>
     <xacro:if value="${use_gpu}">
       <xacro:if value="${simulation_engine == 'gazebo-classic'}">
@@ -89,6 +96,6 @@
     <xacro:if value="${simulation_engine == 'ignition-gazebo'}">
       <gazebo reference="${tf_prefix_ext}${frame_id}">
-        <sensor type="${ray_type}" name="${tf_prefix_ext}rplidar_a2_sensor">
-          <topic>${topic}</topic>
+        <sensor type="${ray_type}" name="${namespace_ext}${tf_prefix_ext}rplidar_a2_sensor">
+          <topic>${namespace_ext}scan</topic>
           <frame_id>${tf_prefix_ext}${frame_id}</frame_id>
           <ignition_frame_id>${tf_prefix_ext}${frame_id}</ignition_frame_id>
@@ -116,11 +123,9 @@
           <always_on>true</always_on>
           <visualize>false</visualize>
+          <ros>
+            <namespace>${namespace_ext}</namespace>
+          </ros>
         </sensor>
       </gazebo>
-      <gazebo>
-          <plugin filename="libignition-gazebo-sensors-system.so" name="ignition::gazebo::systems::Sensors">
-            <render_engine>ogre2</render_engine>
-          </plugin>
-        </gazebo>
     </xacro:if>
     <xacro:if value="${simulation_engine == 'gazebo-classic'}">

File: urdf/slamtec_rplidar_a3.urdf.xacro (robot description, xacro)
@@ -7,5 +7,12 @@
                        topic:=scan
                        frame_id:=laser
+                       namespace:=None
                        simulation_engine:=gazebo-classic">
+    <xacro:if value="${namespace == 'None'}">
+      <xacro:property name="namespace_ext" value="" />
+    </xacro:if>
+    <xacro:unless value="${namespace == 'None'}">
+        <xacro:property name="namespace_ext" value="${namespace}/" />
+    </xacro:unless>
     <xacro:if value="${use_gpu}">
       <xacro:if value="${simulation_engine == 'gazebo-classic'}">
@@ -67,6 +74,6 @@
     <xacro:if value="${simulation_engine == 'ignition-gazebo'}">
       <gazebo reference="${tf_prefix_ext}${frame_id}">
-        <sensor type="${ray_type}" name="${tf_prefix_ext}rplidar_a3_sensor">
-          <topic>${topic}</topic>
+        <sensor type="${ray_type}" name="${namespace_ext}${tf_prefix_ext}rplidar_a3_sensor">
+          <topic>${namespace_ext}${topic}</topic>
           <frame_id>${tf_prefix_ext}${frame_id}</frame_id>
           <ignition_frame_id>${tf_prefix_ext}${frame_id}</ignition_frame_id>
@@ -95,11 +102,9 @@
           <always_on>true</always_on>
           <visualize>false</visualize>
+          <ros>
+            <namespace>${namespace_ext}</namespace>
+          </ros>
         </sensor>
       </gazebo>
-      <gazebo>
-          <plugin filename="libignition-gazebo-sensors-system.so" name="ignition::gazebo::systems::Sensors">
-            <render_engine>ogre2</render_engine>
-          </plugin>
-        </gazebo>
     </xacro:if>
     <xacro:if value="${simulation_engine == 'gazebo-classic'}">

File: urdf/slamtec_rplidar_s1.urdf.xacro (robot description, xacro)
@@ -7,5 +7,12 @@
                        topic:=scan
                        frame_id:=laser
+                       namespace=None
                        simulation_engine:=gazebo-classic">
+    <xacro:if value="${namespace == 'None'}">
+      <xacro:property name="namespace_ext" value="" />
+    </xacro:if>
+    <xacro:unless value="${namespace == 'None'}">
+        <xacro:property name="namespace_ext" value="${namespace}/" />
+    </xacro:unless>
     <xacro:if value="${use_gpu}">
       <xacro:if value="${simulation_engine == 'gazebo-classic'}">
@@ -74,6 +81,6 @@
     <xacro:if value="${simulation_engine == 'ignition-gazebo'}">
       <gazebo reference="${tf_prefix_ext}${frame_id}">
-        <sensor type="${ray_type}" name="${tf_prefix_ext}rplidar_s1_sensor">
-          <topic>${topic}</topic>
+        <sensor type="${ray_type}" name="${namespace_ext}${tf_prefix_ext}rplidar_s1_sensor">
+          <topic>${namespace_ext}${topic}</topic>
           <frame_id>${tf_prefix_ext}${frame_id}</frame_id>
           <ignition_frame_id>${tf_prefix_ext}${frame_id}</ignition_frame_id>
@@ -101,10 +108,8 @@
           <always_on>1</always_on>
           <visualize>false</visualize>
+          <ros>
+            <namespace>${namespace_ext}</namespace>
+          </ros>
         </sensor>
-      </gazebo>
-      <gazebo>
-        <plugin filename="libignition-gazebo-sensors-system.so" name="ignition::gazebo::systems::Sensors">
-          <render_engine>ogre2</render_engine>
-        </plugin>
       </gazebo>
     </xacro:if>

Commit message: Tabs + ns

File: urdf/orbbec_astra.urdf.xacro (robot description, xacro)
@@ -7,9 +7,9 @@
                        namespace:=None
                        simulation_engine:=gazebo-classic">
-      <xacro:if value="${namespace == 'None'}">
-      <xacro:property name="namespace_ext" value="" />
+    <xacro:if value="${namespace == 'None'}">
+      <xacro:property name="ns" value="" />
     </xacro:if>
     <xacro:unless value="${namespace == 'None'}">
-        <xacro:property name="namespace_ext" value="${namespace}/" />
+      <xacro:property name="ns" value="${namespace}/" />
     </xacro:unless>
     <xacro:if value="${tf_prefix == 'None'}">
@@ -82,5 +82,5 @@
           <always_on>true</always_on>
           <update_rate>20.0</update_rate>
-          <topic>${namespace_ext}${camera_name}</topic>
+          <topic>${ns}${camera_name}</topic>
           <!-- It is not possible to split the frame of the color and the depth stream.
                The frame of color stream should be ${prefix}${camera_name}_color_optical_frame -->
@@ -98,5 +98,5 @@
           </camera>
           <ros>
-            <namespace>${namespace_ext}</namespace>
+            <namespace>${ns}</namespace>
           </ros>
         </sensor>

File: urdf/slamtec_rplidar_a2.urdf.xacro (robot description, xacro)
@@ -16,8 +16,8 @@
                        simulation_engine:=gazebo-classic">
     <xacro:if value="${namespace == 'None'}">
-      <xacro:property name="namespace_ext" value="" />
+      <xacro:property name="ns" value="" />
     </xacro:if>
     <xacro:unless value="${namespace == 'None'}">
-        <xacro:property name="namespace_ext" value="${namespace}/" />
+      <xacro:property name="ns" value="${namespace}/" />
     </xacro:unless>
     <xacro:if value="${use_gpu}">
@@ -96,6 +96,6 @@
     <xacro:if value="${simulation_engine == 'ignition-gazebo'}">
       <gazebo reference="${prefix}${frame_id}">
-        <sensor type="${ray_type}" name="${namespace_ext}${prefix}rplidar_a2_sensor">
-          <topic>${namespace_ext}${topic}</topic>
+        <sensor type="${ray_type}" name="${ns}${prefix}rplidar_a2_sensor">
+          <topic>${ns}${topic}</topic>
           <frame_id>${prefix}${frame_id}</frame_id>
           <ignition_frame_id>${prefix}${frame_id}</ignition_frame_id>
@@ -124,5 +124,5 @@
           <visualize>false</visualize>
           <ros>
-            <namespace>${namespace_ext}</namespace>
+            <namespace>${ns}</namespace>
           </ros>
         </sensor>

File: urdf/slamtec_rplidar_a3.urdf.xacro (robot description, xacro)
@@ -10,8 +10,8 @@
                        simulation_engine:=gazebo-classic">
     <xacro:if value="${namespace == 'None'}">
-      <xacro:property name="namespace_ext" value="" />
+      <xacro:property name="ns" value="" />
     </xacro:if>
     <xacro:unless value="${namespace == 'None'}">
-        <xacro:property name="namespace_ext" value="${namespace}/" />
+      <xacro:property name="ns" value="${namespace}/" />
     </xacro:unless>
     <xacro:if value="${use_gpu}">
@@ -74,6 +74,6 @@
     <xacro:if value="${simulation_engine == 'ignition-gazebo'}">
       <gazebo reference="${prefix}${frame_id}">
-        <sensor type="${ray_type}" name="${namespace_ext}${prefix}rplidar_a3_sensor">
-          <topic>${namespace_ext}${topic}</topic>
+        <sensor type="${ray_type}" name="${ns}${prefix}rplidar_a3_sensor">
+          <topic>${ns}${topic}</topic>
           <frame_id>${prefix}${frame_id}</frame_id>
           <ignition_frame_id>${prefix}${frame_id}</ignition_frame_id>
@@ -103,5 +103,5 @@
           <visualize>false</visualize>
           <ros>
-            <namespace>${namespace_ext}</namespace>
+            <namespace>${ns}</namespace>
           </ros>
         </sensor>

File: urdf/slamtec_rplidar_s1.urdf.xacro (robot description, xacro)
@@ -10,8 +10,8 @@
                        simulation_engine:=gazebo-classic">
     <xacro:if value="${namespace == 'None'}">
-      <xacro:property name="namespace_ext" value="" />
+      <xacro:property name="ns" value="" />
     </xacro:if>
     <xacro:unless value="${namespace == 'None'}">
-        <xacro:property name="namespace_ext" value="${namespace}/" />
+      <xacro:property name="ns" value="${namespace}/" />
     </xacro:unless>
     <xacro:if value="${use_gpu}">
@@ -81,6 +81,6 @@
     <xacro:if value="${simulation_engine == 'ignition-gazebo'}">
       <gazebo reference="${prefix}${frame_id}">
-        <sensor type="${ray_type}" name="${namespace_ext}${prefix}rplidar_s1_sensor">
-          <topic>${namespace_ext}${topic}</topic>
+        <sensor type="${ray_type}" name="${ns}${prefix}rplidar_s1_sensor">
+          <topic>${ns}${topic}</topic>
           <frame_id>${prefix}${frame_id}</frame_id>
           <ignition_frame_id>${prefix}${frame_id}</ignition_frame_id>
@@ -109,5 +109,5 @@
           <visualize>false</visualize>
           <ros>
-            <namespace>${namespace_ext}</namespace>
+            <namespace>${ns}</namespace>
           </ros>
         </sensor>

File: urdf/slamtec_rplidar_s2.urdf.xacro (robot description, xacro)
@@ -10,8 +10,8 @@
                        simulation_engine:=gazebo-classic">
     <xacro:if value="${namespace == 'None'}">
-      <xacro:property name="namespace_ext" value="" />
+      <xacro:property name="ns" value="" />
     </xacro:if>
     <xacro:unless value="${namespace == 'None'}">
-        <xacro:property name="namespace_ext" value="${namespace}/" />
+      <xacro:property name="ns" value="${namespace}/" />
     </xacro:unless>
     <xacro:if value="${use_gpu}">
@@ -74,6 +74,6 @@
     <xacro:if value="${simulation_engine == 'ignition-gazebo'}">
       <gazebo reference="${prefix}${frame_id}">
-        <sensor type="${ray_type}" name="${namespace_ext}${prefix}rplidar_s2_sensor">
-          <topic>${namespace_ext}${topic}</topic>
+        <sensor type="${ray_type}" name="${ns}${prefix}rplidar_s2_sensor">
+          <topic>${ns}${topic}</topic>
           <frame_id>${prefix}${frame_id}</frame_id>
           <ignition_frame_id>${prefix}${frame_id}</ignition_frame_id>
@@ -102,5 +102,5 @@
           <visualize>false</visualize>
           <ros>
-            <namespace>${namespace_ext}</namespace>
+            <namespace>${ns}</namespace>
           </ros>
         </sensor>

File: urdf/slamtec_rplidar_s3.urdf.xacro (robot description, xacro)
@@ -10,8 +10,8 @@
                        simulation_engine:=gazebo-classic">
     <xacro:if value="${namespace == 'None'}">
-      <xacro:property name="namespace_ext" value="" />
+      <xacro:property name="ns" value="" />
     </xacro:if>
     <xacro:unless value="${namespace == 'None'}">
-        <xacro:property name="namespace_ext" value="${namespace}/" />
+      <xacro:property name="ns" value="${namespace}/" />
     </xacro:unless>
     <xacro:if value="${use_gpu}">
@@ -74,6 +74,6 @@
     <xacro:if value="${simulation_engine == 'ignition-gazebo'}">
       <gazebo reference="${prefix}${frame_id}">
-        <sensor type="${ray_type}" name="${namespace_ext}${prefix}rplidar_s3_sensor">
-          <topic>${namespace_ext}${topic}</topic>
+        <sensor type="${ray_type}" name="${ns}${prefix}rplidar_s3_sensor">
+          <topic>${ns}${topic}</topic>
           <frame_id>${prefix}${frame_id}</frame_id>
           <ignition_frame_id>${prefix}${frame_id}</ignition_frame_id>
@@ -103,5 +103,5 @@
         </sensor>
         <ros>
-          <namespace>${namespace_ext}</namespace>
+          <namespace>${ns}</namespace>
         </ros>
       </gazebo>
