Commit message: Gazebo ignition multirobots (#39)
* added namespaces for astra rplidar

Signed-off-by: Jakub Delicat <jakub.delicat@husarion.com>

* added namespace gazebo to other rplidars

Signed-off-by: Jakub Delicat <jakub.delicat@husarion.com>

* Tabs + ns

---------

Signed-off-by: Jakub Delicat <jakub.delicat@husarion.com>
Co-authored-by: rafal-gorecki <rafal.gorecki@husarion.com>

File: urdf/orbbec_astra.urdf.xacro (robot description, xacro)
@@ -5,5 +5,12 @@
                        tf_prefix:=None
                        camera_name:=camera
+                       namespace:=None
                        simulation_engine:=gazebo-classic">
+    <xacro:if value="${namespace == 'None'}">
+      <xacro:property name="ns" value="" />
+    </xacro:if>
+    <xacro:unless value="${namespace == 'None'}">
+      <xacro:property name="ns" value="${namespace}/" />
+    </xacro:unless>
     <xacro:if value="${tf_prefix == 'None'}">
       <xacro:property name="prefix" value="" />
@@ -75,5 +82,5 @@
           <always_on>true</always_on>
           <update_rate>20.0</update_rate>
-          <topic>${camera_name}</topic>
+          <topic>${ns}${camera_name}</topic>
           <!-- It is not possible to split the frame of the color and the depth stream.
                The frame of color stream should be ${prefix}${camera_name}_color_optical_frame -->
@@ -90,11 +97,9 @@
             </clip>
           </camera>
+          <ros>
+            <namespace>${ns}</namespace>
+          </ros>
         </sensor>
       </gazebo>
-      <!-- <gazebo>
-        <plugin filename="libignition-gazebo-sensors-system.so" name="ignition::gazebo::systems::Sensors">
-          <render_engine>ogre2</render_engine>
-        </plugin>
-      </gazebo>  -->
     </xacro:if>
     <xacro:if value="${simulation_engine == 'gazebo-classic'}">

File: urdf/slamtec_rplidar_a2.urdf.xacro (robot description, xacro)
@@ -13,5 +13,12 @@
                        frame_id:=laser
                        model:=A2M12
+                       namespace:=None
                        simulation_engine:=gazebo-classic">
+    <xacro:if value="${namespace == 'None'}">
+      <xacro:property name="ns" value="" />
+    </xacro:if>
+    <xacro:unless value="${namespace == 'None'}">
+      <xacro:property name="ns" value="${namespace}/" />
+    </xacro:unless>
     <xacro:if value="${use_gpu}">
       <xacro:if value="${simulation_engine == 'gazebo-classic'}">
@@ -89,6 +96,6 @@
     <xacro:if value="${simulation_engine == 'ignition-gazebo'}">
       <gazebo reference="${prefix}${frame_id}">
-        <sensor type="${ray_type}" name="${prefix}rplidar_a2_sensor">
-          <topic>${topic}</topic>
+        <sensor type="${ray_type}" name="${ns}${prefix}rplidar_a2_sensor">
+          <topic>${ns}${topic}</topic>
           <frame_id>${prefix}${frame_id}</frame_id>
           <ignition_frame_id>${prefix}${frame_id}</ignition_frame_id>
@@ -116,11 +123,9 @@
           <always_on>true</always_on>
           <visualize>false</visualize>
+          <ros>
+            <namespace>${ns}</namespace>
+          </ros>
         </sensor>
       </gazebo>
-      <gazebo>
-          <plugin filename="libignition-gazebo-sensors-system.so" name="ignition::gazebo::systems::Sensors">
-            <render_engine>ogre2</render_engine>
-          </plugin>
-        </gazebo>
     </xacro:if>
     <xacro:if value="${simulation_engine == 'gazebo-classic'}">

File: urdf/slamtec_rplidar_a3.urdf.xacro (robot description, xacro)
@@ -7,5 +7,12 @@
                        topic:=scan
                        frame_id:=laser
+                       namespace:=None
                        simulation_engine:=gazebo-classic">
+    <xacro:if value="${namespace == 'None'}">
+      <xacro:property name="ns" value="" />
+    </xacro:if>
+    <xacro:unless value="${namespace == 'None'}">
+      <xacro:property name="ns" value="${namespace}/" />
+    </xacro:unless>
     <xacro:if value="${use_gpu}">
       <xacro:if value="${simulation_engine == 'gazebo-classic'}">
@@ -67,6 +74,6 @@
     <xacro:if value="${simulation_engine == 'ignition-gazebo'}">
       <gazebo reference="${prefix}${frame_id}">
-        <sensor type="${ray_type}" name="${prefix}rplidar_a3_sensor">
-          <topic>${topic}</topic>
+        <sensor type="${ray_type}" name="${ns}${prefix}rplidar_a3_sensor">
+          <topic>${ns}${topic}</topic>
           <frame_id>${prefix}${frame_id}</frame_id>
           <ignition_frame_id>${prefix}${frame_id}</ignition_frame_id>
@@ -95,11 +102,9 @@
           <always_on>true</always_on>
           <visualize>false</visualize>
+          <ros>
+            <namespace>${ns}</namespace>
+          </ros>
         </sensor>
       </gazebo>
-      <gazebo>
-          <plugin filename="libignition-gazebo-sensors-system.so" name="ignition::gazebo::systems::Sensors">
-            <render_engine>ogre2</render_engine>
-          </plugin>
-        </gazebo>
     </xacro:if>
     <xacro:if value="${simulation_engine == 'gazebo-classic'}">

File: urdf/slamtec_rplidar_s1.urdf.xacro (robot description, xacro)
@@ -7,5 +7,12 @@
                        topic:=scan
                        frame_id:=laser
+                       namespace=None
                        simulation_engine:=gazebo-classic">
+    <xacro:if value="${namespace == 'None'}">
+      <xacro:property name="ns" value="" />
+    </xacro:if>
+    <xacro:unless value="${namespace == 'None'}">
+      <xacro:property name="ns" value="${namespace}/" />
+    </xacro:unless>
     <xacro:if value="${use_gpu}">
       <xacro:if value="${simulation_engine == 'gazebo-classic'}">
@@ -74,6 +81,6 @@
     <xacro:if value="${simulation_engine == 'ignition-gazebo'}">
       <gazebo reference="${prefix}${frame_id}">
-        <sensor type="${ray_type}" name="${prefix}rplidar_s1_sensor">
-          <topic>${topic}</topic>
+        <sensor type="${ray_type}" name="${ns}${prefix}rplidar_s1_sensor">
+          <topic>${ns}${topic}</topic>
           <frame_id>${prefix}${frame_id}</frame_id>
           <ignition_frame_id>${prefix}${frame_id}</ignition_frame_id>
@@ -101,10 +108,8 @@
           <always_on>1</always_on>
           <visualize>false</visualize>
+          <ros>
+            <namespace>${ns}</namespace>
+          </ros>
         </sensor>
-      </gazebo>
-      <gazebo>
-        <plugin filename="libignition-gazebo-sensors-system.so" name="ignition::gazebo::systems::Sensors">
-          <render_engine>ogre2</render_engine>
-        </plugin>
       </gazebo>
     </xacro:if>

File: urdf/slamtec_rplidar_s2.urdf.xacro (robot description, xacro)
@@ -7,5 +7,12 @@
                        topic:=scan
                        frame_id:=laser
+                       namespace=None
                        simulation_engine:=gazebo-classic">
+    <xacro:if value="${namespace == 'None'}">
+      <xacro:property name="ns" value="" />
+    </xacro:if>
+    <xacro:unless value="${namespace == 'None'}">
+      <xacro:property name="ns" value="${namespace}/" />
+    </xacro:unless>
     <xacro:if value="${use_gpu}">
       <xacro:if value="${simulation_engine == 'gazebo-classic'}">
@@ -67,6 +74,6 @@
     <xacro:if value="${simulation_engine == 'ignition-gazebo'}">
       <gazebo reference="${prefix}${frame_id}">
-        <sensor type="${ray_type}" name="${prefix}rplidar_s2_sensor">
-          <topic>${topic}</topic>
+        <sensor type="${ray_type}" name="${ns}${prefix}rplidar_s2_sensor">
+          <topic>${ns}${topic}</topic>
           <frame_id>${prefix}${frame_id}</frame_id>
           <ignition_frame_id>${prefix}${frame_id}</ignition_frame_id>
@@ -94,10 +101,8 @@
           <always_on>1</always_on>
           <visualize>false</visualize>
+          <ros>
+            <namespace>${ns}</namespace>
+          </ros>
         </sensor>
-      </gazebo>
-      <gazebo>
-        <plugin filename="libignition-gazebo-sensors-system.so" name="ignition::gazebo::systems::Sensors">
-          <render_engine>ogre2</render_engine>
-        </plugin>
       </gazebo>
     </xacro:if>

File: urdf/slamtec_rplidar_s3.urdf.xacro (robot description, xacro)
@@ -7,5 +7,12 @@
                        topic:=scan
                        frame_id:=laser
+                       namespace=None
                        simulation_engine:=gazebo-classic">
+    <xacro:if value="${namespace == 'None'}">
+      <xacro:property name="ns" value="" />
+    </xacro:if>
+    <xacro:unless value="${namespace == 'None'}">
+      <xacro:property name="ns" value="${namespace}/" />
+    </xacro:unless>
     <xacro:if value="${use_gpu}">
       <xacro:if value="${simulation_engine == 'gazebo-classic'}">
@@ -67,6 +74,6 @@
     <xacro:if value="${simulation_engine == 'ignition-gazebo'}">
       <gazebo reference="${prefix}${frame_id}">
-        <sensor type="${ray_type}" name="${prefix}rplidar_s3_sensor">
-          <topic>${topic}</topic>
+        <sensor type="${ray_type}" name="${ns}${prefix}rplidar_s3_sensor">
+          <topic>${ns}${topic}</topic>
           <frame_id>${prefix}${frame_id}</frame_id>
           <ignition_frame_id>${prefix}${frame_id}</ignition_frame_id>
@@ -95,9 +102,7 @@
           <visualize>false</visualize>
         </sensor>
-      </gazebo>
-      <gazebo>
-        <plugin filename="libignition-gazebo-sensors-system.so" name="ignition::gazebo::systems::Sensors">
-          <render_engine>ogre2</render_engine>
-        </plugin>
+        <ros>
+          <namespace>${ns}</namespace>
+        </ros>
       </gazebo>
     </xacro:if>
