Commit message: Fix floats formatting
Co-authored-by: Krzysztof Wojciechowski <49921081+Kotochleb@users.noreply.github.com>

File: urdf/intel_realsense_d435.urdf.xacro (robot description, xacro)
@@ -112,5 +112,5 @@
       <!-- camera right IR joints and links -->
       <joint name="${name}_to_${name}_infra2_joint" type="fixed">
-        <origin xyz="0 ${d435_cam_depth_to_infra2_offset} 0.0" rpy="0.0 0.0 0.0" />
+        <origin xyz="0.0 ${d435_cam_depth_to_infra2_offset} 0.0" rpy="0.0 0.0 0.0" />
         <parent link="${name}_link" />
         <child link="${name}_infra2_frame" />
@@ -155,5 +155,5 @@
           <clip>
             <near>0.02</near>
-            <far>300</far>
+            <far>300.0</far>
           </clip>
         </sensor>
@@ -177,5 +177,5 @@
           <noise>
             <type>gaussian</type>
-            <mean>0</mean>
+            <mean>0.0</mean>
             <stddev>0.005</stddev>
           </noise>

Commit message: Fix inertia formatting

File: urdf/intel_realsense_d435.urdf.xacro (robot description, xacro)
@@ -78,5 +78,7 @@
         <mass value="0.072" />
         <origin xyz="0.0 0.0 0.0" />
-        <inertia ixx="0.003881243" ixy="0.0" ixz="0.0" iyy="0.000498940" iyz="0.0" izz="0.003879257" />
+        <inertia ixx="0.003881243" ixy="0.0"         ixz="0.0"
+                                   iyy="0.000498940" iyz="0.0"
+                                                     izz="0.003879257" />
       </inertial>
     </link>

Commit message: change mesh files finding method

File: urdf/intel_realsense_d435.urdf.xacro (robot description, xacro)
@@ -65,5 +65,5 @@
         <origin xyz="0.0 0.0 0.0" rpy="0.0 0.0 0.0" />
         <geometry>
-          <mesh filename="file://$(find ros_components_description)/meshes/intel_realsense_d435.dae" />
+          <mesh filename="package://ros_components_description/meshes/intel_realsense_d435.dae" />
         </geometry>
       </visual>

File: urdf/orbbec_astra.urdf.xacro (robot description, xacro)
@@ -22,5 +22,5 @@
         <origin xyz="0.0 0.0 0.0" rpy="0.0 0.0 0.0" />
         <geometry>
-          <mesh filename="file://$(find ros_components_description)/meshes/orbbec_astra.dae" />
+          <mesh filename="package://ros_components_description/meshes/orbbec_astra.dae" />
         </geometry>
       </visual>

File: urdf/ouster_os1_32.urdf.xacro (robot description, xacro)
@@ -31,5 +31,5 @@
         <origin xyz="0.0 0.0 0.0" rpy="0.0 0.0 0.0" />
         <geometry>
-          <mesh filename="file://$(find ros_components_description)/meshes/ouster_os1_32.dae" />
+          <mesh filename="package://ros_components_description/meshes/ouster_os1_32.dae" />
         </geometry>
       </visual>

File: urdf/slamtec_rplidar_a2.urdf.xacro (robot description, xacro)
@@ -54,5 +54,5 @@
         <origin xyz="0.0 0.0 0.0" rpy="0.0 0.0 0.0" />
         <geometry>
-          <mesh filename="file://$(find ros_components_description)/meshes/${mesh}" />
+          <mesh filename="package://ros_components_description/meshes/${mesh}" />
         </geometry>
       </visual>

File: urdf/slamtec_rplidar_a3.urdf.xacro (robot description, xacro)
@@ -32,5 +32,5 @@
         <geometry>
           <!-- slamtec_rplidar_ax.dae is used as a shared mesh for A2 and A3 rplidars -->
-          <mesh filename="file://$(find ros_components_description)/meshes/slamtec_rplidar_ax.dae" />
+          <mesh filename="package://ros_components_description/meshes/slamtec_rplidar_ax.dae" />
         </geometry>
       </visual>

File: urdf/slamtec_rplidar_s1.urdf.xacro (robot description, xacro)
@@ -31,5 +31,5 @@
         <origin xyz="0.0 0.0 0.0" rpy="0.0 0.0 0.0" />
         <geometry>
-          <mesh filename="file://$(find ros_components_description)/meshes/slamtec_rplidar_s1.dae" />
+          <mesh filename="package://ros_components_description/meshes/slamtec_rplidar_s1.dae" />
         </geometry>
       </visual>

File: urdf/velodyne_puck.urdf.xacro (robot description, xacro)
@@ -31,5 +31,5 @@
         <origin xyz="0.0 0.0 0.0" rpy="0.0 0.0 0.0" />
         <geometry>
-          <mesh filename="file://$(find ros_components_description)/meshes/velodyne_puck.dae" />
+          <mesh filename="package://ros_components_description/meshes/velodyne_puck.dae" />
         </geometry>
       </visual>

Commit message: fix resolution

File: urdf/intel_realsense_d435.urdf.xacro (robot description, xacro)
@@ -168,18 +168,21 @@
             way to change it, interestingly depth image is published correctly in the ignition_frame_id -->
           <ignition_frame_id>${name}_depth_optical_frame</ignition_frame_id>
-          <horizontal_fov>${87.0/180.0*pi}</horizontal_fov>
-          <image>
-            <width>1280</width>
-            <height>720</height>
-          </image>
-          <clip>
-            <near>0.28</near>
-            <far>8.0</far>
-          </clip>
-          <noise>
-            <type>gaussian</type>
-            <mean>0.0</mean>
-            <stddev>0.005</stddev>
-          </noise>
+          <camera>
+            <horizontal_fov>${87.0/180.0*pi}</horizontal_fov>
+            <image>
+              <width>1280</width>
+              <height>720</height>
+              <format>R_FLOAT32</format>
+            </image>
+            <clip>
+              <near>0.28</near>
+              <far>8.0</far>
+            </clip>
+            <noise>
+              <type>gaussian</type>
+              <mean>0.0</mean>
+              <stddev>0.005</stddev>
+            </noise>
+          </camera>
         </sensor>
       </gazebo>

File: urdf/stereolabs_zed.urdf.xacro (robot description, xacro)
@@ -101,4 +101,11 @@
       <origin xyz="0 0 ${height/2}" rpy="0 ${bottom_slope} 0" />
     </joint>
+    <!-- Artificially Created Camera Center -->
+    <link name="${name}_center_optical_frame" />
+    <joint name="${name}_center_joint" type="fixed">
+      <parent link="${name}_camera_center" />
+      <child link="${name}_center_optical_frame" />
+      <origin xyz="0.01 0 0" rpy="0 0 0" />
+    </joint>
     <!-- Left Camera -->
     <link name="${name}_left_camera_frame" />
@@ -157,5 +164,5 @@
       <!-- It is also possible to use single rgbd_camera sensor, but using separate rgb and depth camera
         should be more accurate different frames and fovs can be set -->
-      <gazebo reference="${name}_link">
+      <gazebo reference="${name}_center_optical_frame">
         <sensor type="camera" name="${name}_color">
           <always_on>true</always_on>
@@ -163,15 +170,17 @@
           <topic>${topic}/color/image_raw</topic>
           <visualize>false</visualize>
-          <ignition_frame_id>${name}_left_camera_optical_frame</ignition_frame_id>
-          <horizontal_fov>${110.0/180.0*pi}</horizontal_fov>
-          <image>
-            <width>1920</width>
-            <height>1080</height>
-            <format>R8G8B8</format>
-          </image>
-          <clip>
-            <near>0.02</near>
-            <far>300.0</far>
-          </clip>
+          <ignition_frame_id>${name}_center_optical_frame</ignition_frame_id>
+          <camera>
+            <horizontal_fov>${110.0/180.0*pi}</horizontal_fov>
+            <image>
+              <width>1920</width>
+              <height>1080</height>
+              <format>R8G8B8</format>
+            </image>
+            <clip>
+              <near>0.02</near>
+              <far>300.0</far>
+            </clip>
+          </camera>
         </sensor>
         <sensor type="depth_camera" name="${name}_depth">
@@ -182,18 +191,21 @@
           <!-- Pointcloud is published in internal gazebo frame name, and there seem to be no
             way to change it, interestingly depth image is published correctly in the ignition_frame_id -->
-          <ignition_frame_id>${name}_left_camera_optical_frame</ignition_frame_id>
-          <horizontal_fov>${110.0/180.0*pi}</horizontal_fov>
-          <image>
-            <width>1920</width>
-            <height>1080</height>
-          </image>
-          <clip>
-            <near>0.3</near>
-            <far>20.0</far>
-          </clip>
-          <noise type="gaussian">
-            <mean>0.0</mean>
-            <stddev>0.03</stddev>
-          </noise>
+          <ignition_frame_id>${name}_center_optical_frame</ignition_frame_id>
+          <camera>
+            <horizontal_fov>${110.0/180.0*pi}</horizontal_fov>
+            <image>
+              <width>1920</width>
+              <height>1080</height>
+              <format>R_FLOAT32</format>
+            </image>
+            <clip>
+              <near>0.3</near>
+              <far>20.0</far>
+            </clip>
+            <noise type="gaussian">
+              <mean>0.0</mean>
+              <stddev>0.03</stddev>
+            </noise>
+          </camera>
         </sensor>
       </gazebo>

Commit message: Fix Point Cloud

File: urdf/intel_realsense_d435.urdf.xacro (robot description, xacro)
@@ -139,4 +139,12 @@
       <link name="${name}_color_optical_frame" />
     </xacro:if>
+    <!-- To be removed after changing the version to a newer version of Gazebo (current Fortress)
+    Causing this bag https://github.com/gazebosim/gz-sensors/issues/239 -->
+    <link name="rosbot_xl/base_link/camera_depth" />
+    <joint name="${name}_workaround_joint" type="fixed">
+      <parent link="${name}_depth_frame" />
+      <child link="rosbot_xl/base_link/camera_depth" />
+      <origin xyz="0 0 0" rpy="0 0 0" />
+    </joint>
     <xacro:if value="${simulation_engine == 'ignition-gazebo'}">
       <!-- It is also possible to use single rgbd_camera sensor, but using separate rgb and depth camera
@@ -165,6 +173,4 @@
           <topic>${topic}/depth</topic>
           <visualize>false</visualize>
-          <!-- Pointcloud is published in internal gazebo frame name, and there seem to be no
-            way to change it, interestingly depth image is published correctly in the ignition_frame_id -->
           <ignition_frame_id>${name}_depth_optical_frame</ignition_frame_id>
           <camera>

File: urdf/stereolabs_zed.urdf.xacro (robot description, xacro)
@@ -87,5 +87,5 @@
         </geometry>
         <material name="mat">
-          <color rgba="0.25 0.25 0.25 0.99"/>
+          <color rgba="0.25 0.25 0.25 0.99" />
         </material>
       </visual>
@@ -154,13 +154,16 @@
         <origin xyz="0 0 0" rpy="0 0 0" />
       </joint>
-      <link name="${name}_temp_right_link" />
-      <joint name="${name}_temp_right_joint" type="fixed">
-        <parent link="${name}_right_camera_frame" />
-        <child link="${name}_temp_right_link" />
-        <origin xyz="0 0 0" rpy="0 0 0" />
-      </joint>
-    </xacro:if>
+    </xacro:if>
+    <!-- To be removed after changing the version to a newer version of Gazebo (current Fortress)
+    Causing this bag https://github.com/gazebosim/gz-sensors/issues/239 -->
+    <link name="rosbot_xl/base_link/camera_depth" />
+    <joint name="${name}_workaround_joint" type="fixed">
+      <parent link="${name}_center_optical_frame" />
+      <child link="rosbot_xl/base_link/camera_depth" />
+      <origin xyz="0 0 0" rpy="0 0 0" />
+    </joint>
     <xacro:if value="${simulation_engine == 'ignition-gazebo'}">
-      <!-- It is also possible to use single rgbd_camera sensor, but using separate rgb and depth camera
+      <!-- It is also possible to use single rgbd_camera sensor, but using separate rgb and depth
+      camera
         should be more accurate different frames and fovs can be set -->
       <gazebo reference="${name}_center_optical_frame">
@@ -168,5 +171,5 @@
           <always_on>true</always_on>
           <update_rate>30.0</update_rate>
-          <topic>${topic}/color/image_raw</topic>
+          <topic>${model}/zed_node/rgb/image_rect_color</topic>
           <visualize>false</visualize>
           <ignition_frame_id>${name}_center_optical_frame</ignition_frame_id>
@@ -187,8 +190,6 @@
           <always_on>true</always_on>
           <update_rate>30.0</update_rate>
-          <topic>${topic}/depth</topic>
+          <topic>${model}/zed_node/point_cloud/cloud_registered</topic>
           <visualize>false</visualize>
-          <!-- Pointcloud is published in internal gazebo frame name, and there seem to be no
-            way to change it, interestingly depth image is published correctly in the ignition_frame_id -->
           <ignition_frame_id>${name}_center_optical_frame</ignition_frame_id>
           <camera>

Commit message: delete pointcloud tf

File: urdf/intel_realsense_d435.urdf.xacro (robot description, xacro)
@@ -139,12 +139,4 @@
       <link name="${name}_color_optical_frame" />
     </xacro:if>
-    <!-- To be removed after changing the version to a newer version of Gazebo (current Fortress)
-    Causing this bag https://github.com/gazebosim/gz-sensors/issues/239 -->
-    <link name="rosbot_xl/base_link/camera_depth" />
-    <joint name="${name}_workaround_joint" type="fixed">
-      <parent link="${name}_depth_frame" />
-      <child link="rosbot_xl/base_link/camera_depth" />
-      <origin xyz="0 0 0" rpy="0 0 0" />
-    </joint>
     <xacro:if value="${simulation_engine == 'ignition-gazebo'}">
       <!-- It is also possible to use single rgbd_camera sensor, but using separate rgb and depth camera

File: urdf/stereolabs_zed.urdf.xacro (robot description, xacro)
@@ -155,12 +155,4 @@
       </joint>
     </xacro:if>
-    <!-- To be removed after changing the version to a newer version of Gazebo (current Fortress)
-    Causing this bag https://github.com/gazebosim/gz-sensors/issues/239 -->
-    <link name="rosbot_xl/base_link/camera_depth" />
-    <joint name="${name}_workaround_joint" type="fixed">
-      <parent link="${name}_center_optical_frame" />
-      <child link="rosbot_xl/base_link/camera_depth" />
-      <origin xyz="0 0 0" rpy="0 0 0" />
-    </joint>
     <xacro:if value="${simulation_engine == 'ignition-gazebo'}">
       <!-- It is also possible to use single rgbd_camera sensor, but using separate rgb and depth

Commit message: Fix rviz model paths (#28)
* added env hook for gazebo

* use package:// instead of file://

File: urdf/intel_realsense_d435.urdf.xacro (robot description, xacro)
@@ -65,5 +65,5 @@
         <origin xyz="0.0 0.0 0.0" rpy="0.0 0.0 0.0" />
         <geometry>
-          <mesh filename="file://$(find ros_components_description)/meshes/intel_realsense_d435.dae" />
+          <mesh filename="package://ros_components_description/meshes/intel_realsense_d435.dae" />
         </geometry>
       </visual>

File: urdf/orbbec_astra.urdf.xacro (robot description, xacro)
@@ -21,5 +21,5 @@
         <origin xyz="0.0 0.0 0.0" rpy="0.0 0.0 0.0" />
         <geometry>
-          <mesh filename="file://$(find ros_components_description)/meshes/orbbec_astra.dae" />
+          <mesh filename="package://ros_components_description/meshes/orbbec_astra.dae" />
         </geometry>
       </visual>
