Commit message: Undo formatting

File: urdf/intel_realsense_d435.urdf.xacro (robot description, xacro)
@@ -24,8 +24,10 @@
             use_nominal_extrinsics:=false
             simulation_engine:=ignition-gazebo">
-    <xacro:property name="prefix" value="${tf_prefix}" lazy_eval="false" />
-    <xacro:if value="${prefix != ''}">
+    <xacro:if value="${tf_prefix == ''}">
+      <xacro:property name="prefix" value="" />
+    </xacro:if>
+    <xacro:unless value="${tf_prefix == ''}">
       <xacro:property name="prefix" value="${tf_prefix}_" />
-    </xacro:if>
+    </xacro:unless>
     <!-- The following values are approximate, and the camera node
       publishing TF values with actual calibrated camera extrinsic values -->

File: urdf/orbbec_astra.urdf.xacro (robot description, xacro)
@@ -2,15 +2,15 @@
 <robot name="orbbec_astra" xmlns:xacro="http://www.ros.org/wiki/xacro">
   <xacro:macro name="orbbec_astra"
-    params="parent_link xyz rpy
-            tf_prefix:=''
-            name:=camera
-            simulation_engine:=ignition-gazebo">
-    <xacro:property name="prefix" value="${tf_prefix}" lazy_eval="false" />
-    <xacro:if value="${prefix != ''}">
+               params="parent_link xyz rpy
+                       tf_prefix:=''
+                       name:=camera
+                       simulation_engine:=ignition-gazebo">
+    <xacro:if value="${tf_prefix == ''}">
+      <xacro:property name="prefix" value="" />
+    </xacro:if>
+    <xacro:unless value="${tf_prefix == ''}">
       <xacro:property name="prefix" value="${tf_prefix}_" />
-    </xacro:if>
-    <joint
-      name="${parent_link.rstrip('_link')}_to_${prefix}${name}_orbbec_astra_joint"
-      type="fixed">
+    </xacro:unless>
+    <joint name="${parent_link.rstrip('_link')}_to_${prefix}${name}_orbbec_astra_joint" type="fixed">
       <origin xyz="${xyz}" rpy="${rpy}" />
       <parent link="${parent_link}" />
@@ -41,11 +41,10 @@
         <origin xyz="0.0 0.0 ${0.019+0.01}" rpy="0.0 0.0 0.0" />
         <mass value="0.300" />
-        <inertia ixx="0.00073916" ixy="0.0" ixz="0.0"
-          iyy="0.00015435" iyz="0.0"
-          izz="0.00077395" />
+        <inertia ixx="0.00073916" ixy="0.0"        ixz="0.0"
+                                  iyy="0.00015435" iyz="0.0"
+                                                   izz="0.00077395" />
       </inertial>
     </link>
-    <joint name="${parent_link.rstrip('_link')}_to_${prefix}${name}_color_joint"
-      type="fixed">
+    <joint name="${parent_link.rstrip('_link')}_to_${prefix}${name}_color_joint" type="fixed">
       <origin xyz="-0.002 0.0125 0.03325" rpy="-0.003 0.0 -0.003" />
       <parent link="${parent_link}" />
@@ -60,7 +59,5 @@
     </joint>
     <link name="${prefix}${name}_color_frame" />
-    <joint
-      name="${prefix}${name}_color_to_${prefix}${name}_color_optical_joint"
-      type="fixed">
+    <joint name="${prefix}${name}_color_to_${prefix}${name}_color_optical_joint" type="fixed">
       <origin xyz="0.0 0.0 0.0" rpy="${-pi/2} 0.0 ${-pi/2}" />
       <parent link="${prefix}${name}_color_frame" />
@@ -83,5 +80,5 @@
           <topic>${name}</topic>
           <!-- It is not possible to split the frame of the color and the depth stream.
-                                 The frame of color stream should be ${prefix}${name}_color_optical_frame -->
+               The frame of color stream should be ${prefix}${name}_color_optical_frame -->
           <ignition_frame_id>${prefix}${name}_depth_optical_frame</ignition_frame_id>
           <camera name="${prefix}camera">
@@ -99,8 +96,8 @@
       </gazebo>
       <!-- <gazebo>
-                          <plugin filename="libignition-gazebo-sensors-system.so" name="ignition::gazebo::systems::Sensors">
-                            <render_engine>ogre2</render_engine>
-                          </plugin>
-                        </gazebo>  -->
+        <plugin filename="libignition-gazebo-sensors-system.so" name="ignition::gazebo::systems::Sensors">
+          <render_engine>ogre2</render_engine>
+        </plugin>
+      </gazebo>  -->
     </xacro:if>
     <xacro:if value="${simulation_engine == 'gazebo-classic'}">

File: urdf/ouster_os1_32.urdf.xacro (robot description, xacro)
@@ -17,8 +17,10 @@
       <xacro:property name="plugin_file_name" value="libgazebo_ros_velodyne_laser.so" />
     </xacro:unless>
-    <xacro:property name="prefix" value="${tf_prefix}" lazy_eval="false" />
-    <xacro:if value="${prefix != ''}">
+    <xacro:if value="${tf_prefix == ''}">
+      <xacro:property name="prefix" value="" />
+    </xacro:if>
+    <xacro:unless value="${tf_prefix == ''}">
       <xacro:property name="prefix" value="${tf_prefix}_" />
-    </xacro:if>
+    </xacro:unless>
     <joint name="${parent_link.rstrip('_link')}_to_${prefix}${name}_joint" type="fixed">
       <origin xyz="${xyz}" rpy="${rpy}" />

File: urdf/slamtec_rplidar_a2.urdf.xacro (robot description, xacro)
@@ -33,10 +33,11 @@
       </xacro:if>
     </xacro:unless>
-    <xacro:property name="prefix" value="${tf_prefix}" lazy_eval="false" />
-    <xacro:if value="${prefix != ''}">
+    <xacro:if value="${tf_prefix == ''}">
+      <xacro:property name="prefix" value="" />
+    </xacro:if>
+    <xacro:unless value="${tf_prefix == ''}">
       <xacro:property name="prefix" value="${tf_prefix}_" />
-    </xacro:if>
-    <!--values
-    of max distance are based on tradeoff values between best and worst case scenarios -->
+    </xacro:unless>
+    <!--values of max distance are based on tradeoff values between best and worst case scenarios -->
     <!-- slamtec_rplidar_ax.dae is used as a shared mesh for A2 and A3 rplidars -->
     <xacro:if value="${model == 'A2M7'}">
@@ -55,6 +56,5 @@
       <xacro:property name="mesh" value="slamtec_rplidar_ax.dae" />
     </xacro:if>
-    <joint name="${parent_link.rstrip('_link')}_to_${prefix}${name}_joint"
-      type="fixed">
+    <joint name="${parent_link.rstrip('_link')}_to_${prefix}${name}_joint" type="fixed">
       <origin xyz="${xyz}" rpy="${rpy}" />
       <parent link="${parent_link}" />
@@ -82,7 +82,5 @@
       </inertial>
     </link>
-    <joint
-      name="${prefix}${name}_to_${prefix}${frame_id.rstrip('_link')}_joint"
-      type="fixed">
+    <joint name="${prefix}${name}_to_${prefix}${frame_id.rstrip('_link')}_joint" type="fixed">
       <origin xyz="0.0 0.0 0.031" rpy="0.0 0.0 ${pi}" />
       <parent link="${prefix}${name}_link" />
@@ -122,6 +120,5 @@
       </gazebo>
       <gazebo>
-        <plugin filename="libignition-gazebo-sensors-system.so"
-          name="ignition::gazebo::systems::Sensors">
+        <plugin filename="libignition-gazebo-sensors-system.so" name="ignition::gazebo::systems::Sensors">
           <render_engine>ogre2</render_engine>
         </plugin>

File: urdf/slamtec_rplidar_a3.urdf.xacro (robot description, xacro)
@@ -27,10 +27,11 @@
       </xacro:if>
     </xacro:unless>
-    <xacro:property name="prefix" value="${tf_prefix}" lazy_eval="false" />
-    <xacro:if value="${prefix != ''}">
+    <xacro:if value="${tf_prefix == ''}">
+      <xacro:property name="prefix" value="" />
+    </xacro:if>
+    <xacro:unless value="${tf_prefix == ''}">
       <xacro:property name="prefix" value="${tf_prefix}_" />
-    </xacro:if>
-    <joint name="${parent_link.rstrip('_link')}_to_${prefix}${name}_joint"
-      type="fixed">
+    </xacro:unless>
+    <joint name="${parent_link.rstrip('_link')}_to_${prefix}${name}_joint" type="fixed">
       <origin xyz="${xyz}" rpy="${rpy}" />
       <parent link="${parent_link}" />
@@ -59,7 +60,5 @@
       </inertial>
     </link>
-    <joint
-      name="${prefix}${name}_to_${prefix}${frame_id.rstrip('_link')}_joint"
-      type="fixed">
+    <joint name="${prefix}${name}_to_${prefix}${frame_id.rstrip('_link')}_joint" type="fixed">
       <origin xyz="0.0 0.0 0.031" rpy="0.0 0.0 ${pi}" />
       <parent link="${prefix}${name}_link" />
@@ -100,6 +99,5 @@
       </gazebo>
       <gazebo>
-        <plugin filename="libignition-gazebo-sensors-system.so"
-          name="ignition::gazebo::systems::Sensors">
+        <plugin filename="libignition-gazebo-sensors-system.so" name="ignition::gazebo::systems::Sensors">
           <render_engine>ogre2</render_engine>
         </plugin>

File: urdf/slamtec_rplidar_s1.urdf.xacro (robot description, xacro)
@@ -27,8 +27,10 @@
       </xacro:if>
     </xacro:unless>
-    <xacro:property name="prefix" value="${tf_prefix}" lazy_eval="false" />
-    <xacro:if value="${prefix != ''}">
+    <xacro:if value="${tf_prefix == ''}">
+      <xacro:property name="prefix" value="" />
+    </xacro:if>
+    <xacro:unless value="${tf_prefix == ''}">
       <xacro:property name="prefix" value="${tf_prefix}_" />
-    </xacro:if>
+    </xacro:unless>
     <joint name="${parent_link.rstrip('_link')}_to_${prefix}${name}_joint"
       type="fixed">

File: urdf/stereolabs_zed.urdf.xacro (robot description, xacro)
@@ -24,8 +24,10 @@
             use_nominal_extrinsics:=false
             simulation_engine:=ignition-gazebo">
-    <xacro:property name="prefix" value="${tf_prefix}" lazy_eval="false" />
-    <xacro:if value="${prefix != ''}">
+    <xacro:if value="${tf_prefix == ''}">
+      <xacro:property name="prefix" value="" />
+    </xacro:if>
+    <xacro:unless value="${tf_prefix == ''}">
       <xacro:property name="prefix" value="${tf_prefix}_" />
-    </xacro:if>
+    </xacro:unless>
     <xacro:if value="${model == 'zed'}">
       <xacro:property name="baseline" value="0.12" />

File: urdf/velodyne_puck.urdf.xacro (robot description, xacro)
@@ -17,8 +17,10 @@
       <xacro:property name="plugin_file_name" value="libgazebo_ros_velodyne_laser.so" />
     </xacro:unless>
-    <xacro:property name="prefix" value="${tf_prefix}" lazy_eval="false" />
-    <xacro:if value="${prefix != ''}">
+    <xacro:if value="${tf_prefix == ''}">
+      <xacro:property name="prefix" value="" />
+    </xacro:if>
+    <xacro:unless value="${tf_prefix == ''}">
       <xacro:property name="prefix" value="${tf_prefix}_" />
-    </xacro:if>
+    </xacro:unless>
     <joint name="${parent_link.rstrip('_link')}_to_${prefix}${name}_joint" type="fixed">
       <origin xyz="${xyz}" rpy="${rpy}" />

Commit message: undo none

File: urdf/intel_realsense_d435.urdf.xacro (robot description, xacro)
@@ -19,13 +19,13 @@
   <xacro:macro name="intel_realsense_d435"
     params="parent_link xyz rpy
-            tf_prefix:=''
+            tf_prefix:=None
             name:=camera
             topic:=camera
             use_nominal_extrinsics:=false
             simulation_engine:=ignition-gazebo">
-    <xacro:if value="${tf_prefix == ''}">
+    <xacro:if value="${tf_prefix == 'None'}">
       <xacro:property name="prefix" value="" />
     </xacro:if>
-    <xacro:unless value="${tf_prefix == ''}">
+    <xacro:unless value="${tf_prefix == 'None'}">
       <xacro:property name="prefix" value="${tf_prefix}_" />
     </xacro:unless>

File: urdf/orbbec_astra.urdf.xacro (robot description, xacro)
@@ -3,12 +3,12 @@
   <xacro:macro name="orbbec_astra"
                params="parent_link xyz rpy
-                       tf_prefix:=''
+                       tf_prefix:=None
                        name:=camera
                        topic:=camera
                        simulation_engine:=ignition-gazebo">
-    <xacro:if value="${tf_prefix == ''}">
+    <xacro:if value="${tf_prefix == 'None'}">
       <xacro:property name="prefix" value="" />
     </xacro:if>
-    <xacro:unless value="${tf_prefix == ''}">
+    <xacro:unless value="${tf_prefix == 'None'}">
       <xacro:property name="prefix" value="${tf_prefix}_" />
     </xacro:unless>
@@ -53,6 +53,5 @@
     </joint>
     <link name="${prefix}${name}_depth_frame" />
-    <joint name="${parent_link.rstrip('_link')}_to_${prefix}${name}_depth_joint"
-      type="fixed">
+    <joint name="${parent_link.rstrip('_link')}_to_${prefix}${name}_depth_joint" type="fixed">
       <origin xyz="0.0 0.0 0.03325" rpy="0.0 0.0 0.0" />
       <parent link="${parent_link}" />
@@ -66,7 +65,5 @@
     </joint>
     <link name="${prefix}${name}_depth_optical_frame" />
-    <joint
-      name="${prefix}${name}_depth_to_${prefix}${name}_depth_optical_joint"
-      type="fixed">
+    <joint name="${prefix}${name}_depth_to_${prefix}${name}_depth_optical_joint" type="fixed">
       <origin xyz="0.0 0.0 0.0" rpy="${-pi/2} 0.0 ${-pi/2}" />
       <parent link="${prefix}${name}_depth_frame" />

File: urdf/ouster_os1_32.urdf.xacro (robot description, xacro)
@@ -4,5 +4,5 @@
     params="parent_link xyz rpy
             use_gpu:=false
-            tf_prefix:=''
+            tf_prefix:=None
             name:=ouster_os1_32
             topic:=os_lidar
@@ -17,8 +17,8 @@
       <xacro:property name="plugin_file_name" value="libgazebo_ros_velodyne_laser.so" />
     </xacro:unless>
-    <xacro:if value="${tf_prefix == ''}">
+    <xacro:if value="${tf_prefix == 'None'}">
       <xacro:property name="prefix" value="" />
     </xacro:if>
-    <xacro:unless value="${tf_prefix == ''}">
+    <xacro:unless value="${tf_prefix == 'None'}">
       <xacro:property name="prefix" value="${tf_prefix}_" />
     </xacro:unless>
@@ -62,5 +62,5 @@
           <scan>
             <horizontal>
-              <samples>2048</samples>
+              <samples>1024</samples>
               <resolution>1</resolution>
               <min_angle>-${pi}</min_angle>

File: urdf/slamtec_rplidar_a2.urdf.xacro (robot description, xacro)
@@ -9,5 +9,5 @@
     params="parent_link xyz rpy
             use_gpu:=false
-            tf_prefix:=''
+            tf_prefix:=None
             name:=slamtec_rplidar_a2
             topic:=scan
@@ -33,8 +33,8 @@
       </xacro:if>
     </xacro:unless>
-    <xacro:if value="${tf_prefix == ''}">
+    <xacro:if value="${tf_prefix == 'None'}">
       <xacro:property name="prefix" value="" />
     </xacro:if>
-    <xacro:unless value="${tf_prefix == ''}">
+    <xacro:unless value="${tf_prefix == 'None'}">
       <xacro:property name="prefix" value="${tf_prefix}_" />
     </xacro:unless>

File: urdf/slamtec_rplidar_a3.urdf.xacro (robot description, xacro)
@@ -4,5 +4,5 @@
     params="parent_link xyz rpy
             use_gpu:=false
-            tf_prefix:=''
+            tf_prefix:=None
             name:=slamtec_rplidar_a3
             topic:=scan
@@ -27,8 +27,8 @@
       </xacro:if>
     </xacro:unless>
-    <xacro:if value="${tf_prefix == ''}">
+    <xacro:if value="${tf_prefix == 'None'}">
       <xacro:property name="prefix" value="" />
     </xacro:if>
-    <xacro:unless value="${tf_prefix == ''}">
+    <xacro:unless value="${tf_prefix == 'None'}">
       <xacro:property name="prefix" value="${tf_prefix}_" />
     </xacro:unless>

File: urdf/slamtec_rplidar_s1.urdf.xacro (robot description, xacro)
@@ -4,5 +4,5 @@
     params="parent_link xyz rpy
             use_gpu:=false
-            tf_prefix:=''
+            tf_prefix:=None
             name:=slamtec_rplidar_s1
             topic:=scan
@@ -27,12 +27,11 @@
       </xacro:if>
     </xacro:unless>
-    <xacro:if value="${tf_prefix == ''}">
+    <xacro:if value="${tf_prefix == 'None'}">
       <xacro:property name="prefix" value="" />
     </xacro:if>
-    <xacro:unless value="${tf_prefix == ''}">
+    <xacro:unless value="${tf_prefix == 'None'}">
       <xacro:property name="prefix" value="${tf_prefix}_" />
     </xacro:unless>
-    <joint name="${parent_link.rstrip('_link')}_to_${prefix}${name}_joint"
-      type="fixed">
+    <joint name="${parent_link.rstrip('_link')}_to_${prefix}${name}_joint" type="fixed">
       <origin xyz="${xyz}" rpy="${rpy}" />
       <parent link="${parent_link}" />
@@ -68,7 +67,5 @@
       </inertial>
     </link>
-    <joint
-      name="${prefix}${name}_to_${prefix}${frame_id.rstrip('_link')}_joint"
-      type="fixed">
+    <joint name="${prefix}${name}_to_${prefix}${frame_id.rstrip('_link')}_joint" type="fixed">
       <origin xyz="0.0 0.0 0.04" rpy="0.0 0.0 ${pi}" />
       <parent link="${prefix}${name}_link" />
@@ -107,6 +104,5 @@
       </gazebo>
       <gazebo>
-        <plugin filename="libignition-gazebo-sensors-system.so"
-          name="ignition::gazebo::systems::Sensors">
+        <plugin filename="libignition-gazebo-sensors-system.so" name="ignition::gazebo::systems::Sensors">
           <render_engine>ogre2</render_engine>
         </plugin>

File: urdf/stereolabs_zed.urdf.xacro (robot description, xacro)
@@ -19,13 +19,13 @@
   <xacro:macro name="zed_camera"
     params="parent_link xyz rpy
-            tf_prefix:=''
+            tf_prefix:=None
             name:=camera
             topic:=zed
             model:=zed
             simulation_engine:=ignition-gazebo">
-    <xacro:if value="${tf_prefix == ''}">
+    <xacro:if value="${tf_prefix == 'None'}">
       <xacro:property name="prefix" value="" />
     </xacro:if>
-    <xacro:unless value="${tf_prefix == ''}">
+    <xacro:unless value="${tf_prefix == 'None'}">
       <xacro:property name="prefix" value="${tf_prefix}_" />
     </xacro:unless>
@@ -165,6 +165,6 @@
       camera
         should be more accurate different frames and fovs can be set -->
-        <gazebo reference="${prefix}${name}_center_optical_frame">
-          <sensor type="rgbd" name="${prefix}${name}_color">
+      <gazebo reference="${prefix}${name}_center_optical_frame">
+        <sensor type="rgbd" name="${prefix}${name}_color">
           <always_on>true</always_on>
           <update_rate>30.0</update_rate>

File: urdf/velodyne_puck.urdf.xacro (robot description, xacro)
@@ -4,5 +4,5 @@
     params="parent_link xyz rpy
             use_gpu:=false
-            tf_prefix:=''
+            tf_prefix:=None
             name:=velodyne_puck
             topic:=scan
@@ -17,8 +17,8 @@
       <xacro:property name="plugin_file_name" value="libgazebo_ros_velodyne_laser.so" />
     </xacro:unless>
-    <xacro:if value="${tf_prefix == ''}">
+    <xacro:if value="${tf_prefix == 'None'}">
       <xacro:property name="prefix" value="" />
     </xacro:if>
-    <xacro:unless value="${tf_prefix == ''}">
+    <xacro:unless value="${tf_prefix == 'None'}">
       <xacro:property name="prefix" value="${tf_prefix}_" />
     </xacro:unless>

Commit message: add suggestions

File: urdf/intel_realsense_d435.urdf.xacro (robot description, xacro)
@@ -21,5 +21,6 @@
             tf_prefix:=None
             name:=camera
-            topic:=camera
+            topic_rgb_camera:=camera/color/image_raw
+            topic_depth_camera:=camera/depth
             use_nominal_extrinsics:=false
             simulation_engine:=ignition-gazebo">
@@ -158,5 +159,5 @@
           <always_on>true</always_on>
           <update_rate>30.0</update_rate>
-          <topic>${topic}/color/image_raw</topic>
+          <topic>${topic_rgb_camera}</topic>
           <visualize>false</visualize>
           <ignition_frame_id>${prefix}${name}_color_optical_frame</ignition_frame_id>
@@ -175,5 +176,5 @@
           <always_on>true</always_on>
           <update_rate>30.0</update_rate>
-          <topic>${topic}/depth</topic>
+          <topic>${topic_depth_camera}</topic>
           <visualize>false</visualize>
           <!-- Depth cannot be optical becaues it roatate output -->

File: urdf/orbbec_astra.urdf.xacro (robot description, xacro)
@@ -13,10 +13,10 @@
       <xacro:property name="prefix" value="${tf_prefix}_" />
     </xacro:unless>
-    <joint name="${parent_link.rstrip('_link')}_to_${prefix}${name}_orbbec_astra_joint" type="fixed">
+    <joint name="${parent_link.rstrip('_link')}_to_${prefix}${name}_visualization_joint" type="fixed">
       <origin xyz="${xyz}" rpy="${rpy}" />
       <parent link="${parent_link}" />
-      <child link="${prefix}${name}_orbbec_astra_link" />
+      <child link="${prefix}${name}_visualization_link" />
     </joint>
-    <link name="${prefix}${name}_orbbec_astra_link">
+    <link name="${prefix}${name}_visualization_link">
       <visual>
         <origin xyz="0.0 0.0 0.0" rpy="0.0 0.0 0.0" />

File: urdf/stereolabs_zed.urdf.xacro (robot description, xacro)
@@ -21,6 +21,6 @@
             tf_prefix:=None
             name:=zed
-            topic:=zed
-            model:=zed
+            topic_rgb_camera:=zed/zed_node/rgb/image_rect_color
+            topic_depth_camera:=zed/zed_node/depth            model:=zed
             simulation_engine:=ignition-gazebo">
     <xacro:if value="${tf_prefix == 'None'}">
@@ -169,5 +169,5 @@
           <always_on>true</always_on>
           <update_rate>30.0</update_rate>
-          <topic>${topic}/zed_node/rgb/image_rect_color</topic>
+          <topic>${topic_rgb_camera}</topic>
           <visualize>false</visualize>
           <ignition_frame_id>${prefix}${name}_left_camera_optical_frame</ignition_frame_id>
@@ -188,5 +188,5 @@
           <always_on>true</always_on>
           <update_rate>30.0</update_rate>
-          <topic>${topic}/zed_node/depth</topic>
+          <topic>${topic_depth_camera}</topic>
           <visualize>false</visualize>
           <!-- Depth cannot be optical becaues it roatate output Point Cloud -->
