Commit message: Maciej suggestions

File: urdf/intel_realsense_d435.urdf.xacro (robot description, xacro)
@@ -21,6 +21,5 @@
             tf_prefix:=None
             name:=camera
-            topic_rgb_camera:=camera/color/image_raw
-            topic_depth_camera:=camera/depth
+            topic_ns:=camera
             use_nominal_extrinsics:=false
             simulation_engine:=ignition-gazebo">
@@ -74,5 +73,5 @@
         <origin xyz="0.0 0.0 0.0" rpy="0.0 0.0 0.0" />
         <geometry>
-          <mesh filename="package://ros_components_description/meshes/intel_realsense_d435.dae" />
+          <mesh filename="file://$(find ros_components_description)/meshes/intel_realsense_d435.dae" />
         </geometry>
       </visual>
@@ -159,5 +158,5 @@
           <always_on>true</always_on>
           <update_rate>30.0</update_rate>
-          <topic>${topic_rgb_camera}</topic>
+          <topic>${topic_ns}/color/image_raw</topic>
           <visualize>false</visualize>
           <ignition_frame_id>${prefix}${name}_color_optical_frame</ignition_frame_id>
@@ -176,5 +175,5 @@
           <always_on>true</always_on>
           <update_rate>30.0</update_rate>
-          <topic>${topic_depth_camera}</topic>
+          <topic>${topic_ns}/depth</topic>
           <visualize>false</visualize>
           <!-- Depth cannot be optical becaues it roatate output -->

File: urdf/orbbec_astra.urdf.xacro (robot description, xacro)
@@ -5,5 +5,5 @@
             tf_prefix:=None
             name:=camera
-            topic:=camera
+            topic_ns:=camera
             simulation_engine:=ignition-gazebo">
     <xacro:if value="${tf_prefix == 'None'}">
@@ -76,5 +76,5 @@
           <always_on>true</always_on>
           <update_rate>20.0</update_rate>
-          <topic>${topic}</topic>
+          <topic>${topic_ns}</topic>
           <!-- It is not possible to split the frame of the color and the depth stream.
                The frame of color stream should be ${prefix}${name}_color_optical_frame, but adding optical rotate pointcloud -->

File: urdf/ouster_os1_32.urdf.xacro (robot description, xacro)
@@ -6,5 +6,5 @@
             tf_prefix:=None
             name:=ouster_os1_32
-            topic:=os_lidar
+            topic_ns:=os_lidar
             frame_id:=os_lidar
             simulation_engine:=ignition-gazebo">
@@ -86,5 +86,5 @@
         </ray>
         <xacro:if value="${simulation_engine == 'ignition-gazebo'}">
-          <topic>${topic}</topic>
+          <topic>${topic_ns}</topic>
           <ignition_frame_id>${prefix}${frame_id}</ignition_frame_id>
           <always_on>true</always_on>
@@ -98,5 +98,5 @@
             <ros>
               <namespace></namespace>
-              <remapping>~/out:=${topic}</remapping>
+              <remapping>~/out:=${topic_ns}</remapping>
             </ros>
             <output_type>sensor_msgs/PointCloud2</output_type>

File: urdf/slamtec_rplidar_a2.urdf.xacro (robot description, xacro)
@@ -11,5 +11,5 @@
             tf_prefix:=None
             name:=slamtec_rplidar_a2
-            topic:=scan
+            topic_ns:=scan
             frame_id:=laser
             model:=A2M12
@@ -91,5 +91,5 @@
       <gazebo reference="${prefix}${frame_id}">
         <sensor type="${ray_type}" name="${prefix}${name}_sensor">
-          <topic>${topic}</topic>
+          <topic>${topic_ns}</topic>
           <ignition_frame_id>${prefix}${frame_id}</ignition_frame_id>
           <update_rate>10.0</update_rate>
@@ -152,5 +152,5 @@
             <ros>
               <namespace></namespace>
-              <remapping>~/out:=${topic}</remapping>
+              <remapping>~/out:=${topic_ns}</remapping>
             </ros>
             <output_type>sensor_msgs/LaserScan</output_type>

File: urdf/slamtec_rplidar_a3.urdf.xacro (robot description, xacro)
@@ -6,5 +6,5 @@
             tf_prefix:=None
             name:=slamtec_rplidar_a3
-            topic:=scan
+            topic_ns:=scan
             frame_id:=laser
             simulation_engine:=ignition-gazebo">
@@ -69,5 +69,5 @@
       <gazebo reference="${prefix}${frame_id}">
         <sensor type="${ray_type}" name="${prefix}${name}_sensor">
-          <topic>${topic}</topic>
+          <topic>${topic_ns}</topic>
           <frame_id>${prefix}${frame_id}</frame_id>
           <ignition_frame_id>${prefix}${frame_id}</ignition_frame_id>
@@ -133,5 +133,5 @@
             <ros>
               <namespace></namespace>
-              <remapping>~/out:=${topic}</remapping>
+              <remapping>~/out:=${topic_ns}</remapping>
             </ros>
             <output_type>sensor_msgs/LaserScan</output_type>

File: urdf/slamtec_rplidar_s1.urdf.xacro (robot description, xacro)
@@ -6,5 +6,5 @@
             tf_prefix:=None
             name:=slamtec_rplidar_s1
-            topic:=scan
+            topic_ns:=scan
             frame_id:=laser
             simulation_engine:=ignition-gazebo">
@@ -76,5 +76,5 @@
       <gazebo reference="${prefix}${frame_id}">
         <sensor type="${ray_type}" name="${prefix}${name}_sensor">
-          <topic>${topic}</topic>
+          <topic>${topic_ns}</topic>
           <ignition_frame_id>${prefix}${frame_id}</ignition_frame_id>
           <update_rate>10.0</update_rate>
@@ -137,5 +137,5 @@
             <ros>
               <namespace></namespace>
-              <remapping>~/out:=${topic}</remapping>
+              <remapping>~/out:=${topic_ns}</remapping>
             </ros>
             <output_type>sensor_msgs/LaserScan</output_type>

File: urdf/slamtec_rplidar_s2.urdf.xacro (robot description, xacro)
@@ -6,5 +6,5 @@
             tf_prefix:=None
             name:=slamtec_rplidar_s2
-            topic:=scan
+            topic_ns:=scan
             frame_id:=laser
             simulation_engine:=ignition-gazebo">
@@ -69,5 +69,5 @@
       <gazebo reference="${prefix}${frame_id}">
         <sensor type="${ray_type}" name="${prefix}rplidar_s2_sensor">
-          <topic>${topic}</topic>
+          <topic>${topic_ns}</topic>
           <frame_id>${prefix}${frame_id}</frame_id>
           <ignition_frame_id>${prefix}${frame_id}</ignition_frame_id>
@@ -131,5 +131,5 @@
             <ros>
               <namespace></namespace>
-              <remapping>~/out:=${topic}</remapping>
+              <remapping>~/out:=${topic_ns}</remapping>
             </ros>
             <output_type>sensor_msgs/LaserScan</output_type>

File: urdf/slamtec_rplidar_s3.urdf.xacro (robot description, xacro)
@@ -6,5 +6,5 @@
             tf_prefix:=None
             name:=slamtec_rplidar_s3
-            topic:=scan
+            topic_ns:=scan
             frame_id:=laser
             simulation_engine:=ignition-gazebo">
@@ -69,5 +69,5 @@
       <gazebo reference="${prefix}${frame_id}">
         <sensor type="${ray_type}" name="${prefix}rplidar_s3_sensor">
-          <topic>${topic}</topic>
+          <topic>${topic_ns}</topic>
           <frame_id>${prefix}${frame_id}</frame_id>
           <ignition_frame_id>${prefix}${frame_id}</ignition_frame_id>
@@ -131,5 +131,5 @@
             <ros>
               <namespace></namespace>
-              <remapping>~/out:=${topic}</remapping>
+              <remapping>~/out:=${topic_ns}</remapping>
             </ros>
             <output_type>sensor_msgs/LaserScan</output_type>

File: urdf/stereolabs_zed.urdf.xacro (robot description, xacro)
@@ -21,6 +21,6 @@
             tf_prefix:=None
             name:=zed
-            topic_rgb_camera:=zed/zed_node/rgb/image_rect_color
-            topic_depth_camera:=zed/zed_node/depth            model:=zed
+            topic_ns:=zed
+            model:=zed
             simulation_engine:=ignition-gazebo">
     <xacro:if value="${tf_prefix == 'None'}">
@@ -90,5 +90,5 @@
         <origin xyz="${screw_offset_x} 0 ${screw_offset_z}" rpy="0 0 0" />
         <geometry>
-          <mesh filename="package://ros_components_description/meshes/${model}.stl" />
+          <mesh filename="file://$(find ros_components_description)/meshes/${model}.stl" />
         </geometry>
         <material name="mat">
@@ -98,5 +98,5 @@
       <collision>
         <geometry>
-          <mesh filename="package://ros_components_description/meshes/${model}.stl" />
+          <mesh filename="file://$(find ros_components_description)/meshes/${model}.stl" />
         </geometry>
       </collision>
@@ -169,5 +169,5 @@
           <always_on>true</always_on>
           <update_rate>30.0</update_rate>
-          <topic>${topic_rgb_camera}</topic>
+          <topic>${topic_ns_ns}/zed_node/rgb/image_rect_color</topic>
           <visualize>false</visualize>
           <ignition_frame_id>${prefix}${name}_left_camera_optical_frame</ignition_frame_id>
@@ -188,5 +188,5 @@
           <always_on>true</always_on>
           <update_rate>30.0</update_rate>
-          <topic>${topic_depth_camera}</topic>
+          <topic>${topic_ns_ns}/zed_node/depth</topic>
           <visualize>false</visualize>
           <!-- Depth cannot be optical becaues it roatate output Point Cloud -->

File: urdf/velodyne_puck.urdf.xacro (robot description, xacro)
@@ -6,5 +6,5 @@
             tf_prefix:=None
             name:=velodyne_puck
-            topic:=scan
+            topic_ns:=scan
             frame_id:=velodyne
             simulation_engine:=ignition-gazebo">
@@ -87,5 +87,5 @@
         </ray>
         <xacro:if value="${simulation_engine == 'ignition-gazebo'}">
-          <topic>${topic}</topic>
+          <topic>${topic_ns}</topic>
           <frame_id>${prefix}${frame_id}</frame_id>
           <ignition_frame_id>${prefix}${frame_id}</ignition_frame_id>
@@ -101,5 +101,5 @@
             <ros>
               <namespace></namespace>
-              <remapping>~/out:=${topic}</remapping>
+              <remapping>~/out:=${topic_ns}</remapping>
             </ros>
             <output_type>sensor_msgs/PointCloud2</output_type>
