Commit message: Revert "Add prefix (#36)"
This reverts commit 4f1bc6fab4fd327a2d0f44dccfa7138ba06fbe95.

File: urdf/intel_realsense_d435.urdf.xacro (robot description, xacro)
@@ -16,18 +16,11 @@
 # limitations under the License.
 -->
-<robot name="intel_realsense_d435" xmlns:xacro="http://ros.org/wiki/xacro">
+<robot name="intel_camera" xmlns:xacro="http://ros.org/wiki/xacro">
   <xacro:macro name="intel_realsense_d435"
     params="parent_link xyz rpy
-            tf_prefix:=None
             name:=camera
             topic:=camera
             use_nominal_extrinsics:=false
             simulation_engine:=ignition-gazebo">
-    <xacro:if value="${tf_prefix == 'None'}">
-      <xacro:property name="prefix" value="" />
-    </xacro:if>
-    <xacro:unless value="${tf_prefix == 'None'}">
-      <xacro:property name="prefix" value="${tf_prefix}_" />
-    </xacro:unless>
     <!-- The following values are approximate, and the camera node
       publishing TF values with actual calibrated camera extrinsic values -->
@@ -56,17 +49,17 @@
     <xacro:property name="d435_cam_depth_pz" value="${d435_cam_height/2}" />
     <!-- camera body, with origin at bottom screw mount -->
-    <joint name="${parent_link.rstrip('_link')}_to_${prefix}${name}_bottom_screw_joint" type="fixed">
+    <joint name="${parent_link.rstrip('_link')}_to_${name}_bottom_screw_joint" type="fixed">
       <origin xyz="${xyz}" rpy="${rpy}" />
       <parent link="${parent_link}" />
-      <child link="${prefix}${name}_bottom_screw_frame" />
+      <child link="${name}_bottom_screw_frame" />
     </joint>
-    <link name="${prefix}${name}_bottom_screw_frame" />
-    <joint name="${prefix}${name}_bottom_screw_to_${prefix}${name}_joint" type="fixed">
+    <link name="${name}_bottom_screw_frame" />
+    <joint name="${name}_bottom_screw_to_${name}_joint" type="fixed">
       <origin xyz="${d435_mesh_x_offset} ${d435_cam_depth_py} ${d435_cam_depth_pz}"
         rpy="0.0 0.0 0.0" />
-      <parent link="${prefix}${name}_bottom_screw_frame" />
-      <child link="${prefix}${name}_link" />
+      <parent link="${name}_bottom_screw_frame" />
+      <child link="${name}_link" />
     </joint>
-    <link name="${prefix}${name}_link">
+    <link name="${name}_link">
       <visual>
         <origin xyz="0.0 0.0 0.0" rpy="0.0 0.0 0.0" />
@@ -94,66 +87,66 @@
     <xacro:if value="${use_nominal_extrinsics}">
       <!-- camera depth joints and links -->
-      <joint name="${prefix}${name}_to_${prefix}${name}_depth_joint" type="fixed">
+      <joint name="${name}_to_${name}_depth_joint" type="fixed">
         <origin xyz="0.0 0.0 0.0" rpy="0.0 0.0 0.0" />
-        <parent link="${prefix}${name}_link" />
-        <child link="${prefix}${name}_depth_frame" />
+        <parent link="${name}_link" />
+        <child link="${name}_depth_frame" />
       </joint>
-      <link name="${prefix}${name}_depth_frame" />
-      <joint name="${prefix}${name}_depth_to_${prefix}${name}_depth_optical_joint" type="fixed">
+      <link name="${name}_depth_frame" />
+      <joint name="${name}_depth_to_${name}_depth_optical_joint" type="fixed">
         <origin xyz="0.0 0.0 0.0" rpy="${-pi/2.0} 0.0 ${-pi/2.0}" />
-        <parent link="${prefix}${name}_depth_frame" />
-        <child link="${prefix}${name}_depth_optical_frame" />
+        <parent link="${name}_depth_frame" />
+        <child link="${name}_depth_optical_frame" />
       </joint>
-      <link name="${prefix}${name}_depth_optical_frame" />
+      <link name="${name}_depth_optical_frame" />
       <!-- camera left IR joints and links -->
-      <joint name="${prefix}${name}_to_${prefix}${name}_infra1_joint" type="fixed">
+      <joint name="${name}_to_${name}_infra1_joint" type="fixed">
         <origin xyz="0.0 ${d435_cam_depth_to_infra1_offset} 0.0" rpy="0.0 0.0 0.0" />
-        <parent link="${prefix}${name}_link" />
-        <child link="${prefix}${name}_infra1_frame" />
+        <parent link="${name}_link" />
+        <child link="${name}_infra1_frame" />
       </joint>
-      <link name="${prefix}${name}_infra1_frame" />
-      <joint name="${prefix}${name}_infra1_to_${prefix}${name}_infra1_optical_joint" type="fixed">
+      <link name="${name}_infra1_frame" />
+      <joint name="${name}_infra1_to_${name}_infra1_optical_joint" type="fixed">
         <origin xyz="0.0 0.0 0.0" rpy="${-pi/2.0} 0.0 ${-pi/2.0}" />
-        <parent link="${prefix}${name}_infra1_frame" />
-        <child link="${prefix}${name}_infra1_optical_frame" />
+        <parent link="${name}_infra1_frame" />
+        <child link="${name}_infra1_optical_frame" />
       </joint>
-      <link name="${prefix}${name}_infra1_optical_frame" />
+      <link name="${name}_infra1_optical_frame" />
       <!-- camera right IR joints and links -->
-      <joint name="${prefix}${name}_to_${prefix}${name}_infra2_joint" type="fixed">
+      <joint name="${name}_to_${name}_infra2_joint" type="fixed">
         <origin xyz="0.0 ${d435_cam_depth_to_infra2_offset} 0.0" rpy="0.0 0.0 0.0" />
-        <parent link="${prefix}${name}_link" />
-        <child link="${prefix}${name}_infra2_frame" />
+        <parent link="${name}_link" />
+        <child link="${name}_infra2_frame" />
       </joint>
-      <link name="${prefix}${name}_infra2_frame" />
-      <joint name="${prefix}${name}_infra2_to_${prefix}${name}_infra2_optical_joint" type="fixed">
+      <link name="${name}_infra2_frame" />
+      <joint name="${name}_infra2_to_${name}_infra2_optical_joint" type="fixed">
         <origin xyz="0.0 0.0 0.0" rpy="${-pi/2.0} 0.0 ${-pi/2.0}" />
-        <parent link="${prefix}${name}_infra2_frame" />
-        <child link="${prefix}${name}_infra2_optical_frame" />
+        <parent link="${name}_infra2_frame" />
+        <child link="${name}_infra2_optical_frame" />
       </joint>
-      <link name="${prefix}${name}_infra2_optical_frame" />
+      <link name="${name}_infra2_optical_frame" />
       <!-- camera color joints and links -->
-      <joint name="${prefix}${name}_to_${prefix}${name}_color_joint" type="fixed">
+      <joint name="${name}_to_${name}_color_joint" type="fixed">
         <origin xyz="0.0 ${d435_cam_depth_to_color_offset} 0.0" rpy="0.0 0.0 0.0" />
-        <parent link="${prefix}${name}_link" />
-        <child link="${prefix}${name}_color_frame" />
+        <parent link="${name}_link" />
+        <child link="${name}_color_frame" />
       </joint>
-      <link name="${prefix}${name}_color_frame" />
-      <joint name="${prefix}${name}_color_to_${prefix}${name}_color_optical_joint" type="fixed">
+      <link name="${name}_color_frame" />
+      <joint name="${name}_color_to_${name}_color_optical_joint" type="fixed">
         <origin xyz="0.0 0.0 0.0" rpy="${-pi/2.0} 0.0 ${-pi/2.0}" />
-        <parent link="${prefix}${name}_color_frame" />
-        <child link="${prefix}${name}_color_optical_frame" />
+        <parent link="${name}_color_frame" />
+        <child link="${name}_color_optical_frame" />
       </joint>
-      <link name="${prefix}${name}_color_optical_frame" />
+      <link name="${name}_color_optical_frame" />
     </xacro:if>
     <xacro:if value="${simulation_engine == 'ignition-gazebo'}">
       <!-- It is also possible to use single rgbd_camera sensor, but using separate rgb and depth camera
         should be more accurate for D435 - different frames and fovs can be set -->
-      <gazebo reference="${prefix}${name}_link">
-        <sensor type="camera" name="${prefix}${name}_color">
+      <gazebo reference="${name}_link">
+        <sensor type="camera" name="${name}_color">
           <always_on>true</always_on>
           <update_rate>30.0</update_rate>
           <topic>${topic}/color/image_raw</topic>
           <visualize>false</visualize>
-          <ignition_frame_id>${prefix}${name}_color_optical_frame</ignition_frame_id>
+          <ignition_frame_id>${name}_color_optical_frame</ignition_frame_id>
           <horizontal_fov>${69.0/180.0*pi}</horizontal_fov>
           <image>
@@ -167,10 +160,10 @@
           </clip>
         </sensor>
-        <sensor type="depth_camera" name="${prefix}${name}_depth">
+        <sensor type="depth_camera" name="${name}_depth">
           <always_on>true</always_on>
           <update_rate>30.0</update_rate>
           <topic>${topic}/depth</topic>
           <visualize>false</visualize>
-          <ignition_frame_id>${prefix}${name}_depth_optical_frame</ignition_frame_id>
+          <ignition_frame_id>${name}_depth_optical_frame</ignition_frame_id>
           <camera>
             <horizontal_fov>${87.0/180.0*pi}</horizontal_fov>

File: urdf/orbbec_astra.urdf.xacro (robot description, xacro)
@@ -7,15 +7,15 @@
                        simulation_engine:=gazebo-classic">
     <xacro:if value="${tf_prefix == 'None'}">
-      <xacro:property name="prefix" value="" />
+      <xacro:property name="tf_prefix_ext" value="" />
     </xacro:if>
     <xacro:unless value="${tf_prefix == 'None'}">
-      <xacro:property name="prefix" value="${tf_prefix}_" />
+      <xacro:property name="tf_prefix_ext" value="${tf_prefix}_" />
     </xacro:unless>
-    <joint name="${parent_link.rstrip('_link')}_to_${prefix}${camera_name}_orbbec_astra_joint" type="fixed">
+    <joint name="${parent_link.rstrip('_link')}_to_${tf_prefix_ext}${camera_name}_orbbec_astra_joint" type="fixed">
       <origin xyz="${xyz}" rpy="${rpy}" />
       <parent link="${parent_link}" />
-      <child link="${prefix}${camera_name}_orbbec_astra_link" />
+      <child link="${tf_prefix_ext}${camera_name}_orbbec_astra_link" />
     </joint>
-    <link name="${prefix}${camera_name}_orbbec_astra_link">
+    <link name="${tf_prefix_ext}${camera_name}_orbbec_astra_link">
       <visual>
         <origin xyz="0.0 0.0 0.0" rpy="0.0 0.0 0.0" />
@@ -46,38 +46,38 @@
       </inertial>
     </link>
-    <joint name="${parent_link.rstrip('_link')}_to_${prefix}${camera_name}_color_joint" type="fixed">
+    <joint name="${parent_link.rstrip('_link')}_to_${tf_prefix_ext}${camera_name}_color_joint" type="fixed">
       <origin xyz="-0.002 0.0125 0.03325" rpy="-0.003 0.0 -0.003" />
       <parent link="${parent_link}" />
-      <child link="${prefix}${camera_name}_color_frame" />
+      <child link="${tf_prefix_ext}${camera_name}_color_frame" />
     </joint>
-    <link name="${prefix}${camera_name}_depth_frame" />
-    <joint name="${parent_link.rstrip('_link')}_to_${prefix}${camera_name}_depth_joint" type="fixed">
+    <link name="${tf_prefix_ext}${camera_name}_depth_frame" />
+    <joint name="${parent_link.rstrip('_link')}_to_${tf_prefix_ext}${camera_name}_depth_joint" type="fixed">
       <origin xyz="0.0 0.0 0.03325" rpy="0.0 0.0 0.0" />
       <parent link="${parent_link}" />
-      <child link="${prefix}${camera_name}_depth_frame" />
+      <child link="${tf_prefix_ext}${camera_name}_depth_frame" />
     </joint>
-    <link name="${prefix}${camera_name}_color_frame" />
-    <joint name="${prefix}${camera_name}_color_to_${prefix}${camera_name}_color_optical_joint" type="fixed">
+    <link name="${tf_prefix_ext}${camera_name}_color_frame" />
+    <joint name="${tf_prefix_ext}${camera_name}_color_to_${tf_prefix_ext}${camera_name}_color_optical_joint" type="fixed">
       <origin xyz="0.0 0.0 0.0" rpy="${-pi/2} 0.0 ${-pi/2}" />
-      <parent link="${prefix}${camera_name}_color_frame" />
-      <child link="${prefix}${camera_name}_color_optical_frame" />
+      <parent link="${tf_prefix_ext}${camera_name}_color_frame" />
+      <child link="${tf_prefix_ext}${camera_name}_color_optical_frame" />
     </joint>
-    <link name="${prefix}${camera_name}_depth_optical_frame" />
-    <joint name="${prefix}${camera_name}_depth_to_${prefix}${camera_name}_depth_optical_joint" type="fixed">
+    <link name="${tf_prefix_ext}${camera_name}_depth_optical_frame" />
+    <joint name="${tf_prefix_ext}${camera_name}_depth_to_${tf_prefix_ext}${camera_name}_depth_optical_joint" type="fixed">
       <origin xyz="0.0 0.0 0.0" rpy="${-pi/2} 0.0 ${-pi/2}" />
-      <parent link="${prefix}${camera_name}_depth_frame" />
-      <child link="${prefix}${camera_name}_depth_optical_frame" />
+      <parent link="${tf_prefix_ext}${camera_name}_depth_frame" />
+      <child link="${tf_prefix_ext}${camera_name}_depth_optical_frame" />
     </joint>
-    <link name="${prefix}${camera_name}_color_optical_frame" />
+    <link name="${tf_prefix_ext}${camera_name}_color_optical_frame" />
     <xacro:if value="${simulation_engine == 'ignition-gazebo'}">
-      <gazebo reference="${prefix}${camera_name}_orbbec_astra_link">
-        <sensor type="rgbd_camera" name="${prefix}${camera_name}_orbbec_astra_camera">
+      <gazebo reference="${tf_prefix_ext}${camera_name}_orbbec_astra_link">
+        <sensor type="rgbd_camera" name="${tf_prefix_ext}${camera_name}_orbbec_astra_camera">
           <always_on>true</always_on>
           <update_rate>20.0</update_rate>
           <topic>${camera_name}</topic>
           <!-- It is not possible to split the frame of the color and the depth stream.
-               The frame of color stream should be ${prefix}${camera_name}_color_optical_frame -->
-          <ignition_frame_id>${prefix}${camera_name}_depth_optical_frame</ignition_frame_id>
-          <camera name="${prefix}camera">
+               The frame of color stream should be ${tf_prefix_ext}${camera_name}_color_optical_frame -->
+          <ignition_frame_id>${tf_prefix_ext}${camera_name}_depth_optical_frame</ignition_frame_id>
+          <camera name="${tf_prefix_ext}camera">
             <horizontal_fov>${60.0/180.0*pi}</horizontal_fov>
             <image>
@@ -99,9 +99,9 @@
     </xacro:if>
     <xacro:if value="${simulation_engine == 'gazebo-classic'}">
-      <gazebo reference="${prefix}orbbec_astra_link">
-        <sensor type="depth" name="${prefix}orbbec_astra_camera">
+      <gazebo reference="${tf_prefix_ext}orbbec_astra_link">
+        <sensor type="depth" name="${tf_prefix_ext}orbbec_astra_camera">
           <always_on>true</always_on>
           <update_rate>20.0</update_rate>
-          <camera name="${prefix}camera">
+          <camera name="${tf_prefix_ext}camera">
             <horizontal_fov>${60.0/180.0*pi}</horizontal_fov>
             <image>
@@ -111,5 +111,5 @@
             </image>
           </camera>
-          <plugin name="${prefix}orbbec_astra_camera" filename="libgazebo_ros_camera.so">
+          <plugin name="${tf_prefix_ext}orbbec_astra_camera" filename="libgazebo_ros_camera.so">
             <ros>
               <namespace>orbbec_astra_camera</namespace>
@@ -120,6 +120,6 @@
               <remapping>custom_camera/points:=depth/points</remapping>
             </ros>
-            <camera_name>${prefix}camera</camera_name>
-            <frame_name>${prefix}${frame_id}</frame_name>
+            <camera_name>${tf_prefix_ext}camera</camera_name>
+            <frame_name>${tf_prefix_ext}${frame_id}</frame_name>
             <hack_baseline>0.07</hack_baseline>
             <min_depth>0.6</min_depth>

File: urdf/ouster_os1_32.urdf.xacro (robot description, xacro)
@@ -17,15 +17,15 @@
     </xacro:unless>
     <xacro:if value="${tf_prefix == 'None'}">
-      <xacro:property name="prefix" value="" />
+      <xacro:property name="tf_prefix_ext" value="" />
     </xacro:if>
     <xacro:unless value="${tf_prefix == 'None'}">
-      <xacro:property name="prefix" value="${tf_prefix}" />
+      <xacro:property name="tf_prefix_ext" value="${tf_prefix}" />
     </xacro:unless>
-    <joint name="${parent_link.rstrip('_link')}_to_${prefix}ouster_os1_32_joint" type="fixed">
+    <joint name="${parent_link.rstrip('_link')}_to_${tf_prefix_ext}ouster_os1_32_joint" type="fixed">
       <origin xyz="${xyz}" rpy="${rpy}" />
       <parent link="${parent_link}" />
-      <child link="${prefix}ouster_os1_32_link" />
+      <child link="${tf_prefix_ext}ouster_os1_32_link" />
     </joint>
-    <link name="${prefix}ouster_os1_32_link">
+    <link name="${tf_prefix_ext}ouster_os1_32_link">
       <visual>
         <origin xyz="0.0 0.0 0.0" rpy="0.0 0.0 0.0" />
@@ -48,12 +48,12 @@
       </inertial>
     </link>
-    <joint name="${prefix}ouster_os1_32_to_${prefix}${frame_id.rstrip('_link')}_joint" type="fixed">
+    <joint name="${tf_prefix_ext}ouster_os1_32_to_${tf_prefix_ext}${frame_id.rstrip('_link')}_joint" type="fixed">
       <origin xyz="0.0 0.0 0.03618" rpy="0.0 0.0 0.0" />
-      <parent link="${prefix}ouster_os1_32_link" />
-      <child link="${prefix}${frame_id}" />
+      <parent link="${tf_prefix_ext}ouster_os1_32_link" />
+      <child link="${tf_prefix_ext}${frame_id}" />
     </joint>
-    <link name="${prefix}${frame_id}" />
-    <gazebo reference="${prefix}${frame_id}">
-      <sensor type="${ray_type}" name="${prefix}ouster_os1_32_sensor">
+    <link name="${tf_prefix_ext}${frame_id}" />
+    <gazebo reference="${tf_prefix_ext}${frame_id}">
+      <sensor type="${ray_type}" name="${tf_prefix_ext}ouster_os1_32_sensor">
         <visualize>false</visualize>
         <ray>
@@ -84,5 +84,5 @@
         </ray>
         <update_rate>20.0</update_rate>
-        <plugin name="${prefix}ouster_os1_32_${ray_type}" filename="libgazebo_ros_ray_sensor.so">
+        <plugin name="${tf_prefix_ext}ouster_os1_32_${ray_type}" filename="libgazebo_ros_ray_sensor.so">
           <ros>
             <namespace></namespace>
@@ -90,5 +90,5 @@
           </ros>
           <output_type>sensor_msgs/PointCloud2</output_type>
-          <frame_name>${prefix}${frame_id}</frame_name>
+          <frame_name>${tf_prefix_ext}${frame_id}</frame_name>
         </plugin>
       </sensor>

File: urdf/slamtec_rplidar_a2.urdf.xacro (robot description, xacro)
@@ -33,8 +33,8 @@
     </xacro:unless>
     <xacro:if value="${tf_prefix == 'None'}">
-      <xacro:property name="prefix" value="" />
+      <xacro:property name="tf_prefix_ext" value="" />
     </xacro:if>
     <xacro:unless value="${tf_prefix == 'None'}">
-      <xacro:property name="prefix" value="${tf_prefix}_" />
+      <xacro:property name="tf_prefix_ext" value="${tf_prefix}_" />
     </xacro:unless>
     <!--values of max distance are based on tradeoff values between best and worst case scenarios -->
@@ -55,10 +55,10 @@
       <xacro:property name="mesh" value="slamtec_rplidar_ax.dae" />
     </xacro:if>
-    <joint name="${parent_link.rstrip('_link')}_to_${prefix}slamtec_rplidar_a2_joint" type="fixed">
+    <joint name="${parent_link.rstrip('_link')}_to_${tf_prefix_ext}slamtec_rplidar_a2_joint" type="fixed">
       <origin xyz="${xyz}" rpy="${rpy}" />
       <parent link="${parent_link}" />
-      <child link="${prefix}slamtec_rplidar_a2_link" />
+      <child link="${tf_prefix_ext}slamtec_rplidar_a2_link" />
     </joint>
-    <link name="${prefix}slamtec_rplidar_a2_link">
+    <link name="${tf_prefix_ext}slamtec_rplidar_a2_link">
       <visual>
         <origin xyz="0.0 0.0 0.0" rpy="0.0 0.0 0.0" />
@@ -81,16 +81,16 @@
       </inertial>
     </link>
-    <joint name="${prefix}slamtec_rplidar_a2_to_${prefix}${frame_id.rstrip('_link')}_joint" type="fixed">
+    <joint name="${tf_prefix_ext}slamtec_rplidar_a2_to_${tf_prefix_ext}${frame_id.rstrip('_link')}_joint" type="fixed">
       <origin xyz="0.0 0.0 0.031" rpy="0.0 0.0 ${pi}" />
-      <parent link="${prefix}slamtec_rplidar_a2_link" />
-      <child link="${prefix}${frame_id}" />
+      <parent link="${tf_prefix_ext}slamtec_rplidar_a2_link" />
+      <child link="${tf_prefix_ext}${frame_id}" />
     </joint>
-    <link name="${prefix}${frame_id}" />
+    <link name="${tf_prefix_ext}${frame_id}" />
     <xacro:if value="${simulation_engine == 'ignition-gazebo'}">
-      <gazebo reference="${prefix}${frame_id}">
-        <sensor type="${ray_type}" name="${prefix}rplidar_a2_sensor">
+      <gazebo reference="${tf_prefix_ext}${frame_id}">
+        <sensor type="${ray_type}" name="${tf_prefix_ext}rplidar_a2_sensor">
           <topic>${topic}</topic>
-          <frame_id>${prefix}${frame_id}</frame_id>
-          <ignition_frame_id>${prefix}${frame_id}</ignition_frame_id>
+          <frame_id>${tf_prefix_ext}${frame_id}</frame_id>
+          <ignition_frame_id>${tf_prefix_ext}${frame_id}</ignition_frame_id>
           <update_rate>10.0</update_rate>
           <ray>
@@ -125,6 +125,6 @@
     </xacro:if>
     <xacro:if value="${simulation_engine == 'gazebo-classic'}">
-      <gazebo reference="${prefix}${frame_id}">
-        <sensor type="${ray_type}" name="${prefix}slamtec_rplidar_a2_sensor">
+      <gazebo reference="${tf_prefix_ext}${frame_id}">
+        <sensor type="${ray_type}" name="${tf_prefix_ext}slamtec_rplidar_a2_sensor">
           <visualize>false</visualize>
           <ray>
@@ -155,5 +155,5 @@
             </ros>
             <output_type>sensor_msgs/LaserScan</output_type>
-            <frame_name>${prefix}${frame_id}</frame_name>
+            <frame_name>${tf_prefix_ext}${frame_id}</frame_name>
           </plugin>
         </sensor>
