Commit message: Revert "Add prefix (#36)"
This reverts commit 4f1bc6fab4fd327a2d0f44dccfa7138ba06fbe95.

File: urdf/slamtec_rplidar_a3.urdf.xacro (robot description, xacro)
@@ -27,15 +27,15 @@
     </xacro:unless>
     <xacro:if value="${tf_prefix == 'None'}">
-      <xacro:property name="prefix" value="" />
+      <xacro:property name="tf_prefix_ext" value="" />
     </xacro:if>
     <xacro:unless value="${tf_prefix == 'None'}">
-      <xacro:property name="prefix" value="${tf_prefix}_" />
+      <xacro:property name="tf_prefix_ext" value="${tf_prefix}_" />
     </xacro:unless>
-    <joint name="${parent_link.rstrip('_link')}_to_${prefix}slamtec_rplidar_a3_joint" type="fixed">
+    <joint name="${parent_link.rstrip('_link')}_to_${tf_prefix_ext}slamtec_rplidar_a3_joint" type="fixed">
       <origin xyz="${xyz}" rpy="${rpy}" />
       <parent link="${parent_link}" />
-      <child link="${prefix}slamtec_rplidar_a3_link" />
+      <child link="${tf_prefix_ext}slamtec_rplidar_a3_link" />
     </joint>
-    <link name="${prefix}slamtec_rplidar_a3_link">
+    <link name="${tf_prefix_ext}slamtec_rplidar_a3_link">
       <visual>
         <origin xyz="0.0 0.0 0.0" rpy="0.0 0.0 0.0" />
@@ -59,16 +59,16 @@
       </inertial>
     </link>
-    <joint name="${prefix}slamtec_rplidar_a3_to_${prefix}${frame_id.rstrip('_link')}_joint" type="fixed">
+    <joint name="${tf_prefix_ext}slamtec_rplidar_a3_to_${tf_prefix_ext}${frame_id.rstrip('_link')}_joint" type="fixed">
       <origin xyz="0.0 0.0 0.031" rpy="0.0 0.0 ${pi}" />
-      <parent link="${prefix}slamtec_rplidar_a3_link" />
-      <child link="${prefix}${frame_id}" />
+      <parent link="${tf_prefix_ext}slamtec_rplidar_a3_link" />
+      <child link="${tf_prefix_ext}${frame_id}" />
     </joint>
-    <link name="${prefix}${frame_id}" />
+    <link name="${tf_prefix_ext}${frame_id}" />
     <xacro:if value="${simulation_engine == 'ignition-gazebo'}">
-      <gazebo reference="${prefix}${frame_id}">
-        <sensor type="${ray_type}" name="${prefix}rplidar_a3_sensor">
+      <gazebo reference="${tf_prefix_ext}${frame_id}">
+        <sensor type="${ray_type}" name="${tf_prefix_ext}rplidar_a3_sensor">
           <topic>${topic}</topic>
-          <frame_id>${prefix}${frame_id}</frame_id>
-          <ignition_frame_id>${prefix}${frame_id}</ignition_frame_id>
+          <frame_id>${tf_prefix_ext}${frame_id}</frame_id>
+          <ignition_frame_id>${tf_prefix_ext}${frame_id}</ignition_frame_id>
           <update_rate>10.0</update_rate>
           <ray>
@@ -104,6 +104,6 @@
     </xacro:if>
     <xacro:if value="${simulation_engine == 'gazebo-classic'}">
-      <gazebo reference="${prefix}${frame_id}">
-        <sensor type="${ray_type}" name="${prefix}slamtec_rplidar_a3_sensor">
+      <gazebo reference="${tf_prefix_ext}${frame_id}">
+        <sensor type="${ray_type}" name="${tf_prefix_ext}slamtec_rplidar_a3_sensor">
           <visualize>false</visualize>
           <ray>
@@ -135,5 +135,5 @@
             </ros>
             <output_type>sensor_msgs/LaserScan</output_type>
-            <frame_name>${prefix}${frame_id}</frame_name>
+            <frame_name>${tf_prefix_ext}${frame_id}</frame_name>
           </plugin>
         </sensor>

File: urdf/slamtec_rplidar_s1.urdf.xacro (robot description, xacro)
@@ -27,15 +27,15 @@
     </xacro:unless>
     <xacro:if value="${tf_prefix == 'None'}">
-      <xacro:property name="prefix" value="" />
+      <xacro:property name="tf_prefix_ext" value="" />
     </xacro:if>
     <xacro:unless value="${tf_prefix == 'None'}">
-      <xacro:property name="prefix" value="${tf_prefix}_" />
+      <xacro:property name="tf_prefix_ext" value="${tf_prefix}_" />
     </xacro:unless>
-    <joint name="${parent_link.rstrip('_link')}_to_${prefix}slamtec_rplidar_s1_joint" type="fixed">
+    <joint name="${parent_link.rstrip('_link')}_to_${tf_prefix_ext}slamtec_rplidar_s1_joint" type="fixed">
       <origin xyz="${xyz}" rpy="${rpy}" />
       <parent link="${parent_link}" />
-      <child link="${prefix}slamtec_rplidar_s1_link" />
+      <child link="${tf_prefix_ext}slamtec_rplidar_s1_link" />
     </joint>
-    <link name="${prefix}slamtec_rplidar_s1_link">
+    <link name="${tf_prefix_ext}slamtec_rplidar_s1_link">
       <visual>
         <origin xyz="0.0 0.0 0.0" rpy="0.0 0.0 0.0" />
@@ -66,16 +66,16 @@
       </inertial>
     </link>
-    <joint name="${prefix}slamtec_rplidar_s1_to_${prefix}${frame_id.rstrip('_link')}_joint" type="fixed">
+    <joint name="${tf_prefix_ext}slamtec_rplidar_s1_to_${tf_prefix_ext}${frame_id.rstrip('_link')}_joint" type="fixed">
       <origin xyz="0.0 0.0 0.04" rpy="0.0 0.0 ${pi}" />
-      <parent link="${prefix}slamtec_rplidar_s1_link" />
-      <child link="${prefix}${frame_id}" />
+      <parent link="${tf_prefix_ext}slamtec_rplidar_s1_link" />
+      <child link="${tf_prefix_ext}${frame_id}" />
     </joint>
-    <link name="${prefix}${frame_id}" />
+    <link name="${tf_prefix_ext}${frame_id}" />
     <xacro:if value="${simulation_engine == 'ignition-gazebo'}">
-      <gazebo reference="${prefix}${frame_id}">
-        <sensor type="${ray_type}" name="${prefix}rplidar_s1_sensor">
+      <gazebo reference="${tf_prefix_ext}${frame_id}">
+        <sensor type="${ray_type}" name="${tf_prefix_ext}rplidar_s1_sensor">
           <topic>${topic}</topic>
-          <frame_id>${prefix}${frame_id}</frame_id>
-          <ignition_frame_id>${prefix}${frame_id}</ignition_frame_id>
+          <frame_id>${tf_prefix_ext}${frame_id}</frame_id>
+          <ignition_frame_id>${tf_prefix_ext}${frame_id}</ignition_frame_id>
           <update_rate>10.0</update_rate>
           <ray>
@@ -110,6 +110,6 @@
     </xacro:if>
     <xacro:if value="${simulation_engine == 'gazebo-classic'}">
-      <gazebo reference="${prefix}${frame_id}">
-        <sensor type="${ray_type}" name="${prefix}slamtec_rplidar_s1_sensor">
+      <gazebo reference="${tf_prefix_ext}${frame_id}">
+        <sensor type="${ray_type}" name="${tf_prefix_ext}slamtec_rplidar_s1_sensor">
           <visualize>false</visualize>
           <ray>
@@ -140,5 +140,5 @@
             </ros>
             <output_type>sensor_msgs/LaserScan</output_type>
-            <frame_name>${prefix}${frame_id}</frame_name>
+            <frame_name>${tf_prefix_ext}${frame_id}</frame_name>
           </plugin>
         </sensor>

File: urdf/slamtec_rplidar_s2.urdf.xacro (robot description, xacro)
@@ -41,5 +41,5 @@
         <origin xyz="0.0 0.0 0.0" rpy="0.0 0.0 0.0" />
         <geometry>
-          <mesh filename="package://ros_components_description/meshes/slamtec_rplidar_s2.dae" />
+          <mesh filename="file://$(find ros_components_description)/meshes/slamtec_rplidar_s2.dae" />
         </geometry>
       </visual>

File: urdf/slamtec_rplidar_s3.urdf.xacro (robot description, xacro)
@@ -41,5 +41,5 @@
         <origin xyz="0.0 0.0 0.0" rpy="0.0 0.0 0.0" />
         <geometry>
-          <mesh filename="package://ros_components_description/meshes/slamtec_rplidar_s3.dae" />
+          <mesh filename="file://$(find ros_components_description)/meshes/slamtec_rplidar_s3.dae" />
         </geometry>
       </visual>

File: urdf/stereolabs_zed.urdf.xacro (robot description, xacro)
@@ -20,15 +20,8 @@
     params="parent_link xyz rpy
     model:=zed
-    tf_prefix:=None
     name:=camera
     topic:=camera
     use_nominal_extrinsics:=false
     simulation_engine:=ignition-gazebo">
-    <xacro:if value="${tf_prefix == 'None'}">
-      <xacro:property name="prefix" value="" />
-    </xacro:if>
-    <xacro:unless value="${tf_prefix == 'None'}">
-      <xacro:property name="prefix" value="${tf_prefix}_" />
-    </xacro:unless>
     <xacro:if value="${model == 'zed'}">
       <xacro:property name="baseline" value="0.12" />
@@ -80,12 +73,12 @@
     </xacro:if>
     <!-- Camera mounting point (the threaded screw hole in the bottom) -->
-    <link name="${prefix}${name}_link" />
-    <joint name="${prefix}${name}_base_joint" type="fixed">
+    <link name="${name}_link" />
+    <joint name="${name}_base_joint" type="fixed">
       <parent link="${parent_link}" />
-      <child link="${prefix}${name}_link" />
+      <child link="${name}_link" />
       <origin xyz="${xyz}" rpy="${rpy}" />
     </joint>
     <!-- Camera Center -->
-    <link name="${prefix}${name}_camera_center">
+    <link name="${name}_camera_center">
       <visual>
         <origin xyz="${screw_offset_x} 0 ${screw_offset_z}" rpy="0 0 0" />
@@ -103,60 +96,60 @@
       </collision>
     </link>
-    <joint name="${prefix}${name}_camera_center_joint" type="fixed">
-      <parent link="${prefix}${name}_link" />
-      <child link="${prefix}${name}_camera_center" />
+    <joint name="${name}_camera_center_joint" type="fixed">
+      <parent link="${name}_link" />
+      <child link="${name}_camera_center" />
       <origin xyz="0 0 ${height/2}" rpy="0 ${bottom_slope} 0" />
     </joint>
     <!-- Artificially Created Camera Center -->
-    <link name="${prefix}${name}_center_optical_frame" />
-    <joint name="${prefix}${name}_center_joint" type="fixed">
-      <parent link="${prefix}${name}_camera_center" />
-      <child link="${prefix}${name}_center_optical_frame" />
+    <link name="${name}_center_optical_frame" />
+    <joint name="${name}_center_joint" type="fixed">
+      <parent link="${name}_camera_center" />
+      <child link="${name}_center_optical_frame" />
       <origin xyz="0.01 0 0" rpy="0 0 0" />
     </joint>
     <!-- Left Camera -->
-    <link name="${prefix}${name}_left_camera_frame" />
-    <joint name="${prefix}${name}_left_camera_joint" type="fixed">
-      <parent link="${prefix}${name}_camera_center" />
-      <child link="${prefix}${name}_left_camera_frame" />
+    <link name="${name}_left_camera_frame" />
+    <joint name="${name}_left_camera_joint" type="fixed">
+      <parent link="${name}_camera_center" />
+      <child link="${name}_left_camera_frame" />
       <origin xyz="${optical_offset_x} ${baseline/2} 0" rpy="0 0 0" />
     </joint>
-    <link name="${prefix}${name}_left_camera_optical_frame" />
-    <joint name="${prefix}${name}_left_camera_optical_joint" type="fixed">
+    <link name="${name}_left_camera_optical_frame" />
+    <joint name="${name}_left_camera_optical_joint" type="fixed">
       <origin xyz="0 0 0" rpy="-${M_PI/2} 0.0 -${M_PI/2}" />
-      <parent link="${prefix}${name}_left_camera_frame" />
-      <child link="${prefix}${name}_left_camera_optical_frame" />
+      <parent link="${name}_left_camera_frame" />
+      <child link="${name}_left_camera_optical_frame" />
     </joint>
     <!-- Right Camera -->
-    <link name="${prefix}${name}_right_camera_frame" />
-    <joint name="${prefix}${name}_right_camera_joint" type="fixed">
-      <parent link="${prefix}${name}_camera_center" />
-      <child link="${prefix}${name}_right_camera_frame" />
+    <link name="${name}_right_camera_frame" />
+    <joint name="${name}_right_camera_joint" type="fixed">
+      <parent link="${name}_camera_center" />
+      <child link="${name}_right_camera_frame" />
       <origin xyz="${optical_offset_x} -${baseline/2} 0" rpy="0 0 0" />
     </joint>
-    <link name="${prefix}${name}_right_camera_optical_frame" />
-    <joint name="${prefix}${name}_right_camera_optical_joint" type="fixed">
+    <link name="${name}_right_camera_optical_frame" />
+    <joint name="${name}_right_camera_optical_joint" type="fixed">
       <origin xyz="0 0 0" rpy="-${M_PI/2} 0.0 -${M_PI/2}" />
-      <parent link="${prefix}${name}_right_camera_frame" />
-      <child link="${prefix}${name}_right_camera_optical_frame" />
+      <parent link="${name}_right_camera_frame" />
+      <child link="${name}_right_camera_optical_frame" />
     </joint>
     <!-- ZED2 Sensors -->
     <xacro:if value="${model == 'zed2'}">
-      <link name="${prefix}${name}_mag_link" />
-      <joint name="${prefix}${name}_mag_joint" type="fixed">
-        <parent link="${prefix}${name}_camera_center" />
-        <child link="${prefix}${name}_mag_link" />
+      <link name="${name}_mag_link" />
+      <joint name="${name}_mag_joint" type="fixed">
+        <parent link="${name}_camera_center" />
+        <child link="${name}_mag_link" />
         <origin xyz="0 0 0" rpy="0 0 0" />
       </joint>
-      <link name="${prefix}${name}_baro_link" />
-      <joint name="${prefix}${name}_baro_joint" type="fixed">
-        <parent link="${prefix}${name}_camera_center" />
-        <child link="${prefix}${name}_baro_link" />
+      <link name="${name}_baro_link" />
+      <joint name="${name}_baro_joint" type="fixed">
+        <parent link="${name}_camera_center" />
+        <child link="${name}_baro_link" />
         <origin xyz="0 0 0" rpy="0 0 0" />
       </joint>
-      <link name="${prefix}${name}_temp_left_link" />
-      <joint name="${prefix}${name}_temp_left_joint" type="fixed">
-        <parent link="${prefix}${name}_left_camera_frame" />
-        <child link="${prefix}${name}_temp_left_link" />
+      <link name="${name}_temp_left_link" />
+      <joint name="${name}_temp_left_joint" type="fixed">
+        <parent link="${name}_left_camera_frame" />
+        <child link="${name}_temp_left_link" />
         <origin xyz="0 0 0" rpy="0 0 0" />
       </joint>
@@ -166,11 +159,11 @@
       camera
         should be more accurate different frames and fovs can be set -->
-      <gazebo reference="${prefix}${name}_center_optical_frame">
-        <sensor type="camera" name="${prefix}${name}_color">
+      <gazebo reference="${name}_center_optical_frame">
+        <sensor type="camera" name="${name}_color">
           <always_on>true</always_on>
           <update_rate>30.0</update_rate>
           <topic>${model}/zed_node/rgb/image_rect_color</topic>
           <visualize>false</visualize>
-          <ignition_frame_id>${prefix}${name}_center_optical_frame</ignition_frame_id>
+          <ignition_frame_id>${name}_center_optical_frame</ignition_frame_id>
           <camera>
             <horizontal_fov>${110.0/180.0*pi}</horizontal_fov>
@@ -186,10 +179,10 @@
           </camera>
         </sensor>
-        <sensor type="depth_camera" name="${prefix}${name}_depth">
+        <sensor type="depth_camera" name="${name}_depth">
           <always_on>true</always_on>
           <update_rate>30.0</update_rate>
           <topic>${model}/zed_node/depth</topic>
           <visualize>false</visualize>
-          <ignition_frame_id>${prefix}${name}_center_optical_frame</ignition_frame_id>
+          <ignition_frame_id>${name}_center_optical_frame</ignition_frame_id>
           <camera>
             <horizontal_fov>${110.0/180.0*pi}</horizontal_fov>

File: urdf/velodyne_puck.urdf.xacro (robot description, xacro)
@@ -17,15 +17,15 @@
     </xacro:unless>
     <xacro:if value="${tf_prefix == 'None'}">
-      <xacro:property name="prefix" value="" />
+      <xacro:property name="tf_prefix_ext" value="" />
     </xacro:if>
     <xacro:unless value="${tf_prefix == 'None'}">
-      <xacro:property name="prefix" value="${tf_prefix}_" />
+      <xacro:property name="tf_prefix_ext" value="${tf_prefix}_" />
     </xacro:unless>
-    <joint name="${parent_link.rstrip('_link')}_to_${prefix}velodyne_puck_joint" type="fixed">
+    <joint name="${parent_link.rstrip('_link')}_to_${tf_prefix_ext}velodyne_puck_joint" type="fixed">
       <origin xyz="${xyz}" rpy="${rpy}" />
       <parent link="${parent_link}" />
-      <child link="${prefix}velodyne_puck_link" />
+      <child link="${tf_prefix_ext}velodyne_puck_link" />
     </joint>
-    <link name="${prefix}velodyne_puck_link">
+    <link name="${tf_prefix_ext}velodyne_puck_link">
       <visual>
         <origin xyz="0.0 0.0 0.0" rpy="0.0 0.0 0.0" />
@@ -48,13 +48,13 @@
       </inertial>
     </link>
-    <joint name="${prefix}velodyne_puck_to_${prefix}${frame_id.rstrip('_link')}_joint"
+    <joint name="${tf_prefix_ext}velodyne_puck_to_${tf_prefix_ext}${frame_id.rstrip('_link')}_joint"
       type="fixed">
       <origin xyz="0.0 0.0 0.0378" rpy="0.0 0.0 0.0" />
-      <parent link="${prefix}velodyne_puck_link" />
-      <child link="${prefix}${frame_id}" />
+      <parent link="${tf_prefix_ext}velodyne_puck_link" />
+      <child link="${tf_prefix_ext}${frame_id}" />
     </joint>
-    <link name="${prefix}${frame_id}" />
-    <gazebo reference="${prefix}${frame_id}">
-      <sensor type="${ray_type}" name="${prefix}velodyne_puck_sensor">
+    <link name="${tf_prefix_ext}${frame_id}" />
+    <gazebo reference="${tf_prefix_ext}${frame_id}">
+      <sensor type="${ray_type}" name="${tf_prefix_ext}velodyne_puck_sensor">
         <visualize>false</visualize>
         <update_rate>10.0</update_rate>
@@ -87,6 +87,6 @@
         <xacro:if value="${simulation_engine == 'ignition-gazebo'}">
           <topic>${topic}</topic>
-          <frame_id>${prefix}${frame_id}</frame_id>
-          <ignition_frame_id>${prefix}${frame_id}</ignition_frame_id>
+          <frame_id>${tf_prefix_ext}${frame_id}</frame_id>
+          <ignition_frame_id>${tf_prefix_ext}${frame_id}</ignition_frame_id>
           <always_on>true</always_on>
           <plugin filename="libignition-gazebo-sensors-system.so"
@@ -96,5 +96,5 @@
         </xacro:if>
         <xacro:if value="${simulation_engine == 'gazebo-classic'}">
-          <plugin name="${prefix}velodyne_puck_${ray_type}"
+          <plugin name="${tf_prefix_ext}velodyne_puck_${ray_type}"
             filename="libgazebo_ros_ray_sensor.so">
             <ros>
@@ -103,5 +103,5 @@
             </ros>
             <output_type>sensor_msgs/PointCloud2</output_type>
-            <frame_name>${prefix}${frame_id}</frame_name>
+            <frame_name>${tf_prefix_ext}${frame_id}</frame_name>
           </plugin>
         </xacro:if>

Commit message: realsense | added namespaces | changed topic of depth
Signed-off-by: Jakub Delicat <jakub.delicat@husarion.com>

File: urdf/intel_realsense_d435.urdf.xacro (robot description, xacro)
@@ -23,5 +23,12 @@
             topic:=camera
             use_nominal_extrinsics:=false
+            namespace:=None
             simulation_engine:=ignition-gazebo">
+    <xacro:if value="${namespace == 'None'}">
+      <xacro:property name="namespace_ext" value="" />
+    </xacro:if>
+    <xacro:unless value="${namespace == 'None'}">
+        <xacro:property name="namespace_ext" value="${namespace}/" />
+    </xacro:unless>
     <xacro:if value="${tf_prefix == 'None'}">
       <xacro:property name="prefix" value="" />
@@ -150,8 +157,8 @@
         should be more accurate for D435 - different frames and fovs can be set -->
       <gazebo reference="${prefix}${name}_link">
-        <sensor type="camera" name="${prefix}${name}_color">
+        <sensor type="camera" name="$${namespace_ext}{prefix}${name}_color">
           <always_on>true</always_on>
           <update_rate>30.0</update_rate>
-          <topic>${topic}/color/image_raw</topic>
+          <topic>${namespace_ext}${topic}/color/image_raw</topic>
           <visualize>false</visualize>
           <ignition_frame_id>${prefix}${name}_color_optical_frame</ignition_frame_id>
@@ -166,9 +173,12 @@
             <far>300.0</far>
           </clip>
+          <ros>
+            <namespace>${namespace_ext}</namespace>
+          </ros>
         </sensor>
-        <sensor type="depth_camera" name="${prefix}${name}_depth">
+        <sensor type="depth_camera" name="${namespace_ext}${prefix}${name}_depth">
           <always_on>true</always_on>
           <update_rate>30.0</update_rate>
-          <topic>${topic}/depth</topic>
+          <topic>${namespace_ext}${topic}/depth/image_raw</topic>
           <visualize>false</visualize>
           <ignition_frame_id>${prefix}${name}_depth_optical_frame</ignition_frame_id>
@@ -190,4 +200,7 @@
             </noise>
           </camera>
+          <ros>
+            <namespace>${namespace_ext}</namespace>
+          </ros>
         </sensor>
       </gazebo>
