Commit message: changed astra plugin | changed names of sensors for astra and realsense
Signed-off-by: Jakub Delicat <jakub.delicat@husarion.com>

File: urdf/intel_realsense_d435.urdf.xacro (robot description, xacro)
@@ -26,8 +26,8 @@
             simulation_engine:=ignition-gazebo">
     <xacro:if value="${namespace == 'None'}">
-      <xacro:property name="namespace_ext" value="" />
+      <xacro:property name="ns" value="" />
     </xacro:if>
     <xacro:unless value="${namespace == 'None'}">
-        <xacro:property name="namespace_ext" value="${namespace}/" />
+        <xacro:property name="ns" value="${namespace}/" />
     </xacro:unless>
     <xacro:if value="${tf_prefix == 'None'}">
@@ -158,8 +158,8 @@
       <gazebo reference="${prefix}${name}_link">
         <!-- https://github.com/IntelRealSense/realsense-ros#published-topics -->
-        <sensor type="camera" name="$${namespace_ext}{prefix}${name}_color">
+        <sensor type="camera" name="${ns}{prefix}${name}_intel_realsense_d435_color">
           <always_on>true</always_on>
           <update_rate>30.0</update_rate>
-          <topic>${namespace_ext}${topic}/color/image_raw</topic>
+          <topic>${ns}${topic}/color/image_raw</topic>
           <visualize>false</visualize>
           <ignition_frame_id>${prefix}${name}_color_optical_frame</ignition_frame_id>
@@ -175,11 +175,11 @@
           </clip>
           <ros>
-            <namespace>${namespace_ext}</namespace>
+            <namespace>${ns}</namespace>
           </ros>
         </sensor>
-        <sensor type="depth_camera" name="${namespace_ext}${prefix}${name}_depth">
+        <sensor type="depth_camera" name="${ns}${prefix}${name}_intel_realsense_d435_depth">
           <always_on>true</always_on>
           <update_rate>30.0</update_rate>
-          <topic>${namespace_ext}${topic}/depth/image_rect_raw</topic>
+          <topic>${ns}${topic}/depth/image_rect_raw</topic>
           <visualize>false</visualize>
           <ignition_frame_id>${prefix}${name}_depth_optical_frame</ignition_frame_id>
@@ -202,5 +202,5 @@
           </camera>
           <ros>
-            <namespace>${namespace_ext}</namespace>
+            <namespace>${ns}</namespace>
           </ros>
         </sensor>

File: urdf/orbbec_astra.urdf.xacro (robot description, xacro)
@@ -79,12 +79,31 @@
     <xacro:if value="${simulation_engine == 'ignition-gazebo'}">
       <gazebo reference="${prefix}${camera_name}_orbbec_astra_link">
-        <sensor type="rgbd_camera" name="${prefix}${camera_name}_orbbec_astra_camera">
+        <!-- https://github.com/orbbec/OrbbecSDK_ROS2#all-available-topics -->
+        <sensor type="camera" name="${ns}{prefix}${camera_name}_orbbec_astra_color">
           <always_on>true</always_on>
-          <update_rate>20.0</update_rate>
-          <topic>${ns}${camera_name}</topic>
-          <!-- It is not possible to split the frame of the color and the depth stream.
-               The frame of color stream should be ${prefix}${camera_name}_color_optical_frame -->
+          <update_rate>30.0</update_rate>
+          <topic>${ns}${camera_name}/color/image_raw</topic>
+          <visualize>false</visualize>
+          <ignition_frame_id>${prefix}${camera_name}_color_optical_frame</ignition_frame_id>
+          <horizontal_fov>${60.0/180.0*pi}</horizontal_fov>
+          <image>
+            <width>640</width>
+            <height>480</height>
+          </image>
+          <clip>
+            <near>0.6</near>
+            <far>8.0</far>
+          </clip>
+          <ros>
+            <namespace>${ns}</namespace>
+          </ros>
+        </sensor>
+        <sensor type="depth_camera" name="${ns}${prefix}${camera_name}_orbbec_astra_depth">
+          <always_on>true</always_on>
+          <update_rate>10.0</update_rate>
+          <topic>${ns}${camera_name}/depth/image_raw</topic>
+          <visualize>false</visualize>
           <ignition_frame_id>${prefix}${camera_name}_depth_optical_frame</ignition_frame_id>
-          <camera name="${prefix}camera">
+          <camera>
             <horizontal_fov>${60.0/180.0*pi}</horizontal_fov>
             <image>
@@ -96,4 +115,9 @@
               <far>8.0</far>
             </clip>
+            <noise>
+              <type>gaussian</type>
+              <mean>0.0</mean>
+              <stddev>0.005</stddev>
+            </noise>
           </camera>
           <ros>
