Commit message: Fixed <ros> tag in s3 | added namespace to velodyne puck
Signed-off-by: Jakub Delicat <jakub.delicat@husarion.com>

File: urdf/slamtec_rplidar_s3.urdf.xacro (robot description, xacro)
@@ -101,8 +101,8 @@
           <always_on>1</always_on>
           <visualize>false</visualize>
+          <ros>
+            <namespace>${ns}</namespace>
+          </ros>
         </sensor>
-        <ros>
-          <namespace>${ns}</namespace>
-        </ros>
       </gazebo>
     </xacro:if>

File: urdf/velodyne_puck.urdf.xacro (robot description, xacro)
@@ -7,5 +7,12 @@
                        topic:=scan
                        frame_id:=velodyne
+                       namespace:=None
                        simulation_engine:=gazebo-classic">
+    <xacro:if value="${namespace == 'None'}">
+      <xacro:property name="ns" value="" />
+    </xacro:if>
+    <xacro:unless value="${namespace == 'None'}">
+      <xacro:property name="ns" value="${namespace}/" />
+    </xacro:unless>
     <xacro:if value="${use_gpu}">
       <xacro:property name="ray_type" value="gpu_ray" />
@@ -56,5 +63,5 @@
     <link name="${prefix}${frame_id}" />
     <gazebo reference="${prefix}${frame_id}">
-      <sensor type="${ray_type}" name="${prefix}velodyne_puck_sensor">
+      <sensor type="${ray_type}" name="${ns}${prefix}velodyne_puck_sensor">
         <visualize>false</visualize>
         <update_rate>10.0</update_rate>
@@ -86,12 +93,8 @@
         </ray>
         <xacro:if value="${simulation_engine == 'ignition-gazebo'}">
-          <topic>${topic}</topic>
+          <topic>${ns}${topic}</topic>
           <frame_id>${prefix}${frame_id}</frame_id>
           <ignition_frame_id>${prefix}${frame_id}</ignition_frame_id>
           <always_on>true</always_on>
-          <plugin filename="libignition-gazebo-sensors-system.so"
-            name="ignition::gazebo::systems::Sensors">
-            <render_engine>ogre2</render_engine>
-          </plugin>
         </xacro:if>
         <xacro:if value="${simulation_engine == 'gazebo-classic'}">
@@ -106,4 +109,7 @@
           </plugin>
         </xacro:if>
+        <ros>
+          <namespace>${ns}</namespace>
+        </ros>
       </sensor>
     </gazebo>
