Commit message: ZED: Use package:// instead file://

File: urdf/stereolabs_zed.urdf.xacro (robot description, xacro)
@@ -84,5 +84,5 @@
         <origin xyz="${screw_offset_x} 0 ${screw_offset_z}" rpy="0 0 0" />
         <geometry>
-          <mesh filename="file://$(find ros_components_description)/meshes/${model}.stl" />
+          <mesh filename="package://ros_components_description/meshes/${model}.stl" />
         </geometry>
         <material name="mat">
@@ -92,5 +92,5 @@
       <collision>
         <geometry>
-          <mesh filename="file://$(find ros_components_description)/meshes/${model}.stl" />
+          <mesh filename="package://ros_components_description/meshes/${model}.stl" />
         </geometry>
       </collision>

Commit message: Added namespace to zed
Signed-off-by: Jakub Delicat <jakub.delicat@husarion.com>

File: urdf/stereolabs_zed.urdf.xacro (robot description, xacro)
@@ -24,5 +24,12 @@
     topic:=camera
     use_nominal_extrinsics:=false
+    namespace:=None
     simulation_engine:=ignition-gazebo">
+    <xacro:if value="${namespace == 'None'}">
+      <xacro:property name="ns" value="" />
+    </xacro:if>
+    <xacro:unless value="${namespace == 'None'}">
+      <xacro:property name="ns" value="${namespace}/" />
+    </xacro:unless>
     <xacro:if value="${tf_prefix == 'None'}">
       <xacro:property name="prefix" value="" />
@@ -167,8 +174,8 @@
         should be more accurate different frames and fovs can be set -->
       <gazebo reference="${prefix}${name}_center_optical_frame">
-        <sensor type="camera" name="${prefix}${name}_color">
+        <sensor type="camera" name="${ns}${prefix}${name}_stereolabs_zed_color">
           <always_on>true</always_on>
           <update_rate>30.0</update_rate>
-          <topic>${model}/zed_node/rgb/image_rect_color</topic>
+          <topic>${ns}${model}/zed_node/rgb/image_rect_color</topic>
           <visualize>false</visualize>
           <ignition_frame_id>${prefix}${name}_center_optical_frame</ignition_frame_id>
@@ -185,9 +192,12 @@
             </clip>
           </camera>
+          <ros>
+            <namespace>${ns}</namespace>
+          </ros>
         </sensor>
-        <sensor type="depth_camera" name="${prefix}${name}_depth">
+        <sensor type="depth_camera" name="${ns}${prefix}${name}_stereolabs_zed_depth">
           <always_on>true</always_on>
           <update_rate>30.0</update_rate>
-          <topic>${model}/zed_node/depth</topic>
+          <topic>${ns}${model}/zed_node/depth</topic>
           <visualize>false</visualize>
           <ignition_frame_id>${prefix}${name}_center_optical_frame</ignition_frame_id>
@@ -208,4 +218,7 @@
             </noise>
           </camera>
+          <ros>
+            <namespace>${ns}</namespace>
+          </ros>
         </sensor>
       </gazebo>

Commit message: Suggestions

File: urdf/stereolabs_zed.urdf.xacro (robot description, xacro)
@@ -20,9 +20,7 @@
     params="parent_link xyz rpy
     model:=zed
+    namespace:=None
     tf_prefix:=None
     name:=camera
-    topic:=camera
-    use_nominal_extrinsics:=false
-    namespace:=None
     simulation_engine:=ignition-gazebo">
     <xacro:if value="${namespace == 'None'}">
@@ -87,8 +85,8 @@
     </xacro:if>
     <!-- Camera mounting point (the threaded screw hole in the bottom) -->
-    <link name="${prefix}${name}_link" />
+    <link name="${prefix}${name}_camera_link" />
     <joint name="${prefix}${name}_base_joint" type="fixed">
       <parent link="${parent_link}" />
-      <child link="${prefix}${name}_link" />
+      <child link="${prefix}${name}_camera_link" />
       <origin xyz="${xyz}" rpy="${rpy}" />
     </joint>
@@ -177,5 +175,5 @@
           <always_on>true</always_on>
           <update_rate>30.0</update_rate>
-          <topic>${ns}zed/zed_node/rgb/image_rect_color</topic>
+          <topic>${ns}${prefix}${name}/zed_node/rgb/image_rect_color</topic>
           <visualize>false</visualize>
           <ignition_frame_id>${prefix}${name}_center_optical_frame</ignition_frame_id>
@@ -199,5 +197,5 @@
           <always_on>true</always_on>
           <update_rate>30.0</update_rate>
-          <topic>${ns}zed/zed_node/depth</topic>
+          <topic>${ns}${prefix}${name}/zed_node/depth</topic>
           <visualize>false</visualize>
           <ignition_frame_id>${prefix}${name}_center_optical_frame</ignition_frame_id>
